Commit message: Update urdf for ros2 control

File: src/rosbot_xl_description/models/rosbot_xl/rosbot_xl.urdf.xacro (robot description, xacro)
@@ -2,4 +2,5 @@
 <robot name="rosbot_xl" xmlns:xacro="http://www.ros.org/wiki/xacro">
   <xacro:arg name="use_sim" default="false" />
+  <!-- Why are we adding husarion namespace here? -->
   <xacro:include filename="$(find rosbot_xl_description)/models/rosbot_xl_base/rosbot_xl_macro.urdf.xacro" ns="husarion" />
   <xacro:husarion.rosbot_xl_robot use_sim="$(arg use_sim)" />

File: src/rosbot_xl_description/models/rosbot_xl_base/rosbot_xl_macro.urdf.xacro (robot description, xacro)
@@ -3,4 +3,5 @@
   <xacro:macro name="rosbot_xl_robot" params="use_sim">
     <xacro:property name="wheel_diameter" value="0.082" />
+    <xacro:property name="wheel_radius" value="${wheel_diameter/2.0}" />
     <!-- INCLUDE ROBOT PARTS DEFINITIONS -->
     <xacro:include filename="$(find rosbot_xl_description)/models/rosbot_xl_base/body.urdf.xacro" ns="body" />

File: src/rosbot_xl_description/models/rosbot_xl_base/wheel.urdf.xacro (robot description, xacro)
@@ -6,4 +6,6 @@
     <xacro:property name="wheel_separation_y" value="0.236" />
     <xacro:property name="wheel_thickness" value="0.032" />
+    <!-- for ros2_control -->
+    <xacro:property name="wheel_separation" value="${wheel_separation_x}" />
     <xacro:if value="${prefix == 'front_left'}">
       <xacro:property name="x" value="${wheel_separation_x/2}" />

Commit message: Basic ign ros bridge configuration

File: src/rosbot_xl_description/models/rosbot_xl/rosbot_xl.urdf.xacro (robot description, xacro)
@@ -4,3 +4,5 @@
   <xacro:include filename="$(find rosbot_xl_description)/models/rosbot_xl_base/rosbot_xl_macro.urdf.xacro" ns="husarion" />
   <xacro:husarion.rosbot_xl_robot use_sim="$(arg use_sim)" />
+  <xacro:include filename="$(find rosbot_xl_description)/models/rosbot_xl_components/slamtec_s1.ign.xacro" ns="lidar" />
+  <xacro:lidar.rplidar_s1 parent_link="cover_link" xyz="0.0 0.0 0.0" rpy="0.0 0.0 0.0" use_gpu="$(arg use_sim)" />
 </robot>

File: src/rosbot_xl_description/models/rosbot_xl_base/plugins.ign.xacro (robot description, xacro)
@@ -15,49 +15,99 @@
         <enable_metrics>false</enable_metrics>
         <pose relative_to='imu_link'>0 0 0 0 0 0</pose>
-        <angular_velocity>
-          <x>
-            <noise type="gaussian">
-              <mean>0.0</mean>
-              <stddev>1</stddev>
-            </noise>
-          </x>
-          <y>
-            <noise type="gaussian">
-              <mean>1.0</mean>
-              <stddev>1</stddev>
-            </noise>
-          </y>
-          <z>
-            <noise type="gaussian">
-              <mean>0.0</mean>
-              <stddev>1</stddev>
-            </noise>
-          </z>
-        </angular_velocity>
-        <linear_acceleration>
-          <x>
-            <noise type="gaussian">
-              <mean>0.0</mean>
-              <stddev>0.1</stddev>
-            </noise>
-          </x>
-          <y>
-            <noise type="gaussian">
-              <mean>0.0</mean>
-              <stddev>0.1</stddev>
-            </noise>
-          </y>
-          <z>
-            <noise type="gaussian">
-              <mean>0.0</mean>
-              <stddev>0.1</stddev>
-            </noise>
-          </z>
-        </linear_acceleration>
+        <imu>
+          <angular_velocity>
+            <x>
+              <noise type="gaussian">
+                <mean>0.0</mean>
+                <stddev>1</stddev>
+              </noise>
+            </x>
+            <y>
+              <noise type="gaussian">
+                <mean>1.0</mean>
+                <stddev>1</stddev>
+              </noise>
+            </y>
+            <z>
+              <noise type="gaussian">
+                <mean>0.0</mean>
+                <stddev>1</stddev>
+              </noise>
+            </z>
+          </angular_velocity>
+          <linear_acceleration>
+            <x>
+              <noise type="gaussian">
+                <mean>0.0</mean>
+                <stddev>0.1</stddev>
+              </noise>
+            </x>
+            <y>
+              <noise type="gaussian">
+                <mean>0.0</mean>
+                <stddev>0.1</stddev>
+              </noise>
+            </y>
+            <z>
+              <noise type="gaussian">
+                <mean>0.0</mean>
+                <stddev>0.1</stddev>
+              </noise>
+            </z>
+          </linear_acceleration>
+        </imu>
       </sensor>
     </gazebo>
-    <gazebo>
+    <!-- <gazebo>
       <plugin filename="ign_ros2_control-system" name="ign_ros2_control::IgnitionROS2ControlPlugin">
         <parameters>$(find rosbot_xl_description)/config/controllers.yaml</parameters>
+      </plugin>
+    </gazebo> -->
+    <gazebo>
+      <plugin
+        filename="libignition-gazebo-diff-drive-system.so"
+        name="ignition::gazebo::systems::DiffDrive">
+        <update_rate>10</update_rate>
+        <always_on>true</always_on>
+        <left_joint>front_left_wheel_joint</left_joint>
+        <right_joint>front_right_wheel_joint</right_joint>
+        <left_joint>rear_left_wheel_joint</left_joint>
+        <right_joint>rear_right_wheel_joint</right_joint>
+        <wheel_separation>0.192</wheel_separation>
+        <wheel_separation>0.192</wheel_separation>
+        <wheel_radius>${wheel_diameter}</wheel_radius>
+        <wheel_radius>${wheel_diameter}</wheel_radius>
+        <odom_publish_frequency>25</odom_publish_frequency>
+        <topic>cmd_vel</topic>
+        <odom_topic>odom/wheels</odom_topic>
+        <tf_topic>tf</tf_topic>
+        <child_frame_id>base_link</child_frame_id>
+      </plugin>
+    </gazebo>
+    <gazebo>
+      <plugin
+        filename="libignition-gazebo-pose-publisher-system.so"
+        name="ignition::gazebo::systems::PosePublisher">
+        <publish_link_pose>true</publish_link_pose>
+        <publish_nested_model_pose>true</publish_nested_model_pose>
+        <use_pose_vector_msg>true</use_pose_vector_msg>
+        <update_frequency>50</update_frequency>
+      </plugin>
+    </gazebo>
+    <gazebo>
+      <plugin
+        filename="libignition-gazebo-sensors-system.so"
+        name="ignition::gazebo::systems::Sensors">
+        <render_engine>ogre</render_engine>
+      </plugin>
+    </gazebo>
+    <gazebo>
+      <plugin
+        filename="libignition-gazebo-joint-state-publisher-system.so"
+        name="ignition::gazebo::systems::JointStatePublisher">
+        <joint name="front_left_wheel_joint"></joint>
+        <joint name="front_right_wheel_joint"></joint>
+        <joint name="rear_left_wheel_joint"></joint>
+        <joint name="rear_right_wheel_joint"></joint>
       </plugin>
     </gazebo>

Commit message: nav2 minimal config

File: src/rosbot_xl_description/models/rosbot_xl/rosbot_xl.urdf.xacro (robot description, xacro)
@@ -2,5 +2,6 @@
 <robot name="rosbot_xl" xmlns:xacro="http://www.ros.org/wiki/xacro">
   <xacro:arg name="use_sim" default="false" />
+  <xacro:arg name="use_gpu" default="false" />
   <xacro:include filename="$(find rosbot_xl_description)/models/rosbot_xl_base/rosbot_xl_macro.urdf.xacro" ns="husarion" />
-  <xacro:husarion.rosbot_xl_robot use_sim="$(arg use_sim)" />
+  <xacro:husarion.rosbot_xl_robot use_sim="$(arg use_sim)" use_gpu="$(arg use_gpu)" />
 </robot>

File: src/rosbot_xl_description/models/rosbot_xl_base/body.urdf.xacro (robot description, xacro)
@@ -18,29 +18,14 @@
       </collision>
       <inertial>
-          <mass value="3.0" />
-          <inertia ixx="1.0" ixy="0.0" ixz="0.0"
-                             iyy="1.0" iyz="0.0"
-                                       izz="0.0" />
+          <mass value="3.5" />
+        <origin xyz="-0.016319 -0.004036 0.02819" rpy="0.0 0.0 0.0"/>
+        <inertia ixx="0.0254042524427888" ixy="-0.0002000608350169362" ixz="-0.0009754256573561553"
+                                          iyy="0.028746423126319035"   iyz="-0.0002603325647592511"
+                                                                       izz="0.046227102375569866" />
       </inertial>
     </link>
     <link name="cover_link">
-      <inertial>
-        <mass value="0.0000001" />
-        <inertia ixx="1.0" ixy="0.0" ixz="0.0"
-                           iyy="1.0" iyz="0.0"
-                                     izz="0.0" />
-      </inertial>
     </link>
     <link name="imu_link">
-      <inertial>
-        <mass value="0.0000001" />
-        <inertia ixx="1" ixy="0" ixz="0" iyy="1" iyz="0" izz="1" />
-      </inertial>
-    </link>
-    <link name="laser">
-      <inertial>
-        <mass value="0.0000001" />
-        <inertia ixx="1" ixy="0" ixz="0" iyy="1" iyz="0" izz="1" />
-      </inertial>
     </link>
     <joint name="base_link_to_body_joint" type="fixed">
@@ -54,9 +39,4 @@
       <child link="cover_link" />
     </joint>
-    <joint name="cover_to_laser_joint" type="fixed">
-      <origin xyz="0.0 0.0 0.08345" rpy="0.0 3.14 0.0" />
-      <parent link="cover_link" />
-      <child link="laser" />
-    </joint>
     <joint name="body_link_to_imu_link_joint" type="fixed">
       <origin xyz="-0.1369 -0.0419 0.0370" rpy="0.0 0.0 0.0" />

File: src/rosbot_xl_description/models/rosbot_xl_base/rosbot_xl_macro.urdf.xacro (robot description, xacro)
@@ -1,5 +1,5 @@
 <?xml version='1.0'?>
 <robot xmlns:xacro="http://wiki.ros.org/xacro">
-  <xacro:macro name="rosbot_xl_robot" params="use_sim">
+  <xacro:macro name="rosbot_xl_robot" params="use_sim use_gpu">
     <xacro:property name="wheel_diameter" value="0.082" />
     <xacro:property name="wheel_radius" value="${wheel_diameter/2.0}" />
@@ -7,5 +7,5 @@
     <xacro:include filename="$(find rosbot_xl_description)/models/rosbot_xl_base/body.urdf.xacro" ns="body" />
     <xacro:include filename="$(find rosbot_xl_description)/models/rosbot_xl_base/wheel.urdf.xacro" ns="wheel" />
-    <!-- <xacro:include filename="$(find rosbot_xl_description)/models/rosbot_xl/gazebo_plugins.gazebo.xacro" ns="gazebo" /> -->
+    <xacro:include filename="$(find rosbot_xl_description)/models/rosbot_xl_base/plugins.gazebo.xacro" ns="gazebo" />
     <!-- BODY DECLARATION -->
     <xacro:body.body wheel_diameter="${wheel_diameter}" />
@@ -15,41 +15,6 @@
     <xacro:wheel.wheel wheel_type="differential" wheel_diameter="${wheel_diameter}" prefix="rear_left" />
     <xacro:wheel.wheel wheel_type="differential" wheel_diameter="${wheel_diameter}" prefix="rear_right" />
-    <ros2_control name="wheels" type="system">
-      <hardware>
-        <xacro:if value="${use_sim}">
-          <plugin>gazebo_ros2_control/GazeboSystem</plugin>
-        </xacro:if>
-        <xacro:unless value="${use_sim}">
-          <plugin>rosbot_xl_hardware/RosbotXLSystem</plugin>
-        </xacro:unless>
-      </hardware>
-      <joint name="front_left_wheel_joint">
-        <command_interface name="velocity"/>
-        <state_interface name="position"/>
-        <state_interface name="velocity"/>
-      </joint>
-      <joint name="front_right_wheel_joint">
-        <command_interface name="velocity"/>
-        <state_interface name="position"/>
-        <state_interface name="velocity"/>
-      </joint>
-      <joint name="rear_left_wheel_joint">
-        <command_interface name="velocity"/>
-        <state_interface name="position"/>
-        <state_interface name="velocity"/>
-      </joint>
-      <joint name="rear_right_wheel_joint">
-        <command_interface name="velocity"/>
-        <state_interface name="position"/>
-        <state_interface name="velocity"/>
-      </joint>
-    </ros2_control>
-    <gazebo>
-      <plugin filename="libgazebo_ros2_control.so" name="gazebo_ros2_control">
-        <robot_param>robot_description</robot_param>
-        <robot_param_node>robot_state_publisher</robot_param_node>
-        <parameters>$(find rosbot_xl_description)/config/controllers_gazebo.yaml</parameters>
-      </plugin>
-    </gazebo>
+    <xacro:gazebo.wheel_plugins />
+    <xacro:gazebo.rplidar_s1 xyz="0.0 0.0 0.0" rpy="0.0 0.0 0.0" use_gpu="${use_gpu}" />
   </xacro:macro>
 </robot>

File: src/rosbot_xl_description/models/rosbot_xl_base/wheel.urdf.xacro (robot description, xacro)
@@ -42,8 +42,8 @@
       </collision>
       <inertial>
-          <mass value="0.100" />
-          <inertia ixx="1.0" ixy="0.0" ixz="0.0"
-                             iyy="1.0" iyz="0.0"
-                                       izz="0.0" />
+          <mass value="0.051" />
+          <inertia  ixx="3.954e-05" ixy="0.000"     ixz="0.000"
+                                    iyy="7.116e-05" iyz="0.000"
+                                                    izz="4.032e-05" />
       </inertial>
     </link>
@@ -53,16 +53,9 @@
       <origin xyz="${x} ${y} 0.0" rpy="0.0 0.0 0.0" />
       <axis xyz="0.0 1.0 0.0" />
-      <limit effort="2.0"
-             velocity="5.0" />
-      <dynamics damping="0.1"
-                friction="0.1"/>
+      <limit effort="1.2"
+             velocity="21.0" />
+      <dynamics damping="0.001"
+                friction="0.001"/>
     </joint>
-    <gazebo reference="${prefix}_wheel_link">
-      <mu1 value="0.5" />
-      <mu2 value="0.5" />
-      <kp value="10000000.0" />
-      <kd value="1.0" />
-      <fdir1 value="1 0 0"/>
-    </gazebo>
   </xacro:macro>
 </robot>
