Commit message: Update to more detailed meshes | fix robot height

File: src/rosbot_xl_description/models/rosbot_xl_base/body.urdf.xacro (robot description, xacro)
@@ -2,5 +2,5 @@
 <robot xmlns:xacro="http://www.ros.org/wiki/xacro">
   <!-- body defining macro -->
-  <xacro:macro name="body" >
+  <xacro:macro name="body" params="wheel_diameter">
     <link name="base_link"></link>
     <link name="body_link">
@@ -39,5 +39,5 @@
     </link>
     <joint name="base_link_to_body_joint" type="fixed">
-      <origin xyz="0.0 0.0 ${0.105/2}" rpy="0.0 0.0 0.0" />
+      <origin xyz="0.0 0.0 ${wheel_diameter/2}" rpy="0.0 0.0 0.0" />
       <parent link="base_link" />
       <child link="body_link" />

File: src/rosbot_xl_description/models/rosbot_xl_base/rosbot_xl_macro.urdf.xacro (robot description, xacro)
@@ -2,4 +2,5 @@
 <robot xmlns:xacro="http://wiki.ros.org/xacro">
   <xacro:macro name="rosbot_xl_robot" params="use_sim">
+    <xacro:property name="wheel_diameter" value="0.082" />
     <!-- INCLUDE ROBOT PARTS DEFINITIONS -->
     <xacro:include filename="$(find rosbot_xl_description)/models/rosbot_xl_base/body.urdf.xacro" ns="body" />
@@ -7,10 +8,10 @@
     <!-- <xacro:include filename="$(find rosbot_xl_description)/models/rosbot_xl/gazebo_plugins.gazebo.xacro" ns="gazebo" /> -->
     <!-- BODY DECLARATION -->
-    <xacro:body.body />
+    <xacro:body.body wheel_diameter="${wheel_diameter}" />
     <!-- WHEEL DECLARATION -->
-    <xacro:wheel.wheel wheel_type="differential" prefix="front_left" />
-    <xacro:wheel.wheel wheel_type="differential" prefix="front_right" />
-    <xacro:wheel.wheel wheel_type="differential" prefix="rear_left" />
-    <xacro:wheel.wheel wheel_type="differential" prefix="rear_right" />
+    <xacro:wheel.wheel wheel_type="differential" wheel_diameter="${wheel_diameter}" prefix="front_left" />
+    <xacro:wheel.wheel wheel_type="differential" wheel_diameter="${wheel_diameter}" prefix="front_right" />
+    <xacro:wheel.wheel wheel_type="differential" wheel_diameter="${wheel_diameter}" prefix="rear_left" />
+    <xacro:wheel.wheel wheel_type="differential" wheel_diameter="${wheel_diameter}" prefix="rear_right" />
     <ros2_control name="wheels" type="system">
       <hardware>

File: src/rosbot_xl_description/models/rosbot_xl_base/wheel.urdf.xacro (robot description, xacro)
@@ -2,8 +2,7 @@
 <robot xmlns:xacro="http://www.ros.org/wiki/xacro">
   <!-- wheel defining macro -->
-  <xacro:macro name="wheel" params="wheel_type prefix">
+  <xacro:macro name="wheel" params="wheel_type wheel_diameter prefix">
     <xacro:property name="wheel_separation_x" value="0.170" />
     <xacro:property name="wheel_separation_y" value="0.236" />
-    <xacro:property name="wheel_diameter" value="0.082" />
     <xacro:property name="wheel_thickness" value="0.032" />
     <xacro:if value="${prefix == 'front_left'}">

Commit message: Working communication with PC

File: src/rosbot_xl_description/models/rosbot_xl_base/body.urdf.xacro (robot description, xacro)
@@ -38,4 +38,10 @@
       </inertial>
     </link>
+    <link name="laser">
+      <inertial>
+        <mass value="0.0000001" />
+        <inertia ixx="1" ixy="0" ixz="0" iyy="1" iyz="0" izz="1" />
+      </inertial>
+    </link>
     <joint name="base_link_to_body_joint" type="fixed">
       <origin xyz="0.0 0.0 ${wheel_diameter/2}" rpy="0.0 0.0 0.0" />
@@ -48,4 +54,9 @@
       <child link="cover_link" />
     </joint>
+    <joint name="cover_to_laser_joint" type="fixed">
+      <origin xyz="0.0 0.0 0.08345" rpy="0.0 3.14 0.0" />
+      <parent link="cover_link" />
+      <child link="laser" />
+    </joint>
     <joint name="body_link_to_imu_link_joint" type="fixed">
       <origin xyz="-0.1369 -0.0419 0.0370" rpy="0.0 0.0 0.0" />

Commit message: Fix docker simulation and paths in urdf files

File: src/rosbot_xl_description/models/rosbot_xl_base/body.urdf.xacro (robot description, xacro)
@@ -7,5 +7,5 @@
       <visual>
         <geometry>
-          <mesh filename="package://rosbot_xl_description/models/rosbot_xl_base/meshes/body.dae" scale="1 1 1"/>
+          <mesh filename="file://$(find rosbot_xl_description)/models/rosbot_xl_base/meshes/body.dae" scale="1 1 1"/>
         </geometry>
         <origin xyz="0.0 0.0 0.0" rpy="0.0 0.0 0.0"/>
@@ -13,5 +13,5 @@
       <collision>
         <geometry>
-          <mesh filename="package://rosbot_xl_description/models/rosbot_xl_base/meshes/body_colision.stl" scale="1 1 1" />
+          <mesh filename="file://$(find rosbot_xl_description)/models/rosbot_xl_base/meshes/body_colision.stl" scale="1 1 1" />
         </geometry>
         <origin xyz="0.0 0.0 0.00" rpy="0.0 0.0 0.0"/>

File: src/rosbot_xl_description/models/rosbot_xl_base/wheel.urdf.xacro (robot description, xacro)
@@ -9,20 +9,20 @@
       <xacro:property name="x" value="${wheel_separation_x/2}" />
       <xacro:property name="y" value="${wheel_separation_y/2}" />
-      <xacro:property name="mesh" value="package://rosbot_xl_description/models/rosbot_xl_base/meshes/wheel_a.dae" />
+      <xacro:property name="mesh" value="file://$(find rosbot_xl_description)/models/rosbot_xl_base/meshes/wheel_a.dae" />
     </xacro:if>
     <xacro:if value="${prefix == 'front_right'}">
       <xacro:property name="x" value="${wheel_separation_x/2}" />
       <xacro:property name="y" value="-${wheel_separation_y/2}" />
-      <xacro:property name="mesh" value="package://rosbot_xl_description/models/rosbot_xl_base/meshes/wheel_b.dae" />
+      <xacro:property name="mesh" value="file://$(find rosbot_xl_description)/models/rosbot_xl_base/meshes/wheel_b.dae" />
     </xacro:if>
     <xacro:if value="${prefix == 'rear_left'}">
       <xacro:property name="x" value="-${wheel_separation_x/2}" />
       <xacro:property name="y" value="${wheel_separation_y/2}" />
-      <xacro:property name="mesh" value="package://rosbot_xl_description/models/rosbot_xl_base/meshes/wheel_a.dae" />
+      <xacro:property name="mesh" value="file://$(find rosbot_xl_description)/models/rosbot_xl_base/meshes/wheel_a.dae" />
     </xacro:if>
     <xacro:if value="${prefix == 'rear_right'}">
       <xacro:property name="x" value="-${wheel_separation_x/2}" />
       <xacro:property name="y" value="-${wheel_separation_y/2}" />
-      <xacro:property name="mesh" value="package://rosbot_xl_description/models/rosbot_xl_base/meshes/wheel_b.dae" />
+      <xacro:property name="mesh" value="file://$(find rosbot_xl_description)/models/rosbot_xl_base/meshes/wheel_b.dae" />
     </xacro:if>
     <link name="${prefix}_wheel_link">

Commit message: Diff drive controller gazebo draft

File: src/rosbot_xl_description/models/rosbot_xl_base/body.urdf.xacro (robot description, xacro)
@@ -15,5 +15,5 @@
           <mesh filename="file://$(find rosbot_xl_description)/models/rosbot_xl_base/meshes/body_colision.stl" scale="1 1 1" />
         </geometry>
-        <origin xyz="0.0 0.0 0.00" rpy="0.0 0.0 0.0"/>
+        <origin xyz="0.0 0.0 0.0" rpy="0.0 0.0 0.0"/>
       </collision>
       <inertial>

File: src/rosbot_xl_description/models/rosbot_xl_base/rosbot_xl_macro.urdf.xacro (robot description, xacro)
@@ -3,9 +3,8 @@
   <xacro:macro name="rosbot_xl_robot" params="use_sim">
     <xacro:property name="wheel_diameter" value="0.082" />
-    <xacro:property name="wheel_radius" value="${wheel_diameter/2.0}" />
     <!-- INCLUDE ROBOT PARTS DEFINITIONS -->
     <xacro:include filename="$(find rosbot_xl_description)/models/rosbot_xl_base/body.urdf.xacro" ns="body" />
     <xacro:include filename="$(find rosbot_xl_description)/models/rosbot_xl_base/wheel.urdf.xacro" ns="wheel" />
-    <!-- <xacro:include filename="$(find rosbot_xl_description)/models/rosbot_xl/gazebo_plugins.gazebo.xacro" ns="gazebo" /> -->
+    <xacro:include filename="$(find rosbot_xl_description)/models/rosbot_xl_base/plugins.gazebo.xacro" ns="gazebo" />
     <!-- BODY DECLARATION -->
     <xacro:body.body wheel_diameter="${wheel_diameter}" />
@@ -15,4 +14,6 @@
     <xacro:wheel.wheel wheel_type="differential" wheel_diameter="${wheel_diameter}" prefix="rear_left" />
     <xacro:wheel.wheel wheel_type="differential" wheel_diameter="${wheel_diameter}" prefix="rear_right" />
+    <!-- GAZEBO PLUGINS DECLARATION -->
+    <xacro:gazebo.rosbot_gazebo_plugins />
     <ros2_control name="wheels" type="system">
       <hardware>
@@ -47,7 +48,5 @@
     <gazebo>
       <plugin filename="libgazebo_ros2_control.so" name="gazebo_ros2_control">
-        <robot_param>robot_description</robot_param>
-        <robot_param_node>robot_state_publisher</robot_param_node>
-        <parameters>$(find rosbot_xl_description)/config/controllers_gazebo.yaml</parameters>
+        <parameters>$(find rosbot_xl_description)/config/controllers.yaml</parameters>
       </plugin>
     </gazebo>

File: src/rosbot_xl_description/models/rosbot_xl_base/wheel.urdf.xacro (robot description, xacro)
@@ -53,8 +53,8 @@
       <origin xyz="${x} ${y} 0.0" rpy="0.0 0.0 0.0" />
       <axis xyz="0.0 1.0 0.0" />
-      <limit effort="2.0"
-             velocity="5.0" />
-      <dynamics damping="0.1"
-                friction="0.1"/>
+      <limit effort="1.2"
+             velocity="21.0" />
+      <dynamics damping="0.001"
+                friction="0.001"/>
     </joint>
     <gazebo reference="${prefix}_wheel_link">

Commit message: Fix inertia

File: src/rosbot_xl_description/models/rosbot_xl_base/body.urdf.xacro (robot description, xacro)
@@ -18,30 +18,13 @@
       </collision>
       <inertial>
-          <mass value="3.0" />
-          <inertia ixx="1.0" ixy="0.0" ixz="0.0"
-                             iyy="1.0" iyz="0.0"
-                                       izz="0.0" />
+        <mass value="3.5" />
+        <origin xyz="-0.016319 -0.004036 0.02819" rpy="0.0 0.0 0.0"/>
+        <inertia ixx="0.0254042524427888" ixy="-0.0002000608350169362" ixz="-0.0009754256573561553"
+                                          iyy="0.028746423126319035"   iyz="-0.0002603325647592511"
+                                                                       izz="0.046227102375569866" />
       </inertial>
     </link>
-    <link name="cover_link">
-      <inertial>
-        <mass value="0.0000001" />
-        <inertia ixx="1.0" ixy="0.0" ixz="0.0"
-                           iyy="1.0" iyz="0.0"
-                                     izz="0.0" />
-      </inertial>
-    </link>
-    <link name="imu_link">
-      <inertial>
-        <mass value="0.0000001" />
-        <inertia ixx="1" ixy="0" ixz="0" iyy="1" iyz="0" izz="1" />
-      </inertial>
-    </link>
-    <link name="laser">
-      <inertial>
-        <mass value="0.0000001" />
-        <inertia ixx="1" ixy="0" ixz="0" iyy="1" iyz="0" izz="1" />
-      </inertial>
-    </link>
+    <link name="cover_link"></link>
+    <link name="imu_link"></link>
     <joint name="base_link_to_body_joint" type="fixed">
       <origin xyz="0.0 0.0 ${wheel_diameter/2}" rpy="0.0 0.0 0.0" />
@@ -54,9 +37,4 @@
       <child link="cover_link" />
     </joint>
-    <joint name="cover_to_laser_joint" type="fixed">
-      <origin xyz="0.0 0.0 0.08345" rpy="0.0 3.14 0.0" />
-      <parent link="cover_link" />
-      <child link="laser" />
-    </joint>
     <joint name="body_link_to_imu_link_joint" type="fixed">
       <origin xyz="-0.1369 -0.0419 0.0370" rpy="0.0 0.0 0.0" />

File: src/rosbot_xl_description/models/rosbot_xl_base/plugins.ign.xacro (robot description, xacro)
@@ -3,5 +3,5 @@
   <xacro:macro name="rosbot_ign_plugins" >
     <!-- publish IMU -->
-    <!-- <gazebo reference="imu_link">
+    <gazebo reference="imu_link">
       <sensor name="imu_link" type="imu">
         <plugin
@@ -56,10 +56,10 @@
         </linear_acceleration>
       </sensor>
-    </gazebo> -->
-    <!-- <gazebo>
+    </gazebo>
+    <gazebo>
       <plugin filename="ign_ros2_control-system" name="ign_ros2_control::IgnitionROS2ControlPlugin">
         <parameters>$(find rosbot_xl_description)/config/controllers.yaml</parameters>
       </plugin>
-    </gazebo> -->
+    </gazebo>
   </xacro:macro>
 </robot>

File: src/rosbot_xl_description/models/rosbot_xl_base/rosbot_xl_macro.urdf.xacro (robot description, xacro)
@@ -46,9 +46,4 @@
       </joint>
     </ros2_control>
-    <gazebo>
-      <plugin filename="ign_ros2_control-system" name="ign_ros2_control::IgnitionROS2ControlPlugin">
-        <parameters>$(find rosbot_xl_description)/config/controllers.yaml</parameters>
-      </plugin>
-    </gazebo>
   </xacro:macro>
 </robot>

File: src/rosbot_xl_description/models/rosbot_xl_base/wheel.urdf.xacro (robot description, xacro)
@@ -42,8 +42,8 @@
       </collision>
       <inertial>
-          <mass value="0.100" />
-          <inertia ixx="1.0" ixy="0.0" ixz="0.0"
-                             iyy="1.0" iyz="0.0"
-                                       izz="0.0" />
+          <mass value="0.051" />
+          <inertia  ixx="3.954e-05" ixy="0.000"     ixz="0.000"
+                                    iyy="7.116e-05" iyz="0.000"
+                                                    izz="4.032e-05" />
       </inertial>
     </link>

Commit message: Fix imu link

File: src/rosbot_xl_description/models/rosbot_xl_base/body.urdf.xacro (robot description, xacro)
@@ -32,5 +32,5 @@
       </inertial>
     </link>
-    <link name="imu_link">
+    <link name="imu">
       <inertial>
         <mass value="0.0000001" />
@@ -59,8 +59,8 @@
       <child link="laser" />
     </joint>
-    <joint name="body_link_to_imu_link_joint" type="fixed">
-      <origin xyz="-0.1369 -0.0419 0.0370" rpy="0.0 0.0 0.0" />
+    <joint name="body_link_to_imu_joint" type="fixed">
+      <origin xyz="-0.1369 -0.0419 0.0370" rpy="3.14159 0.0 0.0" />
       <parent link="body_link" />
-      <child link="imu_link" />
+      <child link="imu" />
     </joint>
   </xacro:macro>
