Commit message: Fix laser transform

File: rosbot_xl_description/models/rosbot_xl_base/body.urdf.xacro (robot description, xacro)
@@ -50,5 +50,5 @@
     </joint>
     <joint name="cover_to_laser_joint" type="fixed">
-      <origin xyz="0.0 0.0 0.08345" rpy="0.0 3.14 0.0" />
+      <origin xyz="0.0 0.0 0.08345" rpy="0.0 0.0 3.14159" />
       <parent link="cover_link" />
       <child link="laser" />

Commit message: Fix lidar position

File: rosbot_xl_description/models/rosbot_xl_base/body.urdf.xacro (robot description, xacro)
@@ -50,5 +50,5 @@
     </joint>
     <joint name="cover_to_laser_joint" type="fixed">
-      <origin xyz="0.0 0.0 0.08345" rpy="0.0 0.0 3.14159" />
+      <origin xyz="0.0 0.0 0.04" rpy="0.0 0.0 3.14159" />
       <parent link="cover_link" />
       <child link="laser" />
