Commit message: Add antenna collision

File: rosbot_xl_description/urdf/components/antenna.urdf.xacro (robot description, xacro)
@@ -2,7 +2,7 @@
 <robot xmlns:xacro="http://www.ros.org/wiki/xacro">
   <xacro:macro name="antenna"
-               params="parent_link xyz rpy
-                       tf_prefix:=None
-                       antenna_angle:=0.0">
+    params="parent_link xyz rpy
+            tf_prefix:=None
+            antenna_angle:=0.0">
     <xacro:if value="${tf_prefix == 'None'}">
       <xacro:property name="tf_prefix_ext" value="" />
@@ -11,4 +11,6 @@
       <xacro:property name="tf_prefix_ext" value="${tf_prefix}_" />
     </xacro:unless>
+    <xacro:property name="antenna_length" value="0.1" />
+    <xacro:property name="antenna_radius" value="0.0052" />
     <joint name="${parent_link.rstrip('_link')}_to_${tf_prefix_ext}antenna_joint" type="fixed">
       <origin xyz="${xyz}" rpy="${rpy}" />
@@ -19,5 +21,6 @@
       <visual>
         <geometry>
-          <mesh filename="file://$(find rosbot_xl_description)/meshes/components/antenna.dae" scale="1 1 1" />
+          <mesh filename="file://$(find rosbot_xl_description)/meshes/components/antenna.dae"
+            scale="1 1 1" />
         </geometry>
         <origin xyz="0.0 0.0 0.0" rpy="0.0 0.0 0.0" />
@@ -32,15 +35,15 @@
       <visual>
         <geometry>
-          <mesh filename="file://$(find rosbot_xl_description)/meshes/components/antenna_top.dae" scale="1 1 1" />
+          <mesh filename="file://$(find rosbot_xl_description)/meshes/components/antenna_top.dae"
+            scale="1 1 1" />
         </geometry>
         <origin xyz="0.0 0.0 0.0" rpy="0.0 0.0 0.0" />
       </visual>
-      <!-- TODO update collision -->
-      <!-- <collision>
+      <collision>
         <geometry>
-          <mesh filename="file://$(find rosbot_xl_description)/meshes/antenna_top.dae" scale="1 1 1" />
+          <cylinder radius="${antenna_radius}" length="${antenna_length}" />
         </geometry>
-        <origin xyz="0.0 0.0 0.0" rpy="0.0 0.0 0.0" />
-      </collision> -->
+        <origin xyz="0.0 0.0 ${antenna_length/2.}" rpy="0.0 0.0 0.0" />
+      </collision>
     </link>
   </xacro:macro>

File: rosbot_xl_description/urdf/rosbot_xl.urdf.xacro (robot description, xacro)
@@ -5,4 +5,10 @@
   <xacro:include filename="$(find rosbot_xl_description)/urdf/rosbot_xl_macro.urdf.xacro" ns="husarion" />
   <xacro:husarion.rosbot_xl_robot use_sim="$(arg use_sim)" mecanum="$(arg mecanum)" />
+  <xacro:include filename="$(find rosbot_xl_description)/urdf/components/antenna.urdf.xacro" ns="antenna" />
+  <xacro:antenna.antenna
+    parent_link="body_link"
+    xyz="-0.155 -0.055 0.065"
+    rpy="0.0 0.0 0.0"
+    antenna_angle="0.0" />
   <xacro:include filename="$(find ros_components_description)/urdf/slamtec_rplidar_s1.urdf.xacro" ns="lidar" />
   <xacro:lidar.slamtec_rplidar_s1
@@ -13,9 +19,3 @@
     simulation_engine="ignition-gazebo" />
   <!-- use_gpu has to be set to true, CPU lidar doesn't work in ignition - https://github.com/gazebosim/gz-sensors/issues/26 -->
-  <xacro:include filename="$(find rosbot_xl_description)/urdf/components/antenna.urdf.xacro" ns="antenna" />
-  <xacro:antenna.antenna
-    parent_link="body_link"
-    xyz="-0.155 -0.055 0.065"
-    rpy="0.0 0.0 0.0"
-    antenna_angle="0.0" />
 </robot>

Commit message: Rename antenna links

File: rosbot_xl_description/urdf/components/antenna.urdf.xacro (robot description, xacro)
@@ -13,7 +13,21 @@
     <xacro:property name="antenna_length" value="0.1" />
     <xacro:property name="antenna_radius" value="0.0052" />
-    <joint name="${parent_link.rstrip('_link')}_to_${tf_prefix_ext}antenna_joint" type="fixed">
+    <joint name="${parent_link.rstrip('_link')}_to_${tf_prefix_ext}antenna_connector_joint" type="fixed">
       <origin xyz="${xyz}" rpy="${rpy}" />
       <parent link="${parent_link}" />
+      <child link="${tf_prefix_ext}antenna_connector_link" />
+    </joint>
+    <link name="${tf_prefix_ext}antenna_connector_link">
+      <visual>
+        <geometry>
+          <mesh filename="file://$(find rosbot_xl_description)/meshes/components/antenna_connector.dae"
+            scale="1 1 1" />
+        </geometry>
+        <origin xyz="0.0 0.0 0.0" rpy="0.0 0.0 0.0" />
+      </visual>
+    </link>
+    <joint name="${tf_prefix_ext}antenna_connector_to_${tf_prefix_ext}antenna_joint" type="fixed">
+      <origin xyz="-0.013 0.0 0.008" rpy="0.0 ${antenna_angle} 0.0" />
+      <parent link="${tf_prefix_ext}antenna_connector_link" />
       <child link="${tf_prefix_ext}antenna_link" />
     </joint>
@@ -22,18 +36,4 @@
         <geometry>
           <mesh filename="file://$(find rosbot_xl_description)/meshes/components/antenna.dae"
-            scale="1 1 1" />
-        </geometry>
-        <origin xyz="0.0 0.0 0.0" rpy="0.0 0.0 0.0" />
-      </visual>
-    </link>
-    <joint name="${tf_prefix_ext}antenna_to_${tf_prefix_ext}antenna_top_joint" type="fixed">
-      <origin xyz="-0.013 0.0 0.008" rpy="0.0 ${antenna_angle} 0.0" />
-      <parent link="${tf_prefix_ext}antenna_link" />
-      <child link="${tf_prefix_ext}antenna_top_link" />
-    </joint>
-    <link name="${tf_prefix_ext}antenna_top_link">
-      <visual>
-        <geometry>
-          <mesh filename="file://$(find rosbot_xl_description)/meshes/components/antenna_top.dae"
             scale="1 1 1" />
         </geometry>
