Commit message: Move simulation config to d435 urdf

File: rosbot_xl_description/urdf/components/d435.urdf.xacro (robot description, xacro)
@@ -2,4 +2,5 @@
 <!--
 # Copyright 2023 Intel Corporation. All Rights Reserved.
+# Copyright 2023 Husarion. All Rights Reserved.
 #
 # Licensed under the Apache License, Version 2.0 (the "License");
@@ -23,39 +24,46 @@
   <xacro:include filename="$(find realsense2_description)/urdf/_materials.urdf.xacro" />
   <xacro:include filename="$(find realsense2_description)/urdf/_usb_plug.urdf.xacro" />
-  <xacro:macro name="sensor_d435" params="parent *origin name:=camera use_nominal_extrinsics:=false add_plug:=false use_mesh:=true">
+  <xacro:macro name="sensor_d435"
+               params="parent *origin
+                       name:=camera
+                       use_nominal_extrinsics:=false
+                       add_plug:=false
+                       use_mesh:=true
+                       simulation_engine:=ignition-gazebo">
     <xacro:property name="M_PI" value="3.1415926535897931" />
     <!-- The following values are approximate, and the camera node
      publishing TF values with actual calibrated camera extrinsic values -->
-    <xacro:property name="d435_cam_depth_to_infra1_offset" value="0.0"/>
-    <xacro:property name="d435_cam_depth_to_infra2_offset" value="-0.050"/>
-    <xacro:property name="d435_cam_depth_to_color_offset" value="0.015"/>
+    <xacro:property name="d435_cam_depth_to_infra1_offset" value="0.0" />
+    <xacro:property name="d435_cam_depth_to_infra2_offset" value="-0.050" />
+    <xacro:property name="d435_cam_depth_to_color_offset" value="0.015" />
     <!-- The following values model the aluminum peripherial case for the
   	D435 camera, with the camera joint represented by the actual
   	peripherial camera tripod mount -->
-    <xacro:property name="d435_cam_width" value="0.090"/>
-    <xacro:property name="d435_cam_height" value="0.025"/>
-    <xacro:property name="d435_cam_depth" value="0.02505"/>
-    <xacro:property name="d435_cam_mount_from_center_offset" value="0.0149"/>
+    <xacro:property name="d435_cam_width" value="0.090" />
+    <xacro:property name="d435_cam_height" value="0.025" />
+    <xacro:property name="d435_cam_depth" value="0.02505" />
+    <xacro:property name="d435_cam_mount_from_center_offset" value="0.0149" />
     <!-- glass cover is 0.1 mm inwards from front aluminium plate -->
-    <xacro:property name="d435_glass_to_front" value="0.1e-3"/>
+    <xacro:property name="d435_glass_to_front" value="0.1e-3" />
     <!-- see datasheet Revision 007, Fig. 4-4 page 65 -->
-    <xacro:property name="d435_zero_depth_to_glass" value="4.2e-3"/>
+    <xacro:property name="d435_zero_depth_to_glass" value="4.2e-3" />
     <!-- convenience precomputation to avoid clutter-->
-    <xacro:property name="d435_mesh_x_offset" value="${d435_cam_mount_from_center_offset-d435_glass_to_front-d435_zero_depth_to_glass}"/>
+    <xacro:property name="d435_mesh_x_offset"
+      value="${d435_cam_mount_from_center_offset-d435_glass_to_front-d435_zero_depth_to_glass}" />
     <!-- The following offset is relative the the physical D435 camera peripherial
   	camera tripod mount -->
-    <xacro:property name="d435_cam_depth_px" value="${d435_cam_mount_from_center_offset}"/>
-    <xacro:property name="d435_cam_depth_py" value="0.0175"/>
-    <xacro:property name="d435_cam_depth_pz" value="${d435_cam_height/2}"/>
+    <xacro:property name="d435_cam_depth_px" value="${d435_cam_mount_from_center_offset}" />
+    <xacro:property name="d435_cam_depth_py" value="0.0175" />
+    <xacro:property name="d435_cam_depth_pz" value="${d435_cam_height/2}" />
     <!-- camera body, with origin at bottom screw mount -->
     <joint name="${name}_joint" type="fixed">
       <xacro:insert_block name="origin" />
-      <parent link="${parent}"/>
+      <parent link="${parent}" />
       <child link="${name}_bottom_screw_frame" />
     </joint>
-    <link name="${name}_bottom_screw_frame"/>
+    <link name="${name}_bottom_screw_frame" />
     <joint name="${name}_link_joint" type="fixed">
-      <origin xyz="${d435_mesh_x_offset} ${d435_cam_depth_py} ${d435_cam_depth_pz}" rpy="0 0 0"/>
-      <parent link="${name}_bottom_screw_frame"/>
+      <origin xyz="${d435_mesh_x_offset} ${d435_cam_depth_py} ${d435_cam_depth_pz}" rpy="0 0 0" />
+      <parent link="${name}_bottom_screw_frame" />
       <child link="${name}_link" />
     </joint>
@@ -64,5 +72,6 @@
         <xacro:if value="${use_mesh}">
           <!-- the mesh origin is at front plate in between the two infrared camera axes -->
-          <origin xyz="${d435_zero_depth_to_glass + d435_glass_to_front} ${-d435_cam_depth_py} 0" rpy="${M_PI/2} 0 ${M_PI/2}"/>
+          <origin xyz="${d435_zero_depth_to_glass + d435_glass_to_front} ${-d435_cam_depth_py} 0"
+            rpy="${M_PI/2} 0 ${M_PI/2}" />
           <geometry>
             <mesh filename="file://$(find realsense2_description)/meshes/d435.dae" />
@@ -70,15 +79,15 @@
         </xacro:if>
         <xacro:unless value="${use_mesh}">
-          <origin xyz="0 ${-d435_cam_depth_py} 0" rpy="0 0 0"/>
+          <origin xyz="0 ${-d435_cam_depth_py} 0" rpy="0 0 0" />
           <geometry>
-            <box size="${d435_cam_depth} ${d435_cam_width} ${d435_cam_height}"/>
+            <box size="${d435_cam_depth} ${d435_cam_width} ${d435_cam_height}" />
           </geometry>
-          <material name="aluminum"/>
+          <material name="aluminum" />
         </xacro:unless>
       </visual>
       <collision>
-        <origin xyz="0 ${-d435_cam_depth_py} 0" rpy="0 0 0"/>
+        <origin xyz="0 ${-d435_cam_depth_py} 0" rpy="0 0 0" />
         <geometry>
-          <box size="${d435_cam_depth} ${d435_cam_width} ${d435_cam_height}"/>
+          <box size="${d435_cam_depth} ${d435_cam_width} ${d435_cam_height}" />
         </geometry>
       </collision>
@@ -90,13 +99,14 @@
       </inertial>
     </link>
-    <!-- Use the nominal extrinsics between camera frames if the calibrated extrinsics aren't being published. e.g. running the device in simulation  -->
+    <!-- Use the nominal extrinsics between camera frames if the calibrated extrinsics aren't being
+    published. e.g. running the device in simulation  -->
     <xacro:if value="${use_nominal_extrinsics}">
       <!-- camera depth joints and links -->
       <joint name="${name}_depth_joint" type="fixed">
-        <origin xyz="0 0 0" rpy="0 0 0"/>
-        <parent link="${name}_link"/>
+        <origin xyz="0 0 0" rpy="0 0 0" />
+        <parent link="${name}_link" />
         <child link="${name}_depth_frame" />
       </joint>
-      <link name="${name}_depth_frame"/>
+      <link name="${name}_depth_frame" />
       <joint name="${name}_depth_optical_joint" type="fixed">
         <origin xyz="0 0 0" rpy="${-M_PI/2} 0 ${-M_PI/2}" />
@@ -104,5 +114,5 @@
         <child link="${name}_depth_optical_frame" />
       </joint>
-      <link name="${name}_depth_optical_frame"/>
+      <link name="${name}_depth_optical_frame" />
       <!-- camera left IR joints and links -->
       <joint name="${name}_infra1_joint" type="fixed">
@@ -111,5 +121,5 @@
         <child link="${name}_infra1_frame" />
       </joint>
-      <link name="${name}_infra1_frame"/>
+      <link name="${name}_infra1_frame" />
       <joint name="${name}_infra1_optical_joint" type="fixed">
         <origin xyz="0 0 0" rpy="${-M_PI/2} 0 ${-M_PI/2}" />
@@ -117,5 +127,5 @@
         <child link="${name}_infra1_optical_frame" />
       </joint>
-      <link name="${name}_infra1_optical_frame"/>
+      <link name="${name}_infra1_optical_frame" />
       <!-- camera right IR joints and links -->
       <joint name="${name}_infra2_joint" type="fixed">
@@ -124,5 +134,5 @@
         <child link="${name}_infra2_frame" />
       </joint>
-      <link name="${name}_infra2_frame"/>
+      <link name="${name}_infra2_frame" />
       <joint name="${name}_infra2_optical_joint" type="fixed">
         <origin xyz="0 0 0" rpy="${-M_PI/2} 0 ${-M_PI/2}" />
@@ -130,5 +140,5 @@
         <child link="${name}_infra2_optical_frame" />
       </joint>
-      <link name="${name}_infra2_optical_frame"/>
+      <link name="${name}_infra2_optical_frame" />
       <!-- camera color joints and links -->
       <joint name="${name}_color_joint" type="fixed">
@@ -137,5 +147,5 @@
         <child link="${name}_color_frame" />
       </joint>
-      <link name="${name}_color_frame"/>
+      <link name="${name}_color_frame" />
       <joint name="${name}_color_optical_joint" type="fixed">
         <origin xyz="0 0 0" rpy="${-M_PI/2} 0 ${-M_PI/2}" />
@@ -143,10 +153,61 @@
         <child link="${name}_color_optical_frame" />
       </joint>
-      <link name="${name}_color_optical_frame"/>
+      <link name="${name}_color_optical_frame" />
     </xacro:if>
     <xacro:if value="${add_plug}">
       <xacro:usb_plug parent="${name}_link" name="${name}_usb_plug">
-        <origin xyz="${d435_cam_mount_from_center_offset - 0.02095} ${-d435_cam_depth_py - 0.0353} 0" rpy="0 0 0"/>
+        <origin
+          xyz="${d435_cam_mount_from_center_offset - 0.02095} ${-d435_cam_depth_py - 0.0353} 0"
+          rpy="0 0 0" />
       </xacro:usb_plug>
+    </xacro:if>
+    <xacro:if value="${simulation_engine == 'ignition-gazebo'}">
+      <gazebo reference="camera_link">
+        <sensor name="d435_color" type="camera">
+          <update_rate>30.0</update_rate>
+          <always_on>true</always_on>
+          <visualize>false</visualize>
+          <topic>/d435/image_raw</topic>
+          <ignition_frame_id>camera_color_optical_frame</ignition_frame_id>
+          <horizontal_fov>1.204277184</horizontal_fov>
+          <image>
+            <width>1280</width>
+            <height>720</height>
+            <format>R8G8B8</format>
+          </image>
+          <clip>
+            <near>0.02</near>
+            <far>300</far>
+          </clip>
+        </sensor>
+        <sensor name="d435_depth" type="depth_camera">
+          <update_rate>30.0</update_rate>
+          <always_on>true</always_on>
+          <visualize>false</visualize>
+          <topic>/d435/depth_camera</topic>
+          <!-- Pointcloud is published in rosbot_xl/base_link/d435_depth, and there seem to be no
+          way to
+        change it, interestingly depth image is published correctly in the ignition_frame_id -->
+          <ignition_frame_id>camera_depth_frame</ignition_frame_id>
+          <horizontal_fov>1.518436449</horizontal_fov>
+          <image>
+            <width>1280</width>
+            <height>720</height>
+          </image>
+          <clip>
+            <near>0.28</near>
+            <far>8.0</far>
+          </clip>
+          <noise>
+            <type>gaussian</type>
+            <mean>0</mean>
+            <stddev>0.005</stddev>
+          </noise>
+          <plugin filename="libignition-gazebo-sensors-system.so"
+            name="ignition::gazebo::systems::Sensors">
+            <render_engine>ogre2</render_engine>
+          </plugin>
+        </sensor>
+      </gazebo>
     </xacro:if>
   </xacro:macro>

File: rosbot_xl_description/urdf/rosbot_xl_realsense.urdf.xacro (robot description, xacro)
@@ -21,56 +21,13 @@
     camera_mount_angle_1="0.0"
     camera_mount_angle_2="0.0" />
-  <!-- <xacro:include filename="$(find realsense2_description)/urdf/_d435.urdf.xacro" ns="camera" /> -->
   <xacro:include filename="$(find rosbot_xl_description)/urdf/components/d435.urdf.xacro"
     ns="camera" />
-  <xacro:camera.sensor_d435 parent="camera_mount_link" use_nominal_extrinsics="true"
-    add_plug="false" use_mesh="true">
+  <xacro:camera.sensor_d435
+    parent="camera_mount_link"
+    use_nominal_extrinsics="true"
+    add_plug="false"
+    use_mesh="true"
+    simulation_engine="ignition-gazebo">
     <origin xyz="0 0 0" rpy="0 0 0" />
   </xacro:camera.sensor_d435>
-  <gazebo reference="camera_link">
-    <sensor name="d435_color" type="camera">
-      <update_rate>30.0</update_rate>
-      <always_on>true</always_on>
-      <visualize>false</visualize>
-      <topic>/d435/image_raw</topic>
-      <ignition_frame_id>camera_color_optical_frame</ignition_frame_id>
-      <horizontal_fov>1.204277184</horizontal_fov>
-      <image>
-        <width>1280</width>
-        <height>720</height>
-        <format>R8G8B8</format>
-      </image>
-      <clip>
-        <near>0.02</near>
-        <far>300</far>
-      </clip>
-    </sensor>
-    <sensor name="d435_depth" type="depth_camera">
-      <update_rate>30.0</update_rate>
-      <always_on>true</always_on>
-      <visualize>false</visualize>
-      <topic>/d435/depth_camera</topic>
-      <!-- Pointcloud is published in rosbot_xl/base_link/d435_depth, and there seem to be no way to
-      change it, interestingly depth image is published correctly in the ignition_frame_id -->
-      <ignition_frame_id>camera_depth_frame</ignition_frame_id>
-      <horizontal_fov>1.518436449</horizontal_fov>
-      <image>
-        <width>1280</width>
-        <height>720</height>
-      </image>
-      <clip>
-        <near>0.28</near>
-        <far>8.0</far>
-      </clip>
-      <noise>
-        <type>gaussian</type>
-        <mean>0</mean>
-        <stddev>0.005</stddev>
-      </noise>
-      <plugin filename="libignition-gazebo-sensors-system.so"
-        name="ignition::gazebo::systems::Sensors">
-        <render_engine>ogre2</render_engine>
-      </plugin>
-    </sensor>
-  </gazebo>
 </robot>
