Commit message: Rename realsense xacro

File: rosbot_xl_description/urdf/components/intel_realsense_d435.urdf.xacro (robot description, xacro)
@@ -20,9 +20,9 @@
 aluminum peripherial evaluation case.
 -->
-<robot name="sensor_d435" xmlns:xacro="http://ros.org/wiki/xacro">
+<robot name="intel_realsense_d435" xmlns:xacro="http://ros.org/wiki/xacro">
   <!-- Includes -->
   <xacro:include filename="$(find realsense2_description)/urdf/_materials.urdf.xacro" />
   <xacro:include filename="$(find realsense2_description)/urdf/_usb_plug.urdf.xacro" />
-  <xacro:macro name="sensor_d435"
+  <xacro:macro name="intel_realsense_d435"
                params="parent *origin
                        name:=camera

File: rosbot_xl_description/urdf/rosbot_xl_realsense.urdf.xacro (robot description, xacro)
@@ -21,7 +21,7 @@
     camera_mount_angle_1="0.0"
     camera_mount_angle_2="0.0" />
-  <xacro:include filename="$(find rosbot_xl_description)/urdf/components/d435.urdf.xacro"
+  <xacro:include filename="$(find rosbot_xl_description)/urdf/components/intel_realsense_d435.urdf.xacro"
     ns="camera" />
-  <xacro:camera.sensor_d435
+  <xacro:camera.intel_realsense_d435
     parent="camera_mount_link"
     use_nominal_extrinsics="true"
@@ -30,4 +30,4 @@
     simulation_engine="ignition-gazebo">
     <origin xyz="0 0 0" rpy="0 0 0" />
-  </xacro:camera.sensor_d435>
+  </xacro:camera.intel_realsense_d435>
 </robot>

Commit message: Fix realsense collision x offset

File: rosbot_xl_description/urdf/components/intel_realsense_d435.urdf.xacro (robot description, xacro)
@@ -54,4 +54,5 @@
   	camera tripod mount -->
     <xacro:property name="d435_cam_depth_px" value="${d435_cam_mount_from_center_offset}" />
+    <xacro:property name="d435_collision_offset_x" value="0.00824" />
     <xacro:property name="d435_cam_depth_py" value="0.0175" />
     <xacro:property name="d435_cam_depth_pz" value="${d435_cam_height/2}" />
@@ -87,5 +88,5 @@
       </visual>
       <collision>
-        <origin xyz="0 ${-d435_cam_depth_py} 0" rpy="0 0 0" />
+        <origin xyz="${-d435_collision_offset_x} ${-d435_cam_depth_py} 0" rpy="0 0 0" />
         <geometry>
           <box size="${d435_cam_depth} ${d435_cam_width} ${d435_cam_height}" />
