Commit message: Add camera mount collisions and visuals

File: rosbot_xl_description/urdf/components/camera_mount.urdf.xacro (robot description, xacro)
@@ -19,5 +19,5 @@
     </joint>
     <link name="${tf_prefix_ext}camera_mount_bot_link">
-      <!-- <visual>
+      <visual>
         <geometry>
           <mesh filename="file://$(find rosbot_xl_description)/meshes/components/camera_mount_bot.dae"
@@ -25,14 +25,20 @@
         </geometry>
         <origin xyz="0.0 0.0 0.0" rpy="0.0 0.0 0.0" />
-      </visual> -->
+      </visual>
+      <collision>
+        <geometry>
+          <box size="0.0275 0.0275 0.023" />
+        </geometry>
+        <origin xyz="0.0 0.0 0.0115" rpy="0.0 0.0 0.0" />
+      </collision>
     </link>
     <joint name="${tf_prefix_ext}camera_mount_bot_to_${tf_prefix_ext}camera_mount_mid_joint"
       type="fixed">
-      <origin xyz="0.0 0.0 0.01" rpy="0.0 ${camera_mount_angle_1} 0.0" />
+      <origin xyz="0.0 0.0 0.016" rpy="0.0 ${camera_mount_angle_1} 0.0" />
       <parent link="${tf_prefix_ext}camera_mount_bot_link" />
       <child link="${tf_prefix_ext}camera_mount_mid_link" />
     </joint>
     <link name="${tf_prefix_ext}camera_mount_mid_link">
-      <!-- <visual>
+      <visual>
         <geometry>
           <mesh filename="file://$(find rosbot_xl_description)/meshes/components/camera_mount_mid.dae"
@@ -40,14 +46,20 @@
         </geometry>
         <origin xyz="0.0 0.0 0.0" rpy="0.0 0.0 0.0" />
-      </visual> -->
+      </visual>
+      <collision>
+        <geometry>
+          <box size="0.015 0.017 0.101" />
+        </geometry>
+        <origin xyz="0.0 0.0 0.0425" rpy="0.0 0.0 0.0" />
+      </collision>
     </link>
     <joint name="${tf_prefix_ext}camera_mount_mid_to_${tf_prefix_ext}camera_mount_top_joint"
       type="fixed">
-      <origin xyz="0.0 0.0 0.1" rpy="0.0 ${camera_mount_angle_2} 0.0" />
+      <origin xyz="0.0 0.0 0.1015" rpy="0.0 ${camera_mount_angle_2} 0.0" />
       <parent link="${tf_prefix_ext}camera_mount_mid_link" />
       <child link="${tf_prefix_ext}camera_mount_top_link" />
     </joint>
     <link name="${tf_prefix_ext}camera_mount_top_link">
-      <!-- <visual>
+      <visual>
         <geometry>
           <mesh filename="file://$(find rosbot_xl_description)/meshes/components/camera_mount_top.dae"
@@ -55,9 +67,15 @@
         </geometry>
         <origin xyz="0.0 0.0 0.0" rpy="0.0 0.0 0.0" />
-      </visual> -->
+      </visual>
+      <collision>
+        <geometry>
+          <box size="0.023 0.023 0.025" />
+        </geometry>
+        <origin xyz="0.0 0.0 0.0065" rpy="0.0 0.0 0.0" />
+      </collision>
     </link>
     <joint name="${tf_prefix_ext}camera_mount_top_to_${tf_prefix_ext}camera_mount_joint"
       type="fixed">
-      <origin xyz="0.0 0.0 0.01" rpy="0.0 0.0 0.0" />
+      <origin xyz="0.0 0.0 0.016" rpy="0.0 0.0 0.0" />
       <parent link="${tf_prefix_ext}camera_mount_top_link" />
       <child link="${tf_prefix_ext}camera_mount_link" />

Commit message: Fix top camera mount position

File: rosbot_xl_description/urdf/components/camera_mount.urdf.xacro (robot description, xacro)
@@ -56,5 +56,5 @@
     <joint name="${tf_prefix_ext}camera_mount_mid_to_${tf_prefix_ext}camera_mount_top_joint"
       type="fixed">
-      <origin xyz="0.0 0.0 0.1015" rpy="0.0 ${camera_mount_angle_2} 0.0" />
+      <origin xyz="0.0 0.0 0.086" rpy="0.0 ${camera_mount_angle_2} 0.0" />
       <parent link="${tf_prefix_ext}camera_mount_mid_link" />
       <child link="${tf_prefix_ext}camera_mount_top_link" />
@@ -72,10 +72,10 @@
           <box size="0.023 0.023 0.025" />
         </geometry>
-        <origin xyz="0.0 0.0 0.0065" rpy="0.0 0.0 0.0" />
+        <origin xyz="0.0 -0.00232 0.0065" rpy="0.0 0.0 0.0" />
       </collision>
     </link>
     <joint name="${tf_prefix_ext}camera_mount_top_to_${tf_prefix_ext}camera_mount_joint"
       type="fixed">
-      <origin xyz="0.0 0.0 0.016" rpy="0.0 0.0 0.0" />
+      <origin xyz="0.0 -0.00232 0.019" rpy="0.0 0.0 0.0" />
       <parent link="${tf_prefix_ext}camera_mount_top_link" />
       <child link="${tf_prefix_ext}camera_mount_link" />
