Commit message: Change friction settings in gazebo

File: rosbot_xl_description/urdf/wheel.urdf.xacro (robot description, xacro)
@@ -30,5 +30,5 @@
       <origin xyz="${x} ${y} 0.0" rpy="0.0 0.0 0.0" />
       <axis xyz="0.0 1.0 0.0" />
-      <limit effort="1.2" velocity="21.0" />
+      <limit effort="1.27" velocity="21.0" />
       <dynamics damping="0.001" friction="0.001" />
     </joint>
@@ -45,19 +45,4 @@
         </geometry>
         <origin xyz="0.0 0.0 0.0" rpy="${pi/2} 0.0 0.0" />
-        <surface>
-          <!-- Surface settings based on https://github.com/gazebosim/gz-sim/blob/gz-sim7/examples/worlds/diff_drive_skid.sdf -->
-          <friction>
-            <ode>
-              <mu>0.5</mu>
-              <mu2>1.0</mu2>
-              <fdir1>0 0 1</fdir1>
-            </ode>
-            <bullet>
-              <friction>1</friction>
-              <friction2>1</friction2>
-              <rolling_friction>0.1</rolling_friction>
-            </bullet>
-          </friction>
-        </surface>
       </collision>
       <inertial>
@@ -68,4 +53,11 @@
       </inertial>
     </link>
+    <gazebo reference="${prefix}_wheel_link">
+      <mu1 value="1.0" />
+      <mu2 value="0.5" />
+      <kp value="10000000.0" />
+      <kd value="1.0" />
+      <fdir1 value="1 0 0" />
+    </gazebo>
   </xacro:macro>
 </robot>

Commit message: Add mecanum meshes

File: rosbot_xl_description/urdf/wheel.urdf.xacro (robot description, xacro)
@@ -3,5 +3,4 @@
   <!-- wheel defining macro -->
   <xacro:macro name="wheel" params="wheel_radius prefix mecanum">
-    <xacro:property name="wheel_separation_y" value="0.236" />
     <xacro:property name="wheel_separation_x" value="0.170" />
     <xacro:if value="${mecanum}">
@@ -9,30 +8,30 @@
       <xacro:property name="wheel_thickness" value="0.05" />
       <xacro:property name="mass" value="0.4" />
-      <!-- TODO: change -->
-      <xacro:property name="ixx" value="3.954e-05" />
-      <xacro:property name="iyy" value="7.116e-05" />
-      <xacro:property name="izz" value="4.032e-05" />
+      <xacro:property name="ixx" value="0.003145" />
+      <xacro:property name="iyy" value="0.004561" />
+      <xacro:property name="izz" value="0.003145" />
+      <xacro:property name="wheel_separation_y" value="0.270" />
     </xacro:if>
     <xacro:unless value="${mecanum}">
+      <!-- todo: change meshes (they are old and too large) -->
       <xacro:property name="wheel_file" value="wheel" />
-      <xacro:property name="wheel_thickness" value="0.032" />
+      <xacro:property name="wheel_thickness" value="0.036" />
       <xacro:property name="mass" value="0.051" />
       <xacro:property name="ixx" value="3.954e-05" />
       <xacro:property name="iyy" value="7.116e-05" />
       <xacro:property name="izz" value="4.032e-05" />
+      <xacro:property name="wheel_separation_y" value="0.248" />
     </xacro:unless>
     <xacro:if value="${prefix == 'fl'}">
       <xacro:property name="x" value="${wheel_separation_x/2}" />
       <xacro:property name="y" value="${wheel_separation_y/2}" />
-      <xacro:property name="mesh" value="file://$(find rosbot_xl_description)/meshes/${wheel_file}_a.dae" />
-      <xacro:property name="visual_rotation" value="0" />
-      <xacro:property name="visual_offset" value="-0.015" />
+      <xacro:property name="mesh" value="file://$(find rosbot_xl_description)/meshes/${wheel_file}_b.dae" />
+      <xacro:property name="visual_rotation" value="${pi}" />
     </xacro:if>
     <xacro:if value="${prefix == 'fr'}">
       <xacro:property name="x" value="${wheel_separation_x/2}" />
       <xacro:property name="y" value="${-wheel_separation_y/2}" />
-      <xacro:property name="mesh" value="file://$(find rosbot_xl_description)/meshes/${wheel_file}_b.dae" />
+      <xacro:property name="mesh" value="file://$(find rosbot_xl_description)/meshes/${wheel_file}_a.dae" />
       <xacro:property name="visual_rotation" value="${pi}" />
-      <xacro:property name="visual_offset" value="0.015" />
     </xacro:if>
     <xacro:if value="${prefix == 'rl'}">
@@ -40,6 +39,5 @@
       <xacro:property name="y" value="${wheel_separation_y/2}" />
       <xacro:property name="mesh" value="file://$(find rosbot_xl_description)/meshes/${wheel_file}_a.dae" />
-      <xacro:property name="visual_rotation" value="0" />
-      <xacro:property name="visual_offset" value="-0.015" />
+      <xacro:property name="visual_rotation" value="${0.0}" />
     </xacro:if>
     <xacro:if value="${prefix == 'rr'}">
@@ -47,6 +45,5 @@
       <xacro:property name="y" value="${-wheel_separation_y/2}" />
       <xacro:property name="mesh" value="file://$(find rosbot_xl_description)/meshes/${wheel_file}_b.dae" />
-      <xacro:property name="visual_rotation" value="${pi}" />
-      <xacro:property name="visual_offset" value="0.015" />
+      <xacro:property name="visual_rotation" value="${0.0}" />
     </xacro:if>
     <joint name="${prefix}_wheel_joint" type="continuous">
@@ -63,5 +60,5 @@
           <mesh filename="${mesh}" scale="1 1 1" />
         </geometry>
-        <origin xyz="0.0 ${visual_offset} 0.0" rpy="0.0 0.0 ${visual_rotation}" />
+        <origin xyz="0.0 0.0 0.0" rpy="0.0 0.0 ${visual_rotation}" />
       </visual>
       <collision>
@@ -73,6 +70,6 @@
       <inertial>
         <mass value="${mass}" />
-        <inertia ixx="${ixx}" ixy="0.000"  ixz="0.000"
-                              iyy="${iyy}" iyz="0.000"
+        <inertia ixx="${ixx}" ixy="0.0"    ixz="0.0"
+                              iyy="${iyy}" iyz="0.0"
                                            izz="${izz}" />
       </inertial>

Commit message: Update tire wheels inertias

File: rosbot_xl_description/urdf/wheel.urdf.xacro (robot description, xacro)
@@ -14,11 +14,10 @@
     </xacro:if>
     <xacro:unless value="${mecanum}">
-      <!-- todo: change meshes (they are old and too large) -->
       <xacro:property name="wheel_file" value="wheel" />
       <xacro:property name="wheel_thickness" value="0.036" />
       <xacro:property name="mass" value="0.051" />
-      <xacro:property name="ixx" value="3.954e-05" />
-      <xacro:property name="iyy" value="7.116e-05" />
-      <xacro:property name="izz" value="4.032e-05" />
+      <xacro:property name="ixx" value="0.000050587413" />
+      <xacro:property name="iyy" value="0.000085933192" />
+      <xacro:property name="izz" value="0.000050587829" />
       <xacro:property name="wheel_separation_y" value="0.248" />
     </xacro:unless>

Commit message: Add mecanum simulation

File: rosbot_xl_description/urdf/wheel.urdf.xacro (robot description, xacro)
@@ -27,4 +27,5 @@
       <xacro:property name="mesh" value="file://$(find rosbot_xl_description)/meshes/${wheel_file}_b.dae" />
       <xacro:property name="visual_rotation" value="${pi}" />
+      <xacro:property name="fdir" value="1 -1 0" />
     </xacro:if>
     <xacro:if value="${prefix == 'fr'}">
@@ -33,4 +34,5 @@
       <xacro:property name="mesh" value="file://$(find rosbot_xl_description)/meshes/${wheel_file}_a.dae" />
       <xacro:property name="visual_rotation" value="${pi}" />
+      <xacro:property name="fdir" value="1 1 0" />
     </xacro:if>
     <xacro:if value="${prefix == 'rl'}">
@@ -39,4 +41,5 @@
       <xacro:property name="mesh" value="file://$(find rosbot_xl_description)/meshes/${wheel_file}_a.dae" />
       <xacro:property name="visual_rotation" value="${0.0}" />
+      <xacro:property name="fdir" value="1 1 0" />
     </xacro:if>
     <xacro:if value="${prefix == 'rr'}">
@@ -45,4 +48,5 @@
       <xacro:property name="mesh" value="file://$(find rosbot_xl_description)/meshes/${wheel_file}_b.dae" />
       <xacro:property name="visual_rotation" value="${0.0}" />
+      <xacro:property name="fdir" value="1 -1 0" />
     </xacro:if>
     <joint name="${prefix}_wheel_joint" type="continuous">
@@ -62,8 +66,16 @@
       </visual>
       <collision>
-        <geometry>
-          <cylinder radius="${wheel_radius}" length="${wheel_thickness}" />
-        </geometry>
-        <origin xyz="0.0 0.0 0.0" rpy="${pi/2} 0.0 0.0" />
+        <xacro:unless value="${mecanum}">
+          <geometry>
+            <cylinder radius="${wheel_radius}" length="${wheel_thickness}" />
+          </geometry>
+          <origin xyz="0.0 0.0 0.0" rpy="${pi/2} 0.0 0.0" />
+        </xacro:unless>
+        <xacro:if value="${mecanum}">
+          <!-- Mecanum simulation in ignition require wheels to be spheres -->
+          <geometry>
+            <sphere radius="${wheel_radius}" />
+          </geometry>
+        </xacro:if>
       </collision>
       <inertial>
@@ -74,10 +86,16 @@
       </inertial>
     </link>
-    <gazebo reference="${prefix}_wheel_link">
-      <mu1 value="1.0" />
-      <mu2 value="0.5" />
-      <kp value="10000000.0" />
-      <kd value="1.0" />
-      <fdir1 value="1 0 0" />
+    <gazebo reference="${prefix}_wheel_link" xmlns:ignition="http://ignitionrobotics.org/schema">
+      <collision>
+        <surface>
+          <friction>
+            <ode>
+              <mu>1.0</mu>
+              <mu2>0.0</mu2>
+              <fdir1 ignition:expressed_in="base_link">${fdir}</fdir1>
+            </ode>
+          </friction>
+        </surface>
+      </collision>
     </gazebo>
   </xacro:macro>

Commit message: Remove setting wheels collision to spheres in mecanum simulation
it wasn't necessary

File: rosbot_xl_description/urdf/wheel.urdf.xacro (robot description, xacro)
@@ -65,16 +65,8 @@
       </visual>
       <collision>
-        <xacro:if value="${not mecanum or not use_sim}">
-          <geometry>
-            <cylinder radius="${wheel_radius}" length="${wheel_thickness}" />
-          </geometry>
-          <origin xyz="0.0 0.0 0.0" rpy="${pi/2} 0.0 0.0" />
-        </xacro:if>
-        <!-- Mecanum simulation in ignition require wheels to be spheres -->
-        <xacro:if value="${mecanum and use_sim}">
-          <geometry>
-            <sphere radius="${wheel_radius}" />
-          </geometry>
-        </xacro:if>
+        <geometry>
+          <cylinder radius="${wheel_radius}" length="${wheel_thickness}" />
+        </geometry>
+        <origin xyz="0.0 0.0 0.0" rpy="${pi/2} 0.0 0.0" />
       </collision>
       <inertial>

Commit message: Fix mecanum wheels inertias

File: rosbot_xl_description/urdf/wheel.urdf.xacro (robot description, xacro)
@@ -7,7 +7,7 @@
       <xacro:property name="wheel_thickness" value="0.05" />
       <xacro:property name="mass" value="0.4" />
-      <xacro:property name="ixx" value="0.003145" />
-      <xacro:property name="iyy" value="0.004561" />
-      <xacro:property name="izz" value="0.003145" />
+      <xacro:property name="ixx" value="0.0003145" />
+      <xacro:property name="iyy" value="0.0004561" />
+      <xacro:property name="izz" value="0.0003145" />
       <xacro:property name="wheel_separation_y" value="0.270" />
     </xacro:if>

Commit message: changed rosbot_xl_gazebo to ament_python | added lidar tests and gazebo moving tests
Signed-off-by: Jakub Delicat <jakub.delicat@husarion.com>

File: rosbot_xl_description/urdf/wheel.urdf.xacro (robot description, xacro)
@@ -54,5 +54,5 @@
       <origin xyz="${x} ${y} 0.0" rpy="0.0 0.0 0.0" />
       <axis xyz="0.0 1.0 0.0" />
-      <limit effort="1.27" velocity="21.0" />
+      <limit effort="1.5" velocity="30.0" />
       <dynamics damping="0.001" friction="0.001" />
     </joint>
