Commit message: Rename imu link

File: rosbot_xl_description/urdf/body.urdf.xacro (robot description, xacro)
@@ -3,5 +3,5 @@
   <!-- body defining macro -->
   <xacro:macro name="body" params="wheel_radius">
-    <link name="base_link"></link>
+    <link name="base_link" />
     <joint name="base_link_to_body_joint" type="fixed">
       <origin xyz="0.0 0.0 ${wheel_radius}" rpy="0.0 0.0 0.0" />
@@ -36,10 +36,10 @@
     </joint>
     <link name="cover_link" />
-    <joint name="body_link_to_imu_joint" type="fixed">
+    <joint name="body_to_imu_joint" type="fixed">
       <origin xyz="-0.1369 -0.0419 0.0370" rpy="3.14159 0.0 0.0" />
       <parent link="body_link" />
-      <child link="imu" />
+      <child link="imu_link" />
     </joint>
-    <link name="imu">
+    <link name="imu_link">
       <inertial>
         <mass value="0.0000001" />

Commit message: Rename joint

File: rosbot_xl_description/urdf/body.urdf.xacro (robot description, xacro)
@@ -4,5 +4,5 @@
   <xacro:macro name="body" params="wheel_radius">
     <link name="base_link" />
-    <joint name="base_link_to_body_joint" type="fixed">
+    <joint name="base_to_body_joint" type="fixed">
       <origin xyz="0.0 0.0 ${wheel_radius}" rpy="0.0 0.0 0.0" />
       <parent link="base_link" />

Commit message: Fix robot inertia

File: rosbot_xl_description/urdf/body.urdf.xacro (robot description, xacro)
@@ -24,8 +24,8 @@
       <inertial>
         <mass value="3.5" />
-        <origin xyz="-0.016319 -0.004036 0.02819" rpy="0.0 0.0 0.0" />
-        <inertia ixx="0.0254042524427888" ixy="-0.0002000608350169362" ixz="-0.0009754256573561553"
-                                          iyy="0.028746423126319035"   iyz="-0.0002603325647592511"
-                                                                       izz="0.046227102375569866" />
+        <origin xyz="-0.0057 -0.0034 0.0358" rpy="0.0 0.0 0.0" />
+        <inertia ixx="0.01393" ixy="-0.000020968097" ixz="0.000010399694"
+                               iyy= "0.01081"        iyz="0.000059372953"
+                                                     izz="0.02048" />
       </inertial>
     </link>
@@ -41,12 +41,5 @@
       <child link="imu_link" />
     </joint>
-    <link name="imu_link">
-      <inertial>
-        <mass value="0.0000001" />
-        <inertia ixx="1" ixy="0" ixz="0"
-                         iyy="1" iyz="0"
-                                 izz="1" />
-      </inertial>
-    </link>
+    <link name="imu_link" />
   </xacro:macro>
 </robot>

Commit message: Remove center of mass xy offset
fixes center of rotation

File: rosbot_xl_description/urdf/body.urdf.xacro (robot description, xacro)
@@ -24,5 +24,5 @@
       <inertial>
         <mass value="3.5" />
-        <origin xyz="-0.0057 -0.0034 0.0358" rpy="0.0 0.0 0.0" />
+        <origin xyz="0.0 0.0 0.0358" rpy="0.0 0.0 0.0" />
         <inertia ixx="0.01393" ixy="-0.000020968097" ixz="0.000010399694"
                                iyy= "0.01081"        iyz="0.000059372953"

Commit message: Add use sim argument to wheel urdf

File: rosbot_xl_description/urdf/body.urdf.xacro (robot description, xacro)
@@ -1,5 +1,4 @@
 <?xml version="1.0" encoding="utf-8"?>
 <robot xmlns:xacro="http://www.ros.org/wiki/xacro">
-  <!-- body defining macro -->
   <xacro:macro name="body" params="wheel_radius">
     <link name="base_link" />

File: rosbot_xl_description/urdf/rosbot_xl_macro.urdf.xacro (robot description, xacro)
@@ -14,8 +14,8 @@
     <xacro:body.body wheel_radius="${wheel_radius}" />
     <!-- WHEEL DECLARATION -->
-    <xacro:wheel.wheel wheel_radius="${wheel_radius}" prefix="fl" mecanum="${mecanum}" />
-    <xacro:wheel.wheel wheel_radius="${wheel_radius}" prefix="fr" mecanum="${mecanum}" />
-    <xacro:wheel.wheel wheel_radius="${wheel_radius}" prefix="rl" mecanum="${mecanum}" />
-    <xacro:wheel.wheel wheel_radius="${wheel_radius}" prefix="rr" mecanum="${mecanum}" />
+    <xacro:wheel.wheel wheel_radius="${wheel_radius}" prefix="fl" mecanum="${mecanum}" use_sim="$(arg use_sim)" />
+    <xacro:wheel.wheel wheel_radius="${wheel_radius}" prefix="fr" mecanum="${mecanum}" use_sim="$(arg use_sim)" />
+    <xacro:wheel.wheel wheel_radius="${wheel_radius}" prefix="rl" mecanum="${mecanum}" use_sim="$(arg use_sim)" />
+    <xacro:wheel.wheel wheel_radius="${wheel_radius}" prefix="rr" mecanum="${mecanum}" use_sim="$(arg use_sim)" />
     <!-- ROS2 CONTROL -->
     <xacro:unless value="$(arg use_sim)">

File: rosbot_xl_description/urdf/wheel.urdf.xacro (robot description, xacro)
@@ -1,6 +1,5 @@
 <?xml version="1.0" encoding="utf-8"?>
 <robot xmlns:xacro="http://www.ros.org/wiki/xacro">
-  <!-- wheel defining macro -->
-  <xacro:macro name="wheel" params="wheel_radius prefix mecanum">
+  <xacro:macro name="wheel" params="wheel_radius prefix mecanum use_sim">
     <xacro:property name="wheel_separation_x" value="0.170" />
     <xacro:if value="${mecanum}">
@@ -66,12 +65,12 @@
       </visual>
       <collision>
-        <xacro:unless value="${mecanum}">
+        <xacro:if value="${not mecanum or not use_sim}">
           <geometry>
             <cylinder radius="${wheel_radius}" length="${wheel_thickness}" />
           </geometry>
           <origin xyz="0.0 0.0 0.0" rpy="${pi/2} 0.0 0.0" />
-        </xacro:unless>
-        <xacro:if value="${mecanum}">
-          <!-- Mecanum simulation in ignition require wheels to be spheres -->
+        </xacro:if>
+        <!-- Mecanum simulation in ignition require wheels to be spheres -->
+        <xacro:if value="${mecanum and use_sim}">
           <geometry>
             <sphere radius="${wheel_radius}" />
@@ -86,17 +85,19 @@
       </inertial>
     </link>
-    <gazebo reference="${prefix}_wheel_link" xmlns:ignition="http://ignitionrobotics.org/schema">
-      <collision>
-        <surface>
-          <friction>
-            <ode>
-              <mu>1.0</mu>
-              <mu2>0.0</mu2>
-              <fdir1 ignition:expressed_in="base_link">${fdir}</fdir1>
-            </ode>
-          </friction>
-        </surface>
-      </collision>
-    </gazebo>
+    <xacro:if value="${use_sim}">
+      <gazebo reference="${prefix}_wheel_link" xmlns:ignition="http://ignitionrobotics.org/schema">
+        <collision>
+          <surface>
+            <friction>
+              <ode>
+                <mu>1.0</mu>
+                <mu2>0.0</mu2>
+                <fdir1 ignition:expressed_in="base_link">${fdir}</fdir1>
+              </ode>
+            </friction>
+          </surface>
+        </collision>
+      </gazebo>
+    </xacro:if>
   </xacro:macro>
 </robot>

Commit message: file:// to package://

File: rosbot_xl_description/urdf/body.urdf.xacro (robot description, xacro)
@@ -11,5 +11,5 @@
       <visual>
         <geometry>
-          <mesh filename="file://$(find rosbot_xl_description)/meshes/body.dae" scale="1 1 1" />
+          <mesh filename="package://rosbot_xl_description/meshes/body.dae" scale="1 1 1" />
         </geometry>
         <origin xyz="0.0 0.0 0.0" rpy="0.0 0.0 0.0" />
@@ -17,5 +17,5 @@
       <collision>
         <geometry>
-          <mesh filename="file://$(find rosbot_xl_description)/meshes/body_colision.stl" scale="1 1 1" />
+          <mesh filename="package://rosbot_xl_description/meshes/body_colision.stl" scale="1 1 1" />
         </geometry>
         <origin xyz="0.0 0.0 0.0" rpy="0.0 0.0 0.0" />

File: rosbot_xl_description/urdf/components/antenna.urdf.xacro (robot description, xacro)
@@ -21,5 +21,5 @@
       <visual>
         <geometry>
-          <mesh filename="file://$(find rosbot_xl_description)/meshes/components/antenna_connector.dae"
+          <mesh filename="package://rosbot_xl_description/meshes/components/antenna_connector.dae"
             scale="1 1 1" />
         </geometry>
@@ -35,5 +35,5 @@
       <visual>
         <geometry>
-          <mesh filename="file://$(find rosbot_xl_description)/meshes/components/antenna.dae"
+          <mesh filename="package://rosbot_xl_description/meshes/components/antenna.dae"
             scale="1 1 1" />
         </geometry>

File: rosbot_xl_description/urdf/components/camera_mount.urdf.xacro (robot description, xacro)
@@ -21,5 +21,5 @@
       <visual>
         <geometry>
-          <mesh filename="file://$(find rosbot_xl_description)/meshes/components/camera_mount_bot.dae"
+          <mesh filename="package://rosbot_xl_description/meshes/components/camera_mount_bot.dae"
       scale="1 1 1" />
         </geometry>
@@ -42,5 +42,5 @@
       <visual>
         <geometry>
-          <mesh filename="file://$(find rosbot_xl_description)/meshes/components/camera_mount_mid.dae"
+          <mesh filename="package://rosbot_xl_description/meshes/components/camera_mount_mid.dae"
       scale="1 1 1" />
         </geometry>
@@ -63,5 +63,5 @@
       <visual>
         <geometry>
-          <mesh filename="file://$(find rosbot_xl_description)/meshes/components/camera_mount_top.dae"
+          <mesh filename="package://rosbot_xl_description/meshes/components/camera_mount_top.dae"
       scale="1 1 1" />
         </geometry>

File: rosbot_xl_description/urdf/wheel.urdf.xacro (robot description, xacro)
@@ -24,5 +24,5 @@
       <xacro:property name="x" value="${wheel_separation_x/2}" />
       <xacro:property name="y" value="${wheel_separation_y/2}" />
-      <xacro:property name="mesh" value="file://$(find rosbot_xl_description)/meshes/${wheel_file}_b.dae" />
+      <xacro:property name="mesh" value="package://rosbot_xl_description/meshes/${wheel_file}_b.dae" />
       <xacro:property name="visual_rotation" value="${pi}" />
       <xacro:property name="fdir" value="1 -1 0" />
@@ -31,5 +31,5 @@
       <xacro:property name="x" value="${wheel_separation_x/2}" />
       <xacro:property name="y" value="${-wheel_separation_y/2}" />
-      <xacro:property name="mesh" value="file://$(find rosbot_xl_description)/meshes/${wheel_file}_a.dae" />
+      <xacro:property name="mesh" value="package://rosbot_xl_description/meshes/${wheel_file}_a.dae" />
       <xacro:property name="visual_rotation" value="${pi}" />
       <xacro:property name="fdir" value="1 1 0" />
@@ -38,5 +38,5 @@
       <xacro:property name="x" value="${-wheel_separation_x/2}" />
       <xacro:property name="y" value="${wheel_separation_y/2}" />
-      <xacro:property name="mesh" value="file://$(find rosbot_xl_description)/meshes/${wheel_file}_a.dae" />
+      <xacro:property name="mesh" value="package://rosbot_xl_description/meshes/${wheel_file}_a.dae" />
       <xacro:property name="visual_rotation" value="${0.0}" />
       <xacro:property name="fdir" value="1 1 0" />
@@ -45,5 +45,5 @@
       <xacro:property name="x" value="${-wheel_separation_x/2}" />
       <xacro:property name="y" value="${-wheel_separation_y/2}" />
-      <xacro:property name="mesh" value="file://$(find rosbot_xl_description)/meshes/${wheel_file}_b.dae" />
+      <xacro:property name="mesh" value="package://rosbot_xl_description/meshes/${wheel_file}_b.dae" />
       <xacro:property name="visual_rotation" value="${0.0}" />
       <xacro:property name="fdir" value="1 -1 0" />
