Commit message: added tf_prefixes to the urdf
Signed-off-by: Jakub Delicat <jakub.delicat@husarion.com>

File: rosbot_xl_description/urdf/body.urdf.xacro (robot description, xacro)
@@ -1,12 +1,18 @@
 <?xml version="1.0" encoding="utf-8"?>
 <robot xmlns:xacro="http://www.ros.org/wiki/xacro">
-  <xacro:macro name="body" params="wheel_radius">
-    <link name="base_link" />
-    <joint name="base_to_body_joint" type="fixed">
+  <xacro:macro name="body" params="wheel_radius tf_prefix">
+    <xacro:if value="${tf_prefix == 'None'}">
+      <xacro:property name="tf_prefix_ext" value="" />
+    </xacro:if>
+    <xacro:unless value="${tf_prefix == 'None'}">
+      <xacro:property name="tf_prefix_ext" value="${tf_prefix}_" />
+    </xacro:unless>
+    <link name="${tf_prefix_ext}base_link" />
+    <joint name="${tf_prefix_ext}base_to_${tf_prefix_ext}body_joint" type="fixed">
       <origin xyz="0.0 0.0 ${wheel_radius}" rpy="0.0 0.0 0.0" />
-      <parent link="base_link" />
-      <child link="body_link" />
+      <parent link="${tf_prefix_ext}base_link" />
+      <child link="${tf_prefix_ext}body_link" />
     </joint>
-    <link name="body_link">
+    <link name="${tf_prefix_ext}body_link">
       <visual>
         <geometry>
@@ -29,16 +35,16 @@
       </inertial>
     </link>
-    <joint name="body_to_cover_joint" type="fixed">
+    <joint name="${tf_prefix_ext}body_to_${tf_prefix_ext}cover_joint" type="fixed">
       <origin xyz="0.0 0.0 0.08345" rpy="0.0 0.0 0.0" />
-      <parent link="body_link" />
-      <child link="cover_link" />
+      <parent link="${tf_prefix_ext}body_link" />
+      <child link="${tf_prefix_ext}cover_link" />
     </joint>
-    <link name="cover_link" />
-    <joint name="body_to_imu_joint" type="fixed">
+    <link name="${tf_prefix_ext}cover_link" />
+    <joint name="${tf_prefix_ext}body_to_${tf_prefix_ext}imu_joint" type="fixed">
       <origin xyz="-0.1369 -0.0419 0.0370" rpy="3.14159 0.0 0.0" />
-      <parent link="body_link" />
-      <child link="imu_link" />
+      <parent link="${tf_prefix_ext}body_link" />
+      <child link="${tf_prefix_ext}imu_link" />
     </joint>
-    <link name="imu_link" />
+    <link name="${tf_prefix_ext}imu_link" />
   </xacro:macro>
 </robot>

File: rosbot_xl_description/urdf/rosbot_xl.urdf.xacro (robot description, xacro)
@@ -9,19 +9,31 @@
   <xacro:arg name="simulation_controllers_config_file"
     default="$(find rosbot_xl_controller)/config/diff_drive_controller.yaml" />
+  <xacro:arg name="tf_prefix" default="None" />
+  <xacro:property name="tf_prefix" value="$(arg tf_prefix)" />
+  <xacro:if value="${tf_prefix == 'None'}">
+    <xacro:property name="tf_prefix_ext" value="" />
+  </xacro:if>
+  <xacro:unless value="${ tf_prefix == 'None'}">
+    <xacro:property name="tf_prefix_ext" value="${tf_prefix}_" />
+  </xacro:unless>
   <xacro:include filename="$(find rosbot_xl_description)/urdf/rosbot_xl_macro.urdf.xacro"
     ns="husarion" />
-  <xacro:husarion.rosbot_xl_robot use_sim="$(arg use_sim)" mecanum="$(arg mecanum)"
+  <xacro:husarion.rosbot_xl_robot
+    use_sim="$(arg use_sim)"
+    mecanum="$(arg mecanum)"
     simulation_engine="$(arg simulation_engine)"
-    simulation_controllers_config_file="$(arg simulation_controllers_config_file)" />
+    simulation_controllers_config_file="$(arg simulation_controllers_config_file)"
+    tf_prefix="$(arg tf_prefix)" />
   <xacro:include filename="$(find rosbot_xl_description)/urdf/components/antenna.urdf.xacro"
     ns="antenna" />
   <xacro:antenna.antenna
-    parent_link="body_link"
+    parent_link="${tf_prefix_ext}body_link"
     xyz="-0.155 -0.055 0.065"
     rpy="0.0 0.0 0.0"
-    antenna_angle="0.0" />
+    antenna_angle="0.0"
+    tf_prefix="$(arg tf_prefix)" />
   <!-- INCLUDE LIDAR -->
   <xacro:property name="lidar_model" value="$(arg lidar_model)" />
-  <xacro:property name="lidar_parent_link" value="cover_link" />
+  <xacro:property name="lidar_parent_link" value="${tf_prefix_ext}cover_link" />
   <xacro:property name="lidar_xyz" value="0.02 0.0 0.0" />
   <xacro:property name="lidar_rpy" value="0.0 0.0 0.0" />
@@ -37,5 +49,6 @@
       rpy="${lidar_rpy}"
       use_gpu="${lidar_use_gpu}"
-      simulation_engine="$(arg simulation_engine)" />
+      simulation_engine="$(arg simulation_engine)"
+      tf_prefix="$(arg tf_prefix)" />
   </xacro:if>
   <xacro:if value="${lidar_model == 'slamtec_rplidar_a2'}">
@@ -47,5 +60,6 @@
       rpy="${lidar_rpy}"
       use_gpu="${lidar_use_gpu}"
-      simulation_engine="$(arg simulation_engine)" />
+      simulation_engine="$(arg simulation_engine)"
+      tf_prefix="$(arg tf_prefix)" />
   </xacro:if>
   <xacro:if value="${lidar_model == 'slamtec_rplidar_a3'}">
@@ -57,5 +71,6 @@
       rpy="${lidar_rpy}"
       use_gpu="${lidar_use_gpu}"
-      simulation_engine="$(arg simulation_engine)" />
+      simulation_engine="$(arg simulation_engine)"
+      tf_prefix="$(arg tf_prefix)" />
   </xacro:if>
   <xacro:if value="${lidar_model == 'velodyne_puck'}">
@@ -68,9 +83,10 @@
       use_gpu="${lidar_use_gpu}"
       simulation_engine="$(arg simulation_engine)"
-      topic="velodyne_points" />
+      topic="velodyne_points"
+      tf_prefix="$(arg tf_prefix)" />
   </xacro:if>
   <!-- INCLUDE CAMERA -->
   <xacro:property name="camera_model" value="$(arg camera_model)" />
-  <xacro:property name="camera_parent_link" value="camera_mount_link" />
+  <xacro:property name="camera_parent_link" value="${tf_prefix_ext}camera_mount_link" />
   <xacro:property name="camera_xyz" value="0.0 0.0 0.0" />
   <xacro:property name="camera_rpy" value="0.0 0.0 0.0" />
@@ -128,9 +144,10 @@
       ns="camera_mount" />
     <xacro:camera_mount.camera_mount
-      parent_link="cover_link"
+      parent_link="${tf_prefix_ext}cover_link"
       xyz="-0.1 0.0 0.0"
       rpy="0.0 0.0 0.0"
       camera_mount_angle_1="0.0"
-      camera_mount_angle_2="0.0" />
+      camera_mount_angle_2="0.0"
+      tf_prefix="$(arg tf_prefix)" />
   </xacro:if>
 </robot>

File: rosbot_xl_description/urdf/rosbot_xl_macro.urdf.xacro (robot description, xacro)
@@ -2,5 +2,5 @@
 <robot xmlns:xacro="http://wiki.ros.org/xacro">
   <xacro:macro name="rosbot_xl_robot"
-    params="use_sim mecanum simulation_engine simulation_controllers_config_file">
+    params="use_sim mecanum simulation_engine simulation_controllers_config_file tf_prefix">
     <xacro:if value="${mecanum}">
       <xacro:property name="wheel_radius" value="0.05" />
@@ -9,18 +9,24 @@
       <xacro:property name="wheel_radius" value="0.048" />
     </xacro:unless>
+    <xacro:if value="${tf_prefix == 'None'}">
+      <xacro:property name="tf_prefix_ext" value="" />
+    </xacro:if>
+    <xacro:unless value="${tf_prefix == 'None'}">
+      <xacro:property name="tf_prefix_ext" value="${tf_prefix}_" />
+    </xacro:unless>
     <!-- INCLUDE ROBOT PARTS DEFINITIONS -->
     <xacro:include filename="$(find rosbot_xl_description)/urdf/body.urdf.xacro" ns="body" />
     <xacro:include filename="$(find rosbot_xl_description)/urdf/wheel.urdf.xacro" ns="wheel" />
     <!-- BODY DECLARATION -->
-    <xacro:body.body wheel_radius="${wheel_radius}" />
+    <xacro:body.body wheel_radius="${wheel_radius}" tf_prefix="${tf_prefix}" />
     <!-- WHEEL DECLARATION -->
-    <xacro:wheel.wheel wheel_radius="${wheel_radius}" prefix="fl" mecanum="${mecanum}"
-      use_sim="$(arg use_sim)" />
-    <xacro:wheel.wheel wheel_radius="${wheel_radius}" prefix="fr" mecanum="${mecanum}"
-      use_sim="$(arg use_sim)" />
-    <xacro:wheel.wheel wheel_radius="${wheel_radius}" prefix="rl" mecanum="${mecanum}"
-      use_sim="$(arg use_sim)" />
-    <xacro:wheel.wheel wheel_radius="${wheel_radius}" prefix="rr" mecanum="${mecanum}"
-      use_sim="$(arg use_sim)" />
+    <xacro:wheel.wheel wheel_radius="${wheel_radius}" side="fl" mecanum="${mecanum}"
+      use_sim="$(arg use_sim)" tf_prefix="${tf_prefix}" />
+    <xacro:wheel.wheel wheel_radius="${wheel_radius}" side="fr" mecanum="${mecanum}"
+      use_sim="$(arg use_sim)" tf_prefix="${tf_prefix}" />
+    <xacro:wheel.wheel wheel_radius="${wheel_radius}" side="rl" mecanum="${mecanum}"
+      use_sim="$(arg use_sim)" tf_prefix="${tf_prefix}" />
+    <xacro:wheel.wheel wheel_radius="${wheel_radius}" side="rr" mecanum="${mecanum}"
+      use_sim="$(arg use_sim)" tf_prefix="${tf_prefix}" />
     <!-- ROS2 CONTROL -->
     <xacro:unless value="$(arg use_sim)">
@@ -59,4 +65,6 @@
           <param name="connection_timeout_ms">120000</param>
           <param name="connection_check_period_ms">500</param>
+          <!-- Firmware from https://github.com/husarion/rosbot_xl_firmware could not override this names -->
+          <!-- The tf_prefix parameter adds correct tf_prefix -->
           <!-- order of velocity commands to be published in motors_cmd Float32MultiArray msg -->
           <param name="velocity_command_joint_order">
@@ -68,20 +76,20 @@
         </xacro:unless>
       </hardware>
-      <joint name="fl_wheel_joint">
+      <joint name="${tf_prefix_ext}fl_wheel_joint">
         <command_interface name="velocity" />
         <state_interface name="position" />
         <state_interface name="velocity" />
       </joint>
-      <joint name="fr_wheel_joint">
+      <joint name="${tf_prefix_ext}fr_wheel_joint">
         <command_interface name="velocity" />
         <state_interface name="position" />
         <state_interface name="velocity" />
       </joint>
-      <joint name="rl_wheel_joint">
+      <joint name="${tf_prefix_ext}rl_wheel_joint">
         <command_interface name="velocity" />
         <state_interface name="position" />
         <state_interface name="velocity" />
       </joint>
-      <joint name="rr_wheel_joint">
+      <joint name="${tf_prefix_ext}rr_wheel_joint">
         <command_interface name="velocity" />
         <state_interface name="position" />
@@ -117,5 +125,5 @@
           </plugin>
         </gazebo>
-        <gazebo reference="imu_link">
+        <gazebo reference="${tf_prefix_ext}imu_link">
           <sensor name="imu" type="imu">
             <plugin filename="ignition-gazebo-imu-system" name="ignition::gazebo::systems::Imu"></plugin>
@@ -125,6 +133,6 @@
             <visualize>false</visualize>
             <enable_metrics>false</enable_metrics>
-            <frame_id>imu_link</frame_id>
-            <ignition_frame_id>imu_link</ignition_frame_id>
+            <frame_id>${tf_prefix_ext}imu_link</frame_id>
+            <ignition_frame_id>${tf_prefix_ext}imu_link</ignition_frame_id>
           </sensor>
         </gazebo>

File: rosbot_xl_description/urdf/wheel.urdf.xacro (robot description, xacro)
@@ -1,5 +1,5 @@
 <?xml version="1.0" encoding="utf-8"?>
 <robot xmlns:xacro="http://www.ros.org/wiki/xacro">
-  <xacro:macro name="wheel" params="wheel_radius prefix mecanum use_sim">
+  <xacro:macro name="wheel" params="wheel_radius side tf_prefix mecanum use_sim">
     <xacro:property name="wheel_separation_x" value="0.170" />
     <xacro:if value="${mecanum}">
@@ -12,4 +12,10 @@
       <xacro:property name="wheel_separation_y" value="0.270" />
     </xacro:if>
+    <xacro:if value="${tf_prefix == 'None'}">
+      <xacro:property name="tf_prefix_ext" value="" />
+    </xacro:if>
+    <xacro:unless value="${ tf_prefix == 'None'}">
+      <xacro:property name="tf_prefix_ext" value="${tf_prefix}_" />
+    </xacro:unless>
     <xacro:unless value="${mecanum}">
       <xacro:property name="wheel_file" value="wheel" />
@@ -21,5 +27,5 @@
       <xacro:property name="wheel_separation_y" value="0.248" />
     </xacro:unless>
-    <xacro:if value="${prefix == 'fl'}">
+    <xacro:if value="${side == 'fl'}">
       <xacro:property name="x" value="${wheel_separation_x/2}" />
       <xacro:property name="y" value="${wheel_separation_y/2}" />
@@ -28,5 +34,5 @@
       <xacro:property name="fdir" value="1 -1 0" />
     </xacro:if>
-    <xacro:if value="${prefix == 'fr'}">
+    <xacro:if value="${side == 'fr'}">
       <xacro:property name="x" value="${wheel_separation_x/2}" />
       <xacro:property name="y" value="${-wheel_separation_y/2}" />
@@ -35,5 +41,5 @@
       <xacro:property name="fdir" value="1 1 0" />
     </xacro:if>
-    <xacro:if value="${prefix == 'rl'}">
+    <xacro:if value="${side == 'rl'}">
       <xacro:property name="x" value="${-wheel_separation_x/2}" />
       <xacro:property name="y" value="${wheel_separation_y/2}" />
@@ -42,5 +48,5 @@
       <xacro:property name="fdir" value="1 1 0" />
     </xacro:if>
-    <xacro:if value="${prefix == 'rr'}">
+    <xacro:if value="${side == 'rr'}">
       <xacro:property name="x" value="${-wheel_separation_x/2}" />
       <xacro:property name="y" value="${-wheel_separation_y/2}" />
@@ -49,7 +55,7 @@
       <xacro:property name="fdir" value="1 -1 0" />
     </xacro:if>
-    <joint name="${prefix}_wheel_joint" type="continuous">
-      <parent link="body_link" />
-      <child link="${prefix}_wheel_link" />
+    <joint name="${tf_prefix_ext}${side}_wheel_joint" type="continuous">
+      <parent link="${tf_prefix_ext}body_link" />
+      <child link="${tf_prefix_ext}${side}_wheel_link" />
       <origin xyz="${x} ${y} 0.0" rpy="0.0 0.0 0.0" />
       <axis xyz="0.0 1.0 0.0" />
@@ -57,5 +63,5 @@
       <dynamics damping="0.001" friction="0.001" />
     </joint>
-    <link name="${prefix}_wheel_link">
+    <link name="${tf_prefix_ext}${side}_wheel_link">
       <visual>
         <geometry>
@@ -78,5 +84,5 @@
     </link>
     <xacro:if value="${use_sim}">
-      <gazebo reference="${prefix}_wheel_link" xmlns:ignition="http://ignitionrobotics.org/schema">
+      <gazebo reference="${tf_prefix_ext}${side}_wheel_link" xmlns:ignition="http://ignitionrobotics.org/schema">
         <collision>
           <surface>
@@ -85,5 +91,5 @@
                 <mu>1.0</mu>
                 <mu2>0.0</mu2>
-                <fdir1 ignition:expressed_in="base_link">${fdir}</fdir1>
+                <fdir1 ignition:expressed_in="${tf_prefix_ext}base_link">${fdir}</fdir1>
               </ode>
             </friction>
