Commit message: added fixed namespaces to description and controller
Signed-off-by: Jakub Delicat <jakub.delicat@husarion.com>

File: rosbot_xl_description/urdf/body.urdf.xacro (robot description, xacro)
@@ -1,18 +1,12 @@
 <?xml version="1.0" encoding="utf-8"?>
 <robot xmlns:xacro="http://www.ros.org/wiki/xacro">
-  <xacro:macro name="body" params="wheel_radius tf_prefix">
-    <xacro:if value="${tf_prefix == 'None'}">
-      <xacro:property name="tf_prefix_ext" value="" />
-    </xacro:if>
-    <xacro:unless value="${tf_prefix == 'None'}">
-      <xacro:property name="tf_prefix_ext" value="${tf_prefix}_" />
-    </xacro:unless>
-    <link name="${tf_prefix_ext}base_link" />
-    <joint name="${tf_prefix_ext}base_to_${tf_prefix_ext}body_joint" type="fixed">
+  <xacro:macro name="body" params="wheel_radius">
+    <link name="base_link" />
+    <joint name="base_to_body_joint" type="fixed">
       <origin xyz="0.0 0.0 ${wheel_radius}" rpy="0.0 0.0 0.0" />
-      <parent link="${tf_prefix_ext}base_link" />
-      <child link="${tf_prefix_ext}body_link" />
+      <parent link="base_link" />
+      <child link="body_link" />
     </joint>
-    <link name="${tf_prefix_ext}body_link">
+    <link name="body_link">
       <visual>
         <geometry>
@@ -35,16 +29,16 @@
       </inertial>
     </link>
-    <joint name="${tf_prefix_ext}body_to_${tf_prefix_ext}cover_joint" type="fixed">
+    <joint name="body_to_cover_joint" type="fixed">
       <origin xyz="0.0 0.0 0.08345" rpy="0.0 0.0 0.0" />
-      <parent link="${tf_prefix_ext}body_link" />
-      <child link="${tf_prefix_ext}cover_link" />
+      <parent link="body_link" />
+      <child link="cover_link" />
     </joint>
-    <link name="${tf_prefix_ext}cover_link" />
-    <joint name="${tf_prefix_ext}body_to_${tf_prefix_ext}imu_joint" type="fixed">
+    <link name="cover_link" />
+    <joint name="body_to_imu_joint" type="fixed">
       <origin xyz="-0.1369 -0.0419 0.0370" rpy="3.14159 0.0 0.0" />
-      <parent link="${tf_prefix_ext}body_link" />
-      <child link="${tf_prefix_ext}imu_link" />
+      <parent link="body_link" />
+      <child link="imu_link" />
     </joint>
-    <link name="${tf_prefix_ext}imu_link" />
+    <link name="imu_link" />
   </xacro:macro>
 </robot>

File: rosbot_xl_description/urdf/rosbot_xl.urdf.xacro (robot description, xacro)
@@ -7,14 +7,5 @@
   <xacro:arg name="use_sim" default="false" />
   <xacro:arg name="simulation_engine" default="ignition-gazebo" />
-  <xacro:arg name="simulation_controllers_config_file"
-    default="$(find rosbot_xl_controller)/config/diff_drive_controller.yaml" />
-  <xacro:arg name="tf_prefix" default="None" />
-  <xacro:property name="tf_prefix" value="$(arg tf_prefix)" />
-  <xacro:if value="${tf_prefix == 'None'}">
-    <xacro:property name="tf_prefix_ext" value="" />
-  </xacro:if>
-  <xacro:unless value="${ tf_prefix == 'None'}">
-    <xacro:property name="tf_prefix_ext" value="${tf_prefix}_" />
-  </xacro:unless>
+  <xacro:arg name="namespace" default="None" />
   <xacro:include filename="$(find rosbot_xl_description)/urdf/rosbot_xl_macro.urdf.xacro"
     ns="husarion" />
@@ -23,17 +14,15 @@
     mecanum="$(arg mecanum)"
     simulation_engine="$(arg simulation_engine)"
-    simulation_controllers_config_file="$(arg simulation_controllers_config_file)"
-    tf_prefix="$(arg tf_prefix)" />
+    namespace="$(arg namespace)" />
   <xacro:include filename="$(find rosbot_xl_description)/urdf/components/antenna.urdf.xacro"
     ns="antenna" />
   <xacro:antenna.antenna
-    parent_link="${tf_prefix_ext}body_link"
+    parent_link="body_link"
     xyz="-0.155 -0.055 0.065"
     rpy="0.0 0.0 0.0"
-    antenna_angle="0.0"
-    tf_prefix="$(arg tf_prefix)" />
+    antenna_angle="0.0" />
   <!-- INCLUDE LIDAR -->
   <xacro:property name="lidar_model" value="$(arg lidar_model)" />
-  <xacro:property name="lidar_parent_link" value="${tf_prefix_ext}cover_link" />
+  <xacro:property name="lidar_parent_link" value="cover_link" />
   <xacro:property name="lidar_xyz" value="0.02 0.0 0.0" />
   <xacro:property name="lidar_rpy" value="0.0 0.0 0.0" />
@@ -50,5 +39,5 @@
       use_gpu="${lidar_use_gpu}"
       simulation_engine="$(arg simulation_engine)"
-      tf_prefix="$(arg tf_prefix)" />
+      namespace="$(arg namespace)" />
   </xacro:if>
   <xacro:if value="${lidar_model == 'slamtec_rplidar_s2'}">
@@ -60,5 +49,6 @@
       rpy="${lidar_rpy}"
       use_gpu="${lidar_use_gpu}"
-      simulation_engine="$(arg simulation_engine)" />
+      simulation_engine="$(arg simulation_engine)"
+      namespace="$(arg namespace)" />
   </xacro:if>
   <xacro:if value="${lidar_model == 'slamtec_rplidar_s3'}">
@@ -70,5 +60,6 @@
       rpy="${lidar_rpy}"
       use_gpu="${lidar_use_gpu}"
-      simulation_engine="$(arg simulation_engine)" />
+      simulation_engine="$(arg simulation_engine)"
+      namespace="$(arg namespace)" />
   </xacro:if>
   <xacro:if value="${lidar_model == 'slamtec_rplidar_a2'}">
@@ -81,5 +72,5 @@
       use_gpu="${lidar_use_gpu}"
       simulation_engine="$(arg simulation_engine)"
-      tf_prefix="$(arg tf_prefix)" />
+      namespace="$(arg namespace)" />
   </xacro:if>
   <xacro:if value="${lidar_model == 'slamtec_rplidar_a3'}">
@@ -92,5 +83,5 @@
       use_gpu="${lidar_use_gpu}"
       simulation_engine="$(arg simulation_engine)"
-      tf_prefix="$(arg tf_prefix)" />
+      namespace="$(arg namespace)" />
   </xacro:if>
   <xacro:if value="${lidar_model == 'velodyne_puck'}">
@@ -103,10 +94,9 @@
       use_gpu="${lidar_use_gpu}"
       simulation_engine="$(arg simulation_engine)"
-      topic="velodyne_points"
-      tf_prefix="$(arg tf_prefix)" />
+      topic="velodyne_points"/>
   </xacro:if>
   <!-- INCLUDE CAMERA -->
   <xacro:property name="camera_model" value="$(arg camera_model)" />
-  <xacro:property name="camera_parent_link" value="${tf_prefix_ext}camera_mount_link" />
+  <xacro:property name="camera_parent_link" value="camera_mount_link" />
   <xacro:property name="camera_xyz" value="0.0 0.0 0.0" />
   <xacro:property name="camera_rpy" value="0.0 0.0 0.0" />
@@ -169,10 +159,9 @@
       ns="camera_mount" />
     <xacro:camera_mount.camera_mount
-      parent_link="${tf_prefix_ext}cover_link"
+      parent_link="cover_link"
       xyz="-0.1 0.0 0.0"
       rpy="0.0 0.0 0.0"
       camera_mount_angle_1="0.0"
-      camera_mount_angle_2="0.0"
-      tf_prefix="$(arg tf_prefix)" />
+      camera_mount_angle_2="0.0" />
   </xacro:if>
 </robot>

File: rosbot_xl_description/urdf/rosbot_xl_macro.urdf.xacro (robot description, xacro)
@@ -2,5 +2,13 @@
 <robot xmlns:xacro="http://wiki.ros.org/xacro">
   <xacro:macro name="rosbot_xl_robot"
-    params="use_sim mecanum simulation_engine simulation_controllers_config_file tf_prefix">
+    params="use_sim mecanum simulation_engine namespace">
+    <xacro:if value="${namespace == 'None'}">
+      <xacro:property name="namespace_ext" value="" />
+      <xacro:property name="gz_control_namespace" value="/" />
+    </xacro:if>
+    <xacro:unless value="${namespace == 'None'}">
+        <xacro:property name="namespace_ext" value="${namespace}/" />
+        <xacro:property name="gz_control_namespace" value="${namespace}" />
+    </xacro:unless>
     <xacro:if value="${mecanum}">
       <xacro:property name="wheel_radius" value="0.05" />
@@ -9,27 +17,21 @@
       <xacro:property name="wheel_radius" value="0.048" />
     </xacro:unless>
-    <xacro:if value="${tf_prefix == 'None'}">
-      <xacro:property name="tf_prefix_ext" value="" />
-    </xacro:if>
-    <xacro:unless value="${tf_prefix == 'None'}">
-      <xacro:property name="tf_prefix_ext" value="${tf_prefix}_" />
-    </xacro:unless>
     <!-- INCLUDE ROBOT PARTS DEFINITIONS -->
     <xacro:include filename="$(find rosbot_xl_description)/urdf/body.urdf.xacro" ns="body" />
     <xacro:include filename="$(find rosbot_xl_description)/urdf/wheel.urdf.xacro" ns="wheel" />
     <!-- BODY DECLARATION -->
-    <xacro:body.body wheel_radius="${wheel_radius}" tf_prefix="${tf_prefix}" />
+    <xacro:body.body wheel_radius="${wheel_radius}" />
     <!-- WHEEL DECLARATION -->
     <xacro:wheel.wheel wheel_radius="${wheel_radius}" side="fl" mecanum="${mecanum}"
-      use_sim="$(arg use_sim)" tf_prefix="${tf_prefix}" />
+      use_sim="$(arg use_sim)" />
     <xacro:wheel.wheel wheel_radius="${wheel_radius}" side="fr" mecanum="${mecanum}"
-      use_sim="$(arg use_sim)" tf_prefix="${tf_prefix}" />
+      use_sim="$(arg use_sim)" />
     <xacro:wheel.wheel wheel_radius="${wheel_radius}" side="rl" mecanum="${mecanum}"
-      use_sim="$(arg use_sim)" tf_prefix="${tf_prefix}" />
+      use_sim="$(arg use_sim)" />
     <xacro:wheel.wheel wheel_radius="${wheel_radius}" side="rr" mecanum="${mecanum}"
-      use_sim="$(arg use_sim)" tf_prefix="${tf_prefix}" />
+      use_sim="$(arg use_sim)" />
     <!-- ROS2 CONTROL -->
     <xacro:unless value="$(arg use_sim)">
-      <ros2_control name="imu" type="sensor">
+      <ros2_control name="${namespace_ext}imu" type="sensor">
         <hardware>
           <plugin>rosbot_hardware_interfaces/RosbotImuSensor</plugin>
@@ -37,5 +39,5 @@
           <param name="connection_check_period_ms">500</param>
         </hardware>
-        <sensor name="imu">
+        <sensor name="${namespace_ext}imu">
           <state_interface name="orientation.x" />
           <state_interface name="orientation.y" />
@@ -51,5 +53,5 @@
       </ros2_control>
     </xacro:unless>
-    <ros2_control name="wheels" type="system">
+    <ros2_control name="${namespace_ext}wheels" type="system">
       <hardware>
         <xacro:if value="${use_sim}">
@@ -65,6 +67,4 @@
           <param name="connection_timeout_ms">120000</param>
           <param name="connection_check_period_ms">500</param>
-          <!-- Firmware from https://github.com/husarion/rosbot_xl_firmware could not override this names -->
-          <!-- The tf_prefix parameter adds correct tf_prefix -->
           <!-- order of velocity commands to be published in motors_cmd Float32MultiArray msg -->
           <param name="velocity_command_joint_order">
@@ -74,23 +74,22 @@
             fl_wheel_joint
           </param>
-          <param name="tf_prefix">${tf_prefix_ext}</param>
         </xacro:unless>
       </hardware>
-      <joint name="${tf_prefix_ext}fl_wheel_joint">
+      <joint name="fl_wheel_joint">
         <command_interface name="velocity" />
         <state_interface name="position" />
         <state_interface name="velocity" />
       </joint>
-      <joint name="${tf_prefix_ext}fr_wheel_joint">
+      <joint name="fr_wheel_joint">
         <command_interface name="velocity" />
         <state_interface name="position" />
         <state_interface name="velocity" />
       </joint>
-      <joint name="${tf_prefix_ext}rl_wheel_joint">
+      <joint name="rl_wheel_joint">
         <command_interface name="velocity" />
         <state_interface name="position" />
         <state_interface name="velocity" />
       </joint>
-      <joint name="${tf_prefix_ext}rr_wheel_joint">
+      <joint name="rr_wheel_joint">
         <command_interface name="velocity" />
         <state_interface name="position" />
@@ -119,21 +118,29 @@
           <plugin filename="ign_ros2_control-system"
             name="ign_ros2_control::IgnitionROS2ControlPlugin">
-            <parameters>${simulation_controllers_config_file}</parameters>
-            <controller_manager_prefix_node_name>simulation</controller_manager_prefix_node_name>
+            <xacro:if value="${mecanum}">
+              <parameters>$(find rosbot_xl_controller)/config/mecanum_drive_controller.yaml</parameters>
+            </xacro:if>
+            <xacro:unless value="${mecanum}">
+              <parameters>$(find rosbot_xl_controller)/config/diff_drive_controller.yaml</parameters>
+            </xacro:unless>
             <ros>
-              <remapping>/rosbot_xl_base_controller/cmd_vel_unstamped:=/cmd_vel</remapping>
+              <namespace>${gz_control_namespace}</namespace>
+              <remapping>rosbot_xl_base_controller/cmd_vel_unstamped:=cmd_vel</remapping>
+              <remapping>/tf:=tf</remapping>
             </ros>
           </plugin>
         </gazebo>
-        <gazebo reference="${tf_prefix_ext}imu_link">
-          <sensor name="imu" type="imu">
-            <plugin filename="ignition-gazebo-imu-system" name="ignition::gazebo::systems::Imu"></plugin>
+        <gazebo reference="imu_link">
+          <sensor name="${namespace_ext}imu" type="imu">
             <always_on>true</always_on>
             <update_rate>25</update_rate>
-            <topic>imu/data_raw</topic>
+            <topic>${namespace_ext}imu/data_raw</topic>
             <visualize>false</visualize>
             <enable_metrics>false</enable_metrics>
-            <frame_id>${tf_prefix_ext}imu_link</frame_id>
-            <ignition_frame_id>${tf_prefix_ext}imu_link</ignition_frame_id>
+            <frame_id>imu_link</frame_id>
+            <ignition_frame_id>imu_link</ignition_frame_id>
+            <ros>
+              <namespace>${namespace_ext}</namespace>
+            </ros>
           </sensor>
         </gazebo>

File: rosbot_xl_description/urdf/wheel.urdf.xacro (robot description, xacro)
@@ -1,5 +1,5 @@
 <?xml version="1.0" encoding="utf-8"?>
 <robot xmlns:xacro="http://www.ros.org/wiki/xacro">
-  <xacro:macro name="wheel" params="wheel_radius side tf_prefix mecanum use_sim">
+  <xacro:macro name="wheel" params="wheel_radius side mecanum use_sim">
     <xacro:property name="wheel_separation_x" value="0.170" />
     <xacro:if value="${mecanum}">
@@ -12,10 +12,4 @@
       <xacro:property name="wheel_separation_y" value="0.270" />
     </xacro:if>
-    <xacro:if value="${tf_prefix == 'None'}">
-      <xacro:property name="tf_prefix_ext" value="" />
-    </xacro:if>
-    <xacro:unless value="${ tf_prefix == 'None'}">
-      <xacro:property name="tf_prefix_ext" value="${tf_prefix}_" />
-    </xacro:unless>
     <xacro:unless value="${mecanum}">
       <xacro:property name="wheel_file" value="wheel" />
@@ -55,7 +49,7 @@
       <xacro:property name="fdir" value="1 -1 0" />
     </xacro:if>
-    <joint name="${tf_prefix_ext}${side}_wheel_joint" type="continuous">
-      <parent link="${tf_prefix_ext}body_link" />
-      <child link="${tf_prefix_ext}${side}_wheel_link" />
+    <joint name="${side}_wheel_joint" type="continuous">
+      <parent link="body_link" />
+      <child link="${side}_wheel_link" />
       <origin xyz="${x} ${y} 0.0" rpy="0.0 0.0 0.0" />
       <axis xyz="0.0 1.0 0.0" />
@@ -63,5 +57,5 @@
       <dynamics damping="0.001" friction="0.001" />
     </joint>
-    <link name="${tf_prefix_ext}${side}_wheel_link">
+    <link name="${side}_wheel_link">
       <visual>
         <geometry>
@@ -84,5 +78,5 @@
     </link>
     <xacro:if value="${use_sim}">
-      <gazebo reference="${tf_prefix_ext}${side}_wheel_link" xmlns:ignition="http://ignitionrobotics.org/schema">
+      <gazebo reference="${side}_wheel_link" xmlns:ignition="http://ignitionrobotics.org/schema">
         <collision>
           <surface>
@@ -91,5 +85,5 @@
                 <mu>1.0</mu>
                 <mu2>0.0</mu2>
-                <fdir1 ignition:expressed_in="${tf_prefix_ext}base_link">${fdir}</fdir1>
+                <fdir1 ignition:expressed_in="base_link">${fdir}</fdir1>
               </ode>
             </friction>
