Commit message: Remove wheel type parameter

File: rosbot_xl_description/urdf/rosbot_xl_macro.urdf.xacro (robot description, xacro)
@@ -10,8 +10,8 @@
     <xacro:body.body wheel_radius="${wheel_radius}" />
     <!-- WHEEL DECLARATION -->
-    <xacro:wheel.wheel wheel_type="differential" wheel_radius="${wheel_radius}" wheel_separation_y="${wheel_separation_y}" prefix="front_left" />
-    <xacro:wheel.wheel wheel_type="differential" wheel_radius="${wheel_radius}" wheel_separation_y="${wheel_separation_y}" prefix="front_right" />
-    <xacro:wheel.wheel wheel_type="differential" wheel_radius="${wheel_radius}" wheel_separation_y="${wheel_separation_y}" prefix="rear_left" />
-    <xacro:wheel.wheel wheel_type="differential" wheel_radius="${wheel_radius}" wheel_separation_y="${wheel_separation_y}" prefix="rear_right" />
+    <xacro:wheel.wheel wheel_radius="${wheel_radius}" wheel_separation_y="${wheel_separation_y}" prefix="front_left" />
+    <xacro:wheel.wheel wheel_radius="${wheel_radius}" wheel_separation_y="${wheel_separation_y}" prefix="front_right" />
+    <xacro:wheel.wheel wheel_radius="${wheel_radius}" wheel_separation_y="${wheel_separation_y}" prefix="rear_left" />
+    <xacro:wheel.wheel wheel_radius="${wheel_radius}" wheel_separation_y="${wheel_separation_y}" prefix="rear_right" />
     <!-- ROS2 CONTROL -->
     <xacro:include filename="$(find rosbot_hardware_interfaces)/urdf/ros2_control.urdf.xacro" />

File: rosbot_xl_description/urdf/wheel.urdf.xacro (robot description, xacro)
@@ -2,5 +2,5 @@
 <robot xmlns:xacro="http://www.ros.org/wiki/xacro">
   <!-- wheel defining macro -->
-  <xacro:macro name="wheel" params="wheel_type wheel_radius wheel_separation_y prefix">
+  <xacro:macro name="wheel" params="wheel_radius wheel_separation_y prefix">
     <xacro:property name="wheel_separation_x" value="0.170" />
     <xacro:property name="wheel_thickness" value="0.032" />

Commit message: Rename wheel joints

File: rosbot_xl_description/urdf/rosbot_xl_macro.urdf.xacro (robot description, xacro)
@@ -10,8 +10,8 @@
     <xacro:body.body wheel_radius="${wheel_radius}" />
     <!-- WHEEL DECLARATION -->
-    <xacro:wheel.wheel wheel_radius="${wheel_radius}" wheel_separation_y="${wheel_separation_y}" prefix="front_left" />
-    <xacro:wheel.wheel wheel_radius="${wheel_radius}" wheel_separation_y="${wheel_separation_y}" prefix="front_right" />
-    <xacro:wheel.wheel wheel_radius="${wheel_radius}" wheel_separation_y="${wheel_separation_y}" prefix="rear_left" />
-    <xacro:wheel.wheel wheel_radius="${wheel_radius}" wheel_separation_y="${wheel_separation_y}" prefix="rear_right" />
+    <xacro:wheel.wheel wheel_radius="${wheel_radius}" wheel_separation_y="${wheel_separation_y}" prefix="fl" />
+    <xacro:wheel.wheel wheel_radius="${wheel_radius}" wheel_separation_y="${wheel_separation_y}" prefix="fr" />
+    <xacro:wheel.wheel wheel_radius="${wheel_radius}" wheel_separation_y="${wheel_separation_y}" prefix="rl" />
+    <xacro:wheel.wheel wheel_radius="${wheel_radius}" wheel_separation_y="${wheel_separation_y}" prefix="rr" />
     <!-- ROS2 CONTROL -->
     <xacro:include filename="$(find rosbot_hardware_interfaces)/urdf/ros2_control.urdf.xacro" />
@@ -24,8 +24,8 @@
           <update_rate>10</update_rate>
           <num_wheel_pairs>2</num_wheel_pairs>
-          <left_joint>front_left_wheel_joint</left_joint>
-          <right_joint>front_right_wheel_joint</right_joint>
-          <left_joint>rear_left_wheel_joint</left_joint>
-          <right_joint>rear_right_wheel_joint</right_joint>
+          <left_joint>fl_wheel_joint</left_joint>
+          <right_joint>fr_wheel_joint</right_joint>
+          <left_joint>rl_wheel_joint</left_joint>
+          <right_joint>rr_wheel_joint</right_joint>
           <wheel_separation>${wheel_separation_y}</wheel_separation>
           <wheel_separation>${wheel_separation_y}</wheel_separation>
@@ -44,8 +44,8 @@
       <gazebo>
         <plugin name="joint_states" filename="libgazebo_ros_joint_state_publisher.so">
-          <joint_name>front_left_wheel_joint</joint_name>
-          <joint_name>front_right_wheel_joint</joint_name>
-          <joint_name>rear_left_wheel_joint</joint_name>
-          <joint_name>rear_right_wheel_joint</joint_name>
+          <joint_name>fl_wheel_joint</joint_name>
+          <joint_name>fr_wheel_joint</joint_name>
+          <joint_name>rl_wheel_joint</joint_name>
+          <joint_name>rr_wheel_joint</joint_name>
         </plugin>
       </gazebo>
@@ -125,8 +125,8 @@
           <update_rate>10</update_rate>
           <always_on>true</always_on>
-          <left_joint>front_left_wheel_joint</left_joint>
-          <right_joint>front_right_wheel_joint</right_joint>
-          <left_joint>rear_left_wheel_joint</left_joint>
-          <right_joint>rear_right_wheel_joint</right_joint>
+          <left_joint>fl_wheel_joint</left_joint>
+          <right_joint>fr_wheel_joint</right_joint>
+          <left_joint>rl_wheel_joint</left_joint>
+          <right_joint>rr_wheel_joint</right_joint>
           <wheel_separation>${wheel_separation_y}</wheel_separation>
           <wheel_separation>${wheel_separation_y}</wheel_separation>
@@ -158,8 +158,8 @@
       <gazebo>
         <plugin filename="libignition-gazebo-joint-state-publisher-system.so" name="ignition::gazebo::systems::JointStatePublisher">
-          <joint name="front_left_wheel_joint"></joint>
-          <joint name="front_right_wheel_joint"></joint>
-          <joint name="rear_left_wheel_joint"></joint>
-          <joint name="rear_right_wheel_joint"></joint>
+          <joint name="fl_wheel_joint"></joint>
+          <joint name="fr_wheel_joint"></joint>
+          <joint name="rl_wheel_joint"></joint>
+          <joint name="rr_wheel_joint"></joint>
         </plugin>
       </gazebo>

File: rosbot_xl_description/urdf/wheel.urdf.xacro (robot description, xacro)
@@ -5,20 +5,20 @@
     <xacro:property name="wheel_separation_x" value="0.170" />
     <xacro:property name="wheel_thickness" value="0.032" />
-    <xacro:if value="${prefix == 'front_left'}">
+    <xacro:if value="${prefix == 'fl'}">
       <xacro:property name="x" value="${wheel_separation_x/2}" />
       <xacro:property name="y" value="${wheel_separation_y/2}" />
       <xacro:property name="mesh" value="file://$(find rosbot_xl_description)/meshes/wheel_a.dae" />
     </xacro:if>
-    <xacro:if value="${prefix == 'front_right'}">
+    <xacro:if value="${prefix == 'fr'}">
       <xacro:property name="x" value="${wheel_separation_x/2}" />
       <xacro:property name="y" value="-${wheel_separation_y/2}" />
       <xacro:property name="mesh" value="file://$(find rosbot_xl_description)/meshes/wheel_b.dae" />
     </xacro:if>
-    <xacro:if value="${prefix == 'rear_left'}">
+    <xacro:if value="${prefix == 'rl'}">
       <xacro:property name="x" value="-${wheel_separation_x/2}" />
       <xacro:property name="y" value="${wheel_separation_y/2}" />
       <xacro:property name="mesh" value="file://$(find rosbot_xl_description)/meshes/wheel_a.dae" />
     </xacro:if>
-    <xacro:if value="${prefix == 'rear_right'}">
+    <xacro:if value="${prefix == 'rr'}">
       <xacro:property name="x" value="-${wheel_separation_x/2}" />
       <xacro:property name="y" value="-${wheel_separation_y/2}" />

Commit message: Define ros2 control directly in urdf instead of including macro

File: rosbot_xl_description/urdf/rosbot_xl_macro.urdf.xacro (robot description, xacro)
@@ -15,6 +15,50 @@
     <xacro:wheel.wheel wheel_radius="${wheel_radius}" wheel_separation_y="${wheel_separation_y}" prefix="rr" />
     <!-- ROS2 CONTROL -->
-    <xacro:include filename="$(find rosbot_hardware_interfaces)/urdf/ros2_control.urdf.xacro" />
-    <xacro:ros2_control_system />
+    <ros2_control name="imu" type="sensor">
+      <hardware>
+        <plugin>rosbot_hardware_interfaces/RosbotImuSensor</plugin>
+        <param name="connection_timeout_ms">120000</param>
+        <param name="connection_check_period_ms">500</param>
+      </hardware>
+      <sensor name="imu">
+        <state_interface name="orientation.x" />
+        <state_interface name="orientation.y" />
+        <state_interface name="orientation.z" />
+        <state_interface name="orientation.w" />
+        <state_interface name="angular_velocity.x" />
+        <state_interface name="angular_velocity.y" />
+        <state_interface name="angular_velocity.z" />
+        <state_interface name="linear_acceleration.x" />
+        <state_interface name="linear_acceleration.y" />
+        <state_interface name="linear_acceleration.z" />
+      </sensor>
+    </ros2_control>
+    <ros2_control name="wheels" type="system">
+      <hardware>
+        <plugin>rosbot_hardware_interfaces/RosbotSystem</plugin>
+        <param name="connection_timeout_ms">120000</param>
+        <param name="connection_check_period_ms">500</param>
+      </hardware>
+      <joint name="fl_wheel_joint">
+        <command_interface name="velocity" />
+        <state_interface name="position" />
+        <state_interface name="velocity" />
+      </joint>
+      <joint name="fr_wheel_joint">
+        <command_interface name="velocity" />
+        <state_interface name="position" />
+        <state_interface name="velocity" />
+      </joint>
+      <joint name="rl_wheel_joint">
+        <command_interface name="velocity" />
+        <state_interface name="position" />
+        <state_interface name="velocity" />
+      </joint>
+      <joint name="rr_wheel_joint">
+        <command_interface name="velocity" />
+        <state_interface name="position" />
+        <state_interface name="velocity" />
+      </joint>
+    </ros2_control>
     <!-- SIMULATION GAZEBO -->
     <xacro:if value="${use_sim and simulation_engine == 'gazebo-classic'}">

Commit message: Move RosbotSystem parameters to urdf

File: rosbot_xl_description/urdf/rosbot_xl_macro.urdf.xacro (robot description, xacro)
@@ -2,5 +2,5 @@
 <robot xmlns:xacro="http://wiki.ros.org/xacro">
   <xacro:macro name="rosbot_xl_robot" params="use_sim use_gpu simulation_engine">
-    <xacro:property name="wheel_radius" value="0.041" />
+    <xacro:property name="wheel_radius" value="0.048" />
     <xacro:property name="wheel_separation_y" value="0.236" />
     <!-- INCLUDE ROBOT PARTS DEFINITIONS -->
@@ -39,4 +39,15 @@
         <param name="connection_timeout_ms">120000</param>
         <param name="connection_check_period_ms">500</param>
+        <!-- for some reason diff drive controller publishes velocities for motors in rad/s, but expects feedback in m/s
+          both commands and feedback from digital board are in rad/s, so it is necessary to convert it
+          maybe will be resolved (https://github.com/ros-controls/ros2_controllers/issues/411), then it can be removed -->
+        <param name="wheel_radius">${wheel_radius}</param>
+        <!-- order of velocity commands to be published in motors_cmd Float32MultiArray msg -->
+        <param name="velocity_command_joint_order">
+              rr_wheel_joint,
+              rl_wheel_joint,
+              fr_wheel_joint,
+              fl_wheel_joint
+        </param>
       </hardware>
       <joint name="fl_wheel_joint">

Commit message: added tests from rosbot_ros | fixed imu
Signed-off-by: Jakub Delicat <jakub.delicat@husarion.com>

File: rosbot_xl_description/urdf/rosbot_xl_macro.urdf.xacro (robot description, xacro)
@@ -4,9 +4,9 @@
     params="use_sim mecanum simulation_engine namespace">
     <xacro:if value="${namespace == 'None'}">
-      <xacro:property name="namespace_ext" value="" />
+      <xacro:property name="ns" value="" />
       <xacro:property name="gz_control_namespace" value="/" />
     </xacro:if>
     <xacro:unless value="${namespace == 'None'}">
-        <xacro:property name="namespace_ext" value="${namespace}/" />
+        <xacro:property name="ns" value="${namespace}/" />
         <xacro:property name="gz_control_namespace" value="${namespace}" />
     </xacro:unless>
@@ -33,5 +33,5 @@
     <!-- ROS2 CONTROL -->
     <xacro:unless value="$(arg use_sim)">
-      <ros2_control name="${namespace_ext}imu" type="sensor">
+      <ros2_control name="${ns}imu" type="sensor">
         <hardware>
           <plugin>rosbot_hardware_interfaces/RosbotImuSensor</plugin>
@@ -39,5 +39,5 @@
           <param name="connection_check_period_ms">500</param>
         </hardware>
-        <sensor name="${namespace_ext}imu">
+        <sensor name="${ns}imu">
           <state_interface name="orientation.x" />
           <state_interface name="orientation.y" />
@@ -53,5 +53,5 @@
       </ros2_control>
     </xacro:unless>
-    <ros2_control name="${namespace_ext}wheels" type="system">
+    <ros2_control name="${ns}wheels" type="system">
       <hardware>
         <xacro:if value="${use_sim}">
@@ -98,5 +98,5 @@
       <xacro:if value="${use_sim}">
         <xacro:if value="${simulation_engine == 'ignition-gazebo'}">
-          <sensor name="imu">
+          <sensor name="${ns}imu">
             <state_interface name="orientation.x" />
             <state_interface name="orientation.y" />
@@ -131,8 +131,8 @@
         </gazebo>
         <gazebo reference="imu_link">
-          <sensor name="${namespace_ext}imu" type="imu">
+          <sensor name="${ns}imu" type="imu">
             <always_on>true</always_on>
             <update_rate>25</update_rate>
-            <topic>${namespace_ext}imu/data_raw</topic>
+            <topic>${ns}imu/data_raw</topic>
             <visualize>false</visualize>
             <enable_metrics>false</enable_metrics>
@@ -140,5 +140,5 @@
             <ignition_frame_id>imu_link</ignition_frame_id>
             <ros>
-              <namespace>${namespace_ext}</namespace>
+              <namespace>${ns}</namespace>
             </ros>
           </sensor>
