Commit message: Merge description

File: rosbot_xl_description/urdf/rosbot.urdf.xacro (robot description, xacro)
@@ -4,5 +4,5 @@
   <xacro:arg name="mecanum" default="false" />
   <xacro:arg name="namespace" default="None" />
-  <xacro:include filename="$(find rosbot_description)/rosbot/urdf/rosbot_macro.urdf.xacro" ns="husarion" />
+  <xacro:include filename="$(find rosbot_xl_description)/urdf/rosbot/rosbot_macro.urdf.xacro" ns="husarion" />
   <xacro:husarion.rosbot
     mecanum="$(arg mecanum)"

File: rosbot_xl_description/urdf/rosbot/body.urdf.xacro (robot description, xacro)
@@ -3,5 +3,5 @@
   <!-- body defining macro -->
   <xacro:macro name="body" params="wheel_radius mecanum namespace">
-    <xacro:include filename="$(find rosbot_description)/urdf/components/vl53lox.urdf.xacro" ns="range_sensor" />
+    <xacro:include filename="$(find rosbot_xl_description)/urdf/rosbot/components/vl53lox.urdf.xacro" ns="range_sensor" />
     <link name="base_link" />
     <joint name="base_to_body_joint" type="fixed">
@@ -13,9 +13,9 @@
       <visual>
         <geometry>
-          <mesh filename="package://rosbot_description/meshes/rosbot/body.stl" scale="0.001 0.001 0.001" />
+          <mesh filename="package://rosbot_xl_description/meshes/rosbot/body.stl" scale="0.001 0.001 0.001" />
         </geometry>
         <origin xyz="0.0 0.0 -0.0173" rpy="${pi/2} 0.0 ${pi/2}" />
         <material name="Black">
-          <color rgba="0.1 0.1 0.1 0.1" />
+          <color rgba="0.1 0.1 0.1 1.0" />
         </material>
       </visual>
@@ -45,5 +45,5 @@
       <visual>
         <geometry>
-          <mesh filename="package://rosbot_description/meshes/rosbot/cover.stl" scale="0.001 0.001 0.001" />
+          <mesh filename="package://rosbot_xl_description/meshes/rosbot/cover.stl" scale="0.001 0.001 0.001" />
         </geometry>
         <origin xyz="0.0 0.0 -0.002" rpy="${pi/2} 0.0 ${pi/2}" />

File: rosbot_xl_description/urdf/rosbot/rosbot_macro.urdf.xacro (robot description, xacro)
@@ -1,10 +1,10 @@
 <?xml version='1.0'?>
 <robot xmlns:xacro="http://wiki.ros.org/xacro">
-  <xacro:macro name="rosbot" params="mecanum use_sim namespace">
+  <xacro:macro name="rosbot" params="mecanum namespace use_sim">
     <xacro:property name="ns" value="${namespace + '/' if namespace != 'None' else ''}" />
     <xacro:property name="wheel_radius" value="${0.0470 if mecanum else 0.0425}" />
     <!-- INCLUDE ROBOT PARTS DEFINITIONS -->
-    <xacro:include filename="$(find rosbot_description)/urdf/body.urdf.xacro" ns="body" />
-    <xacro:include filename="$(find rosbot_description)/urdf/wheel.urdf.xacro" ns="wheel" />
+    <xacro:include filename="$(find rosbot_xl_description)/urdf/rosbot/body.urdf.xacro" ns="body" />
+    <xacro:include filename="$(find rosbot_xl_description)/urdf/rosbot/wheel.urdf.xacro" ns="wheel" />
     <!-- BODY DECLARATION -->
     <xacro:body.body wheel_radius="${wheel_radius}" mecanum="${mecanum}" namespace="${namespace}" />

File: rosbot_xl_description/urdf/rosbot/wheel.urdf.xacro (robot description, xacro)
@@ -25,5 +25,5 @@
       <xacro:property name="x" value="${wheel_separation_x/2.0}" />
       <xacro:property name="y" value="${wheel_separation_y/2.0}" />
-      <xacro:property name="mesh" value="package://rosbot_description/meshes/rosbot/${wheel_file}_b.dae" />
+      <xacro:property name="mesh" value="package://rosbot_xl_description/meshes/rosbot/${wheel_file}_b.dae" />
       <xacro:property name="visual_rotation" value="${pi}" />
       <xacro:property name="fdir" value="1.0 -1.0 0.0" />
@@ -32,5 +32,5 @@
       <xacro:property name="x" value="${wheel_separation_x/2.0}" />
       <xacro:property name="y" value="${-wheel_separation_y/2.0}" />
-      <xacro:property name="mesh" value="package://rosbot_description/meshes/rosbot/${wheel_file}_a.dae" />
+      <xacro:property name="mesh" value="package://rosbot_xl_description/meshes/rosbot/${wheel_file}_a.dae" />
       <xacro:property name="visual_rotation" value="${pi}" />
       <xacro:property name="fdir" value="1.0 1.0 0.0" />
@@ -39,5 +39,5 @@
       <xacro:property name="x" value="${-wheel_separation_x/2.0}" />
       <xacro:property name="y" value="${wheel_separation_y/2.0}" />
-      <xacro:property name="mesh" value="package://rosbot_description/meshes/rosbot/${wheel_file}_a.dae" />
+      <xacro:property name="mesh" value="package://rosbot_xl_description/meshes/rosbot/${wheel_file}_a.dae" />
       <xacro:property name="visual_rotation" value="${0.0}" />
       <xacro:property name="fdir" value="1.0 1.0 0.0" />
@@ -46,5 +46,5 @@
       <xacro:property name="x" value="${-wheel_separation_x/2.0}" />
       <xacro:property name="y" value="${-wheel_separation_y/2.0}" />
-      <xacro:property name="mesh" value="package://rosbot_description/meshes/rosbot/${wheel_file}_b.dae" />
+      <xacro:property name="mesh" value="package://rosbot_xl_description/meshes/rosbot/${wheel_file}_b.dae" />
       <xacro:property name="visual_rotation" value="${0.0}" />
       <xacro:property name="fdir" value="1.0 -1.0 0.0" />

Commit message: Use push namespace

File: rosbot_xl_description/urdf/rosbot.urdf.xacro (robot description, xacro)
@@ -5,16 +5,16 @@
   <xacro:arg name="namespace" default="None" />
   <xacro:include filename="$(find rosbot_xl_description)/urdf/rosbot/rosbot_macro.urdf.xacro" ns="husarion" />
+  <xacro:include filename="$(find ros_components_description)/urdf/slamtec_rplidar.urdf.xacro" ns="lidar" />
+	<xacro:include filename="$(find depthai_descriptions)/urdf/include/depthai_macro.urdf.xacro" ns="camera" />
   <xacro:husarion.rosbot
     mecanum="$(arg mecanum)"
     use_sim="$(arg use_sim)"
     namespace="$(arg namespace)" />
-    <xacro:include filename="$(find ros_components_description)/urdf/slamtec_rplidar.urdf.xacro" ns="lidar" />
-    <xacro:lidar.slamtec_rplidar
-      parent_link="cover_link"
-      xyz="0.02 0.0 0.0"
-      rpy="0.0 0.0 0.0"
-      model="s2"
-      namespace="$(arg namespace)" />
-	<xacro:include filename="$(find depthai_descriptions)/urdf/include/depthai_macro.urdf.xacro" ns="camera" />
+  <xacro:lidar.slamtec_rplidar
+    parent_link="cover_link"
+    xyz="0.02 0.0 0.0"
+    rpy="0.0 0.0 0.0"
+    model="s2"
+    namespace="$(arg namespace)" />
 	<xacro:camera.depthai_camera camera_name="oak_camera" parent="camera_mount_link"
 		camera_model="OAK-D-PRO" base_frame="oak_camera"

File: rosbot_xl_description/urdf/rosbot_xl.urdf.xacro (robot description, xacro)
@@ -1,8 +1,9 @@
 <?xml version='1.0'?>
 <robot name="rosbot_xl" xmlns:xacro="http://www.ros.org/wiki/xacro">
+  <xacro:arg name="components_config_path" default="$(find husarion_ugv_description)/config/components.yaml" />
+  <xacro:arg name="controller_config_file" default="$(find rosbot_xl_controller)/config/diff_drive_controller.yaml" />
   <xacro:arg name="mecanum" default="false" />
+  <xacro:arg name="namespace" default="" />
   <xacro:arg name="use_sim" default="false" />
-  <xacro:arg name="namespace" default="None" />
-  <xacro:arg name="controller_config_file" default="$(find rosbot_xl_controller)/config/diff_drive_controller.yaml" />
   <xacro:include filename="$(find rosbot_xl_description)/urdf/rosbot_xl/rosbot_xl_macro.urdf.xacro"
     ns="husarion" />
@@ -12,14 +13,4 @@
     namespace="$(arg namespace)"
     use_sim="$(arg use_sim)" />
-  <xacro:include filename="$(find rosbot_xl_description)/urdf/rosbot_xl/components/antenna.urdf.xacro"
-    ns="antenna" />
-  <xacro:antenna.antenna
-    parent_link="body_link"
-    xyz="-0.155 -0.055 0.065"
-    rpy="0.0 0.0 0.0"
-    antenna_angle="0.0" />
-  <xacro:property name="camera_parent_link" value="camera_mount_link" />
-  <xacro:property name="camera_xyz" value="0.0 0.0 0.0" />
-  <xacro:property name="camera_rpy" value="0.0 0.0 0.0" />
   <xacro:property name="include_camera_mount" value="$(arg include_camera_mount)" />
   <!-- TODO <xacro:if value="${include_camera_mount or camera_model != 'None'}"> -->
@@ -33,3 +24,12 @@
       camera_mount_angle_2="0.0" />
   <!-- </xacro:if> -->
+  <xacro:property name="components_config_path_property" value="$(arg components_config_path)" />
+  <xacro:unless value="${components_config_path_property == 'None'}">
+    <xacro:include filename="$(find ros_components_description)/urdf/components.urdf.xacro"
+      ns="husarion_components" />
+    <xacro:husarion_components.create_components
+      components_config_path="${components_config_path_property}"
+      namespace="$(arg namespace)"
+    />
+  </xacro:unless>
 </robot>

File: rosbot_xl_description/urdf/rosbot_xl/rosbot_xl_macro.urdf.xacro (robot description, xacro)
@@ -20,10 +20,12 @@
     <!-- INCLUDE ROBOT PARTS DEFINITIONS -->
     <xacro:include filename="$(find rosbot_xl_description)/urdf/rosbot_xl/body.urdf.xacro" ns="body" />
+    <xacro:include filename="$(find rosbot_xl_description)/urdf/rosbot_xl/components/antenna.urdf.xacro" ns="antenna" />
     <xacro:include filename="$(find rosbot_xl_description)/urdf/rosbot_xl/gazebo.urdf.xacro" ns="gazebo" />
     <xacro:include filename="$(find rosbot_xl_description)/urdf/rosbot_xl/webots.urdf.xacro" ns="webots" />
     <xacro:include filename="$(find rosbot_xl_description)/urdf/rosbot_xl/wheel.urdf.xacro" ns="wheel" />
-/rosbot_xl
     <!-- BODY DECLARATION -->
     <xacro:body.body wheel_radius="${wheel_radius}" />
+    <!-- ANTENNA DECLARATION -->
+    <xacro:antenna.antenna parent_link="body_link" xyz="-0.155 -0.055 0.065" rpy="0.0 0.0 0.0" antenna_angle="0.0" />
     <!-- WHEEL DECLARATION -->
     <xacro:wheel.wheel wheel_radius="${wheel_radius}" side="fl" mecanum="${mecanum}" />
