Commit message: Fix lidar position and material

File: rosbot_xl_description/urdf/rosbot_xl.urdf.xacro (robot description, xacro)
@@ -6,8 +6,11 @@
   <xacro:include filename="$(find rosbot_xl_description)/urdf/rosbot_xl_macro.urdf.xacro" ns="husarion" />
   <xacro:husarion.rosbot_xl_robot use_sim="$(arg use_sim)" use_gpu="$(arg use_gpu)" simulation_engine="$(arg simulation_engine)" />
+  <material name="DarkGrey">
+    <color rgba="0.05 0.05 0.05 1.0"/>
+  </material>
   <xacro:include filename="$(find ros_components_description)/urdf/rplidar_s1.gazebo.xacro" ns="lidar" />
   <xacro:lidar.rplidar_s1
     parent_link="cover_link"
-    xyz="0.0 0.0 0.08345"
+    xyz="0.0 0.0 0.0"
     rpy="0.0 0.0 ${pi}"
     use_gpu="$(arg use_gpu)"

Commit message: [WIP] Fix ros2 control gz

File: rosbot_xl_description/urdf/rosbot_xl.urdf.xacro (robot description, xacro)
@@ -7,5 +7,5 @@
   <xacro:husarion.rosbot_xl_robot use_sim="$(arg use_sim)" use_gpu="$(arg use_gpu)" simulation_engine="$(arg simulation_engine)" />
   <!-- material used in rplidar -->
-  <material name="DarkGrey">
+  <!-- <material name="DarkGrey">
     <color rgba="0.05 0.05 0.05 1.0"/>
   </material>
@@ -16,4 +16,4 @@
     rpy="0.0 0.0 ${pi}"
     use_gpu="$(arg use_gpu)"
-    simulation_engine="$(arg simulation_engine)" />
+    simulation_engine="$(arg simulation_engine)" /> -->
 </robot>

File: rosbot_xl_description/urdf/rosbot_xl_macro.urdf.xacro (robot description, xacro)
@@ -15,39 +15,49 @@
     <xacro:wheel.wheel wheel_radius="${wheel_radius}" wheel_separation_y="${wheel_separation_y}" prefix="rr" />
     <!-- ROS2 CONTROL -->
-    <ros2_control name="imu" type="sensor">
-      <hardware>
-        <plugin>rosbot_hardware_interfaces/RosbotImuSensor</plugin>
-        <param name="connection_timeout_ms">120000</param>
-        <param name="connection_check_period_ms">500</param>
-      </hardware>
-      <sensor name="imu">
-        <state_interface name="orientation.x" />
-        <state_interface name="orientation.y" />
-        <state_interface name="orientation.z" />
-        <state_interface name="orientation.w" />
-        <state_interface name="angular_velocity.x" />
-        <state_interface name="angular_velocity.y" />
-        <state_interface name="angular_velocity.z" />
-        <state_interface name="linear_acceleration.x" />
-        <state_interface name="linear_acceleration.y" />
-        <state_interface name="linear_acceleration.z" />
-      </sensor>
-    </ros2_control>
+    <xacro:unless value="$(arg use_sim)">
+      <ros2_control name="imu" type="sensor">
+        <hardware>
+          <plugin>rosbot_hardware_interfaces/RosbotImuSensor</plugin>
+          <param name="connection_timeout_ms">120000</param>
+          <param name="connection_check_period_ms">500</param>
+        </hardware>
+        <sensor name="imu">
+          <state_interface name="orientation.x" />
+          <state_interface name="orientation.y" />
+          <state_interface name="orientation.z" />
+          <state_interface name="orientation.w" />
+          <state_interface name="angular_velocity.x" />
+          <state_interface name="angular_velocity.y" />
+          <state_interface name="angular_velocity.z" />
+          <state_interface name="linear_acceleration.x" />
+          <state_interface name="linear_acceleration.y" />
+          <state_interface name="linear_acceleration.z" />
+        </sensor>
+      </ros2_control>
+    </xacro:unless>
     <ros2_control name="wheels" type="system">
       <hardware>
-        <plugin>rosbot_hardware_interfaces/RosbotSystem</plugin>
-        <param name="connection_timeout_ms">120000</param>
-        <param name="connection_check_period_ms">500</param>
-        <!-- for some reason diff drive controller publishes velocities for motors in rad/s, but expects feedback in m/s
-          both commands and feedback from digital board are in rad/s, so it is necessary to convert it
-          maybe will be resolved (https://github.com/ros-controls/ros2_controllers/issues/411), then it can be removed -->
-        <param name="wheel_radius">${wheel_radius}</param>
-        <!-- order of velocity commands to be published in motors_cmd Float32MultiArray msg -->
-        <param name="velocity_command_joint_order">
-              rr_wheel_joint,
-              rl_wheel_joint,
-              fr_wheel_joint,
-              fl_wheel_joint
-        </param>
+        <xacro:if value="${use_sim and simulation_engine == 'gazebo-classic'}">
+          <plugin>gazebo_ros2_control/GazeboSystem</plugin>
+        </xacro:if>
+        <xacro:if value="${use_sim and simulation_engine == 'ignition'}">
+          <plugin>ign_ros2_control/IgnitionSystem</plugin>
+        </xacro:if>
+        <xacro:unless value="$(arg use_sim)">
+          <plugin>rosbot_hardware_interfaces/RosbotSystem</plugin>
+          <param name="connection_timeout_ms">120000</param>
+          <param name="connection_check_period_ms">500</param>
+          <!-- for some reason diff drive controller publishes velocities for motors in rad/s, but expects feedback in m/s
+            both commands and feedback from digital board are in rad/s, so it is necessary to convert it
+            maybe will be resolved (https://github.com/ros-controls/ros2_controllers/issues/411), then it can be removed -->
+          <param name="wheel_radius">${wheel_radius}</param>
+          <!-- order of velocity commands to be published in motors_cmd Float32MultiArray msg -->
+          <param name="velocity_command_joint_order">
+                rr_wheel_joint,
+                rl_wheel_joint,
+                fr_wheel_joint,
+                fl_wheel_joint
+          </param>
+        </xacro:unless>
       </hardware>
       <joint name="fl_wheel_joint">
@@ -72,155 +82,24 @@
       </joint>
     </ros2_control>
-    <!-- SIMULATION GAZEBO -->
-    <xacro:if value="${use_sim and simulation_engine == 'gazebo-classic'}">
+    <!-- SIMULATION IGNITION -->
+    <xacro:if value="${use_sim and simulation_engine == 'ignition'}">
       <gazebo>
-        <plugin name='skid_steer_drive' filename='libgazebo_ros_diff_drive.so'>
-          <ros></ros>
-          <update_rate>10</update_rate>
-          <num_wheel_pairs>2</num_wheel_pairs>
-          <left_joint>fl_wheel_joint</left_joint>
-          <right_joint>fr_wheel_joint</right_joint>
-          <left_joint>rl_wheel_joint</left_joint>
-          <right_joint>rr_wheel_joint</right_joint>
-          <wheel_separation>${wheel_separation_y}</wheel_separation>
-          <wheel_separation>${wheel_separation_y}</wheel_separation>
-          <wheel_diameter>${wheel_radius*2.0}</wheel_diameter>
-          <wheel_diameter>${wheel_radius*2.0}</wheel_diameter>
-          <max_wheel_torque>1.2</max_wheel_torque>
-          <max_wheel_acceleration>0.5</max_wheel_acceleration>
-          <publish_odom>true</publish_odom>
-          <publish_odom_tf>true</publish_odom_tf>
-          <publish_wheel_tf>true</publish_wheel_tf>
-          <odometry_frame>odom</odometry_frame>
-          <robot_base_frame>base_link</robot_base_frame>
+        <plugin filename="ign_ros2_control-system" name="ign_ros2_control::IgnitionROS2ControlPlugin">
+          <parameters>$(find rosbot_xl_hardware)/config/diff_drive_controller.yaml</parameters>
         </plugin>
       </gazebo>
-      <!-- publish joint states -->
-      <gazebo>
-        <plugin name="joint_states" filename="libgazebo_ros_joint_state_publisher.so">
-          <joint_name>fl_wheel_joint</joint_name>
-          <joint_name>fr_wheel_joint</joint_name>
-          <joint_name>rl_wheel_joint</joint_name>
-          <joint_name>rr_wheel_joint</joint_name>
-        </plugin>
-      </gazebo>
-      <!-- <gazebo>
-        <plugin filename="libgazebo_ros2_control.so" name="gazebo_ros2_control">
-          <robot_param>robot_description</robot_param>
-          <robot_param_node>robot_state_publisher</robot_param_node>
-          <parameters>$(find rosbot_xl_description)/config/controllers_gazebo.yaml</parameters>
-        </plugin>
-      </gazebo> -->
     </xacro:if>
-    <!-- SIMULATION IGNITION -->
-    <xacro:if value="${use_sim and simulation_engine == 'ignition'}">
-      <!-- publish IMU -->
-      <gazebo reference="imu_link">
-        <sensor name="imu_link" type="imu">
-          <plugin filename="ignition-gazebo-imu-system" name="ignition::gazebo::systems::Imu"></plugin>
-          <always_on>true</always_on>
-          <update_rate>25</update_rate>
-          <topic>imu/data_raw</topic>
-          <visualize>false</visualize>
-          <enable_metrics>false</enable_metrics>
-          <frame_id>imu_link</frame_id>
-          <ignition_frame_id>imu_link</ignition_frame_id>
-          <pose relative_to='imu_link'>0 0 0 0 0 0</pose>
-          <imu>
-            <angular_velocity>
-              <x>
-                <noise type="gaussian">
-                  <mean>0.0</mean>
-                  <stddev>1</stddev>
-                </noise>
-              </x>
-              <y>
-                <noise type="gaussian">
-                  <mean>1.0</mean>
-                  <stddev>1</stddev>
-                </noise>
-              </y>
-              <z>
-                <noise type="gaussian">
-                  <mean>0.0</mean>
-                  <stddev>1</stddev>
-                </noise>
-              </z>
-            </angular_velocity>
-            <linear_acceleration>
-              <x>
-                <noise type="gaussian">
-                  <mean>0.0</mean>
-                  <stddev>0.1</stddev>
-                </noise>
-              </x>
-              <y>
-                <noise type="gaussian">
-                  <mean>0.0</mean>
-                  <stddev>0.1</stddev>
-                </noise>
-              </y>
-              <z>
-                <noise type="gaussian">
-                  <mean>0.0</mean>
-                  <stddev>0.1</stddev>
-                </noise>
-              </z>
-            </linear_acceleration>
-          </imu>
-        </sensor>
-      </gazebo>
-      <!-- <gazebo>
-      <plugin filename="ign_ros2_control-system" name="ign_ros2_control::IgnitionROS2ControlPlugin">
-        <parameters>$(find rosbot_xl_gazebo)/config/controllers.yaml</parameters>
-      </plugin>
-    </gazebo> -->
-      <gazebo>
-        <plugin filename="libignition-gazebo-diff-drive-system.so" name="ignition::gazebo::systems::DiffDrive">
-          <update_rate>10</update_rate>
-          <always_on>true</always_on>
-          <left_joint>fl_wheel_joint</left_joint>
-          <right_joint>fr_wheel_joint</right_joint>
-          <left_joint>rl_wheel_joint</left_joint>
-          <right_joint>rr_wheel_joint</right_joint>
-          <wheel_separation>${wheel_separation_y}</wheel_separation>
-          <wheel_separation>${wheel_separation_y}</wheel_separation>
-          <wheel_radius>${wheel_radius}</wheel_radius>
-          <wheel_radius>${wheel_radius}</wheel_radius>
-          <odom_publish_frequency>25</odom_publish_frequency>
-          <topic>cmd_vel</topic>
-          <odom_topic>odom/wheels</odom_topic>
-          <tf_topic>tf</tf_topic>
-          <frame_id>odom</frame_id>
-          <child_frame_id>base_link</child_frame_id>
-        </plugin>
-      </gazebo>
-      <gazebo>
-        <plugin filename="libignition-gazebo-pose-publisher-system.so" name="ignition::gazebo::systems::PosePublisher">
-          <publish_link_pose>true</publish_link_pose>
-          <publish_collision_pose>false</publish_collision_pose>
-          <publish_visual_pose>false</publish_visual_pose>
-          <publish_nested_model_pose>false</publish_nested_model_pose>
-          <use_pose_vector_msg>true</use_pose_vector_msg>
-          <update_frequency>50</update_frequency>
-        </plugin>
-      </gazebo>
-      <gazebo>
-        <plugin filename="libignition-gazebo-sensors-system.so" name="ignition::gazebo::systems::Sensors">
-          <render_engine>ogre2</render_engine>
-        </plugin>
-      </gazebo>
-      <gazebo>
-        <plugin filename="libignition-gazebo-joint-state-publisher-system.so" name="ignition::gazebo::systems::JointStatePublisher">
-          <joint name="fl_wheel_joint"></joint>
-          <joint name="fr_wheel_joint"></joint>
-          <joint name="rl_wheel_joint"></joint>
-          <joint name="rr_wheel_joint"></joint>
-        </plugin>
-      </gazebo>
-      <gazebo>
-        <plugin filename="ignition-gazebo-scene-broadcaster-system" name="ignition::gazebo::systems::SceneBroadcaster"></plugin>
-      </gazebo>
-    </xacro:if>
+    <gazebo reference="imu_link">
+      <sensor name="imu_link" type="imu">
+        <plugin filename="ignition-gazebo-imu-system" name="ignition::gazebo::systems::Imu"></plugin>
+        <always_on>true</always_on>
+        <update_rate>25</update_rate>
+        <topic>imu/data_raw</topic>
+        <visualize>false</visualize>
+        <enable_metrics>false</enable_metrics>
+        <frame_id>imu_link</frame_id>
+        <ignition_frame_id>imu_link</ignition_frame_id>
+      </sensor>
+    </gazebo>
   </xacro:macro>
 </robot>

Commit message: Reenable lidar and remove material

File: rosbot_xl_description/urdf/rosbot_xl.urdf.xacro (robot description, xacro)
@@ -7,7 +7,4 @@
   <xacro:husarion.rosbot_xl_robot use_sim="$(arg use_sim)" use_gpu="$(arg use_gpu)" simulation_engine="$(arg simulation_engine)" />
   <!-- material used in rplidar -->
-  <!-- <material name="DarkGrey">
-    <color rgba="0.05 0.05 0.05 1.0"/>
-  </material>
   <xacro:include filename="$(find ros_components_description)/urdf/rplidar_s1.gazebo.xacro" ns="lidar" />
   <xacro:lidar.rplidar_s1
@@ -16,4 +13,4 @@
     rpy="0.0 0.0 ${pi}"
     use_gpu="$(arg use_gpu)"
-    simulation_engine="$(arg simulation_engine)" /> -->
+    simulation_engine="$(arg simulation_engine)" />
 </robot>

Commit message: Remove simulation engine parameter (only ignition-gazebo will be supported)

File: rosbot_xl_description/urdf/rosbot_xl.urdf.xacro (robot description, xacro)
@@ -3,7 +3,6 @@
   <xacro:arg name="use_sim" default="false" />
   <xacro:arg name="use_gpu" default="false" />
-  <xacro:arg name="simulation_engine" default="gazebo-classic" />
   <xacro:include filename="$(find rosbot_xl_description)/urdf/rosbot_xl_macro.urdf.xacro" ns="husarion" />
-  <xacro:husarion.rosbot_xl_robot use_sim="$(arg use_sim)" use_gpu="$(arg use_gpu)" simulation_engine="$(arg simulation_engine)" />
+  <xacro:husarion.rosbot_xl_robot use_sim="$(arg use_sim)" use_gpu="$(arg use_gpu)" />
   <!-- material used in rplidar -->
   <xacro:include filename="$(find ros_components_description)/urdf/rplidar_s1.gazebo.xacro" ns="lidar" />
@@ -13,4 +12,4 @@
     rpy="0.0 0.0 ${pi}"
     use_gpu="$(arg use_gpu)"
-    simulation_engine="$(arg simulation_engine)" />
+    simulation_engine="ignition-gazebo" />
 </robot>

File: rosbot_xl_description/urdf/rosbot_xl_macro.urdf.xacro (robot description, xacro)
@@ -1,5 +1,5 @@
 <?xml version='1.0'?>
 <robot xmlns:xacro="http://wiki.ros.org/xacro">
-  <xacro:macro name="rosbot_xl_robot" params="use_sim use_gpu simulation_engine">
+  <xacro:macro name="rosbot_xl_robot" params="use_sim use_gpu">
     <xacro:property name="wheel_radius" value="0.048" />
     <xacro:property name="wheel_separation_y" value="0.236" />
@@ -38,8 +38,5 @@
     <ros2_control name="wheels" type="system">
       <hardware>
-        <xacro:if value="${use_sim and simulation_engine == 'gazebo-classic'}">
-          <plugin>gazebo_ros2_control/GazeboSystem</plugin>
-        </xacro:if>
-        <xacro:if value="${use_sim and simulation_engine == 'ignition-gazebo'}">
+        <xacro:if value="${use_sim}">
           <plugin>ign_ros2_control/IgnitionSystem</plugin>
         </xacro:if>
@@ -81,5 +78,5 @@
         <state_interface name="velocity" />
       </joint>
-      <xacro:if value="${use_sim and simulation_engine == 'ignition-gazebo'}">
+      <xacro:if value="${use_sim}">
         <sensor name="imu">
           <state_interface name="orientation.x" />
@@ -96,6 +93,5 @@
       </xacro:if>
     </ros2_control>
-    <!-- SIMULATION IGNITION GAZEBO -->
-    <xacro:if value="${use_sim and simulation_engine == 'ignition-gazebo'}">
+    <xacro:if value="${use_sim}">
       <gazebo>
         <plugin filename="ign_ros2_control-system" name="ign_ros2_control::IgnitionROS2ControlPlugin">
@@ -103,17 +99,17 @@
         </plugin>
       </gazebo>
+      <gazebo reference="imu_link">
+        <sensor name="imu" type="imu">
+          <plugin filename="ignition-gazebo-imu-system" name="ignition::gazebo::systems::Imu"></plugin>
+          <always_on>true</always_on>
+          <update_rate>25</update_rate>
+          <topic>imu/data_raw</topic>
+          <visualize>false</visualize>
+          <enable_metrics>false</enable_metrics>
+          <frame_id>imu_link</frame_id>
+          <ignition_frame_id>imu_link</ignition_frame_id>
+        </sensor>
+      </gazebo>
     </xacro:if>
-    <gazebo reference="imu_link">
-      <sensor name="imu" type="imu">
-        <plugin filename="ignition-gazebo-imu-system" name="ignition::gazebo::systems::Imu"></plugin>
-        <always_on>true</always_on>
-        <update_rate>25</update_rate>
-        <topic>imu/data_raw</topic>
-        <visualize>false</visualize>
-        <enable_metrics>false</enable_metrics>
-        <frame_id>imu_link</frame_id>
-        <ignition_frame_id>imu_link</ignition_frame_id>
-      </sensor>
-    </gazebo>
   </xacro:macro>
 </robot>

Commit message: Remove use gpu parameter

File: rosbot_xl_description/urdf/rosbot_xl.urdf.xacro (robot description, xacro)
@@ -2,8 +2,6 @@
 <robot name="rosbot_xl" xmlns:xacro="http://www.ros.org/wiki/xacro">
   <xacro:arg name="use_sim" default="false" />
-  <xacro:arg name="use_gpu" default="false" />
   <xacro:include filename="$(find rosbot_xl_description)/urdf/rosbot_xl_macro.urdf.xacro" ns="husarion" />
-  <xacro:husarion.rosbot_xl_robot use_sim="$(arg use_sim)" use_gpu="$(arg use_gpu)" />
-  <!-- material used in rplidar -->
+  <xacro:husarion.rosbot_xl_robot use_sim="$(arg use_sim)" />
   <xacro:include filename="$(find ros_components_description)/urdf/rplidar_s1.gazebo.xacro" ns="lidar" />
   <xacro:lidar.rplidar_s1
@@ -11,5 +9,6 @@
     xyz="0.0 0.0 0.0"
     rpy="0.0 0.0 ${pi}"
-    use_gpu="$(arg use_gpu)"
+    use_gpu="true"
     simulation_engine="ignition-gazebo" />
+  <!-- use_gpu has to be set to true, CPU lidar doesn't work in ignition - https://github.com/gazebosim/gz-sensors/issues/26 -->
 </robot>

File: rosbot_xl_description/urdf/rosbot_xl_macro.urdf.xacro (robot description, xacro)
@@ -1,5 +1,5 @@
 <?xml version='1.0'?>
 <robot xmlns:xacro="http://wiki.ros.org/xacro">
-  <xacro:macro name="rosbot_xl_robot" params="use_sim use_gpu">
+  <xacro:macro name="rosbot_xl_robot" params="use_sim">
     <xacro:property name="wheel_radius" value="0.048" />
     <xacro:property name="wheel_separation_y" value="0.236" />
