Commit message: [WIP] Add mecanum meshes

File: rosbot_xl_description/urdf/rosbot_xl.urdf.xacro (robot description, xacro)
@@ -2,6 +2,7 @@
 <robot name="rosbot_xl" xmlns:xacro="http://www.ros.org/wiki/xacro">
   <xacro:arg name="use_sim" default="false" />
+  <xacro:arg name="mecanum" default="false" />
   <xacro:include filename="$(find rosbot_xl_description)/urdf/rosbot_xl_macro.urdf.xacro" ns="husarion" />
-  <xacro:husarion.rosbot_xl_robot use_sim="$(arg use_sim)" />
+  <xacro:husarion.rosbot_xl_robot use_sim="$(arg use_sim)" mecanum="$(arg mecanum)" />
   <xacro:include filename="$(find ros_components_description)/urdf/rplidar_s1.gazebo.xacro" ns="lidar" />
   <xacro:lidar.rplidar_s1

File: rosbot_xl_description/urdf/rosbot_xl_macro.urdf.xacro (robot description, xacro)
@@ -1,7 +1,11 @@
 <?xml version='1.0'?>
 <robot xmlns:xacro="http://wiki.ros.org/xacro">
-  <xacro:macro name="rosbot_xl_robot" params="use_sim">
-    <xacro:property name="wheel_radius" value="0.048" />
-    <xacro:property name="wheel_separation_y" value="0.236" />
+  <xacro:macro name="rosbot_xl_robot" params="use_sim mecanum">
+    <xacro:if value="${mecanum}">
+      <xacro:property name="wheel_radius" value="0.05" />
+    </xacro:if>
+    <xacro:unless value="${mecanum}">
+      <xacro:property name="wheel_radius" value="0.048" />
+    </xacro:unless>
     <!-- INCLUDE ROBOT PARTS DEFINITIONS -->
     <xacro:include filename="$(find rosbot_xl_description)/urdf/body.urdf.xacro" ns="body" />
@@ -10,8 +14,8 @@
     <xacro:body.body wheel_radius="${wheel_radius}" />
     <!-- WHEEL DECLARATION -->
-    <xacro:wheel.wheel wheel_radius="${wheel_radius}" wheel_separation_y="${wheel_separation_y}" prefix="fl" />
-    <xacro:wheel.wheel wheel_radius="${wheel_radius}" wheel_separation_y="${wheel_separation_y}" prefix="fr" />
-    <xacro:wheel.wheel wheel_radius="${wheel_radius}" wheel_separation_y="${wheel_separation_y}" prefix="rl" />
-    <xacro:wheel.wheel wheel_radius="${wheel_radius}" wheel_separation_y="${wheel_separation_y}" prefix="rr" />
+    <xacro:wheel.wheel wheel_radius="${wheel_radius}" prefix="fl" mecanum="${mecanum}" />
+    <xacro:wheel.wheel wheel_radius="${wheel_radius}" prefix="fr" mecanum="${mecanum}" />
+    <xacro:wheel.wheel wheel_radius="${wheel_radius}" prefix="rl" mecanum="${mecanum}" />
+    <xacro:wheel.wheel wheel_radius="${wheel_radius}" prefix="rr" mecanum="${mecanum}" />
     <!-- ROS2 CONTROL -->
     <xacro:unless value="$(arg use_sim)">

File: rosbot_xl_description/urdf/wheel.urdf.xacro (robot description, xacro)
@@ -2,26 +2,51 @@
 <robot xmlns:xacro="http://www.ros.org/wiki/xacro">
   <!-- wheel defining macro -->
-  <xacro:macro name="wheel" params="wheel_radius wheel_separation_y prefix">
+  <xacro:macro name="wheel" params="wheel_radius prefix mecanum">
+    <xacro:property name="wheel_separation_y" value="0.236" />
     <xacro:property name="wheel_separation_x" value="0.170" />
-    <xacro:property name="wheel_thickness" value="0.032" />
+    <xacro:if value="${mecanum}">
+      <xacro:property name="wheel_file" value="mecanum" />
+      <xacro:property name="wheel_thickness" value="0.05" />
+      <xacro:property name="mass" value="0.4" />
+      <!-- TODO: change -->
+      <xacro:property name="ixx" value="3.954e-05" />
+      <xacro:property name="iyy" value="7.116e-05" />
+      <xacro:property name="izz" value="4.032e-05" />
+    </xacro:if>
+    <xacro:unless value="${mecanum}">
+      <xacro:property name="wheel_file" value="wheel" />
+      <xacro:property name="wheel_thickness" value="0.032" />
+      <xacro:property name="mass" value="0.051" />
+      <xacro:property name="ixx" value="3.954e-05" />
+      <xacro:property name="iyy" value="7.116e-05" />
+      <xacro:property name="izz" value="4.032e-05" />
+    </xacro:unless>
     <xacro:if value="${prefix == 'fl'}">
       <xacro:property name="x" value="${wheel_separation_x/2}" />
       <xacro:property name="y" value="${wheel_separation_y/2}" />
-      <xacro:property name="mesh" value="file://$(find rosbot_xl_description)/meshes/wheel_a.dae" />
+      <xacro:property name="mesh" value="file://$(find rosbot_xl_description)/meshes/${wheel_file}_a.dae" />
+      <xacro:property name="visual_rotation" value="0" />
+      <xacro:property name="visual_offset" value="-0.015" />
     </xacro:if>
     <xacro:if value="${prefix == 'fr'}">
       <xacro:property name="x" value="${wheel_separation_x/2}" />
-      <xacro:property name="y" value="-${wheel_separation_y/2}" />
-      <xacro:property name="mesh" value="file://$(find rosbot_xl_description)/meshes/wheel_b.dae" />
+      <xacro:property name="y" value="${-wheel_separation_y/2}" />
+      <xacro:property name="mesh" value="file://$(find rosbot_xl_description)/meshes/${wheel_file}_b.dae" />
+      <xacro:property name="visual_rotation" value="${pi}" />
+      <xacro:property name="visual_offset" value="0.015" />
     </xacro:if>
     <xacro:if value="${prefix == 'rl'}">
-      <xacro:property name="x" value="-${wheel_separation_x/2}" />
+      <xacro:property name="x" value="${-wheel_separation_x/2}" />
       <xacro:property name="y" value="${wheel_separation_y/2}" />
-      <xacro:property name="mesh" value="file://$(find rosbot_xl_description)/meshes/wheel_a.dae" />
+      <xacro:property name="mesh" value="file://$(find rosbot_xl_description)/meshes/${wheel_file}_a.dae" />
+      <xacro:property name="visual_rotation" value="0" />
+      <xacro:property name="visual_offset" value="-0.015" />
     </xacro:if>
     <xacro:if value="${prefix == 'rr'}">
-      <xacro:property name="x" value="-${wheel_separation_x/2}" />
-      <xacro:property name="y" value="-${wheel_separation_y/2}" />
-      <xacro:property name="mesh" value="file://$(find rosbot_xl_description)/meshes/wheel_b.dae" />
+      <xacro:property name="x" value="${-wheel_separation_x/2}" />
+      <xacro:property name="y" value="${-wheel_separation_y/2}" />
+      <xacro:property name="mesh" value="file://$(find rosbot_xl_description)/meshes/${wheel_file}_b.dae" />
+      <xacro:property name="visual_rotation" value="${pi}" />
+      <xacro:property name="visual_offset" value="0.015" />
     </xacro:if>
     <joint name="${prefix}_wheel_joint" type="continuous">
@@ -38,5 +63,5 @@
           <mesh filename="${mesh}" scale="1 1 1" />
         </geometry>
-        <origin xyz="0.0 0.0 0.0" rpy="0.0 0.0 0.0" />
+        <origin xyz="0.0 ${visual_offset} 0.0" rpy="0.0 0.0 ${visual_rotation}" />
       </visual>
       <collision>
@@ -47,8 +72,8 @@
       </collision>
       <inertial>
-        <mass value="0.051" />
-        <inertia  ixx="3.954e-05" ixy="0.000"     ixz="0.000"
-                                  iyy="7.116e-05" iyz="0.000"
-                                                  izz="4.032e-05" />
+        <mass value="${mass}" />
+        <inertia ixx="${ixx}" ixy="0.000"  ixz="0.000"
+                              iyy="${iyy}" iyz="0.000"
+                                           izz="${izz}" />
       </inertial>
     </link>

Commit message: added webots tag | added simulation-engine arg

File: rosbot_xl_description/urdf/rosbot_xl.urdf.xacro (robot description, xacro)
@@ -2,6 +2,7 @@
 <robot name="rosbot_xl" xmlns:xacro="http://www.ros.org/wiki/xacro">
   <xacro:arg name="use_sim" default="false" />
+  <xacro:arg name="simulation_engine" default="gazebo-ignition" />
   <xacro:include filename="$(find rosbot_xl_description)/urdf/rosbot_xl_macro.urdf.xacro" ns="husarion" />
-  <xacro:husarion.rosbot_xl_robot use_sim="$(arg use_sim)" />
+  <xacro:husarion.rosbot_xl_robot use_sim="$(arg use_sim)" simulation_engine="$(arg simulation_engine)"/>
   <xacro:include filename="$(find ros_components_description)/urdf/rplidar_s1.gazebo.xacro" ns="lidar" />
   <xacro:lidar.rplidar_s1
@@ -10,5 +11,5 @@
     rpy="0.0 0.0 ${pi}"
     use_gpu="true"
-    simulation_engine="ignition-gazebo" />
+    simulation_engine="$(arg simulation_engine)" />
   <!-- use_gpu has to be set to true, CPU lidar doesn't work in ignition - https://github.com/gazebosim/gz-sensors/issues/26 -->
 </robot>

File: rosbot_xl_description/urdf/rosbot_xl_macro.urdf.xacro (robot description, xacro)
@@ -1,5 +1,5 @@
 <?xml version='1.0'?>
 <robot xmlns:xacro="http://wiki.ros.org/xacro">
-  <xacro:macro name="rosbot_xl_robot" params="use_sim">
+  <xacro:macro name="rosbot_xl_robot" params="use_sim simulation_engine">
     <xacro:property name="wheel_radius" value="0.048" />
     <xacro:property name="wheel_separation_y" value="0.236" />
@@ -39,5 +39,10 @@
       <hardware>
         <xacro:if value="${use_sim}">
-          <plugin>ign_ros2_control/IgnitionSystem</plugin>
+          <xacro:if value="${simulation_engine == 'gazebo-ignition'}">
+            <plugin>ign_ros2_control/IgnitionSystem</plugin>
+          </xacro:if>
+          <xacro:if value="${simulation_engine == 'webots'}">
+            <plugin>webots_ros2_control::Ros2ControlSystem</plugin>
+          </xacro:if>
         </xacro:if>
         <xacro:unless value="$(arg use_sim)">
@@ -79,39 +84,63 @@
       </joint>
       <xacro:if value="${use_sim}">
-        <sensor name="imu">
-          <state_interface name="orientation.x" />
-          <state_interface name="orientation.y" />
-          <state_interface name="orientation.z" />
-          <state_interface name="orientation.w" />
-          <state_interface name="angular_velocity.x" />
-          <state_interface name="angular_velocity.y" />
-          <state_interface name="angular_velocity.z" />
-          <state_interface name="linear_acceleration.x" />
-          <state_interface name="linear_acceleration.y" />
-          <state_interface name="linear_acceleration.z" />
-        </sensor>
+        <xacro:if value="${simulation_engine == 'gazebo-ignition'}">
+          <sensor name="imu">
+            <state_interface name="orientation.x" />
+            <state_interface name="orientation.y" />
+            <state_interface name="orientation.z" />
+            <state_interface name="orientation.w" />
+            <state_interface name="angular_velocity.x" />
+            <state_interface name="angular_velocity.y" />
+            <state_interface name="angular_velocity.z" />
+            <state_interface name="linear_acceleration.x" />
+            <state_interface name="linear_acceleration.y" />
+            <state_interface name="linear_acceleration.z" />
+          </sensor>
+        </xacro:if>
       </xacro:if>
     </ros2_control>
     <xacro:if value="${use_sim}">
-      <gazebo>
-        <plugin filename="ign_ros2_control-system" name="ign_ros2_control::IgnitionROS2ControlPlugin">
-          <parameters>$(find rosbot_xl_gazebo)/config/diff_drive_controller.yaml</parameters>
-          <ros>
-            <remapping>/rosbot_xl_base_controller/cmd_vel_unstamped:=/cmd_vel</remapping>
-          </ros>
-        </plugin>
-      </gazebo>
-      <gazebo reference="imu_link">
-        <sensor name="imu" type="imu">
-          <plugin filename="ignition-gazebo-imu-system" name="ignition::gazebo::systems::Imu"></plugin>
-          <always_on>true</always_on>
-          <update_rate>25</update_rate>
-          <topic>imu/data_raw</topic>
-          <visualize>false</visualize>
-          <enable_metrics>false</enable_metrics>
-          <frame_id>imu_link</frame_id>
-          <ignition_frame_id>imu_link</ignition_frame_id>
-        </sensor>
-      </gazebo>
+      <xacro:if value="${simulation_engine == 'gazebo-ignition'}">
+        <gazebo>
+          <plugin filename="ign_ros2_control-system" name="ign_ros2_control::IgnitionROS2ControlPlugin">
+            <parameters>$(find rosbot_xl_gazebo)/config/diff_drive_controller.yaml</parameters>
+            <ros>
+              <remapping>/rosbot_xl_base_controller/cmd_vel_unstamped:=/cmd_vel</remapping>
+            </ros>
+          </plugin>
+        </gazebo>
+        <gazebo reference="imu_link">
+          <sensor name="imu" type="imu">
+            <plugin filename="ignition-gazebo-imu-system" name="ignition::gazebo::systems::Imu"></plugin>
+            <always_on>true</always_on>
+            <update_rate>25</update_rate>
+            <topic>imu/data_raw</topic>
+            <visualize>false</visualize>
+            <enable_metrics>false</enable_metrics>
+            <frame_id>imu_link</frame_id>
+            <ignition_frame_id>imu_link</ignition_frame_id>
+          </sensor>
+        </gazebo>
+      </xacro:if>
+      <xacro:if value="${simulation_engine == 'webots'}">
+        <webots>
+          <plugin type="webots_ros2_control::Ros2Control" />
+          <device reference="laser" type="Lidar">
+            <ros>
+              <topicName>/scan</topicName>
+              <updateRate>12</updateRate>
+            </ros>
+          </device>
+          <plugin type="webots_ros2_driver::Ros2IMU">
+            <enabled>true</enabled>
+            <topicName>/imu_broadcaster/imu</topicName>
+            <alwaysOn>true</alwaysOn>
+            <frameName>imu_link</frameName>
+            <gyroName>imu gyro</gyroName>
+            <accelerometerName>imu accelerometer</accelerometerName>
+            <inertialUnitName>imu inertial_unit</inertialUnitName>
+          </plugin>
+        </webots>
+      </xacro:if>
     </xacro:if>
   </xacro:macro>

Commit message: Refactor main urdf to enable selecting lidars and cameras

File: rosbot_xl_description/urdf/rosbot_xl.urdf.xacro (robot description, xacro)
@@ -3,7 +3,13 @@
   <xacro:arg name="use_sim" default="false" />
   <xacro:arg name="mecanum" default="false" />
-  <xacro:include filename="$(find rosbot_xl_description)/urdf/rosbot_xl_macro.urdf.xacro" ns="husarion" />
+  <xacro:arg name="simulation_engine" default="ignition-gazebo" />
+  <xacro:arg name="lidar_model" default="slamtec_rplidar_s1" />
+  <xacro:arg name="camera_model" default="intel_realsense_d435" />
+  <xacro:arg name="include_camera_mount" default="true" />
+  <xacro:include filename="$(find rosbot_xl_description)/urdf/rosbot_xl_macro.urdf.xacro"
+    ns="husarion" />
   <xacro:husarion.rosbot_xl_robot use_sim="$(arg use_sim)" mecanum="$(arg mecanum)" />
-  <xacro:include filename="$(find rosbot_xl_description)/urdf/components/antenna.urdf.xacro" ns="antenna" />
+  <xacro:include filename="$(find rosbot_xl_description)/urdf/components/antenna.urdf.xacro"
+    ns="antenna" />
   <xacro:antenna.antenna
     parent_link="body_link"
@@ -11,11 +17,92 @@
     rpy="0.0 0.0 0.0"
     antenna_angle="0.0" />
-  <xacro:include filename="$(find ros_components_description)/urdf/slamtec_rplidar_s1.urdf.xacro" ns="lidar" />
-  <xacro:lidar.slamtec_rplidar_s1
-    parent_link="cover_link"
-    xyz="0.0 0.0 0.0"
-    rpy="0.0 0.0 0.0"
-    use_gpu="true"
-    simulation_engine="ignition-gazebo" />
-  <!-- use_gpu has to be set to true, CPU lidar doesn't work in ignition - https://github.com/gazebosim/gz-sensors/issues/26 -->
+  <!-- INCLUDE LIDAR -->
+  <xacro:property name="lidar_model" value="$(arg lidar_model)" />
+  <xacro:property name="lidar_parent_link" value="cover_link" />
+  <xacro:property name="lidar_xyz" value="0.0 0.0 0.0" />
+  <xacro:property name="lidar_rpy" value="0.0 0.0 0.0" />
+  <xacro:property name="lidar_use_gpu" value="true" />
+  <!-- use_gpu has to be set to true, CPU lidar doesn't work in ignition -
+    https://github.com/gazebosim/gz-sensors/issues/26 -->
+  <xacro:if value="${lidar_model == 'slamtec_rplidar_s1'}">
+    <xacro:include filename="$(find ros_components_description)/urdf/slamtec_rplidar_s1.urdf.xacro"
+      ns="lidar" />
+    <xacro:lidar.slamtec_rplidar_s1
+      parent_link="${lidar_parent_link}"
+      xyz="${lidar_xyz}"
+      rpy="${lidar_rpy}"
+      use_gpu="${lidar_use_gpu}"
+      simulation_engine="$(arg simulation_engine)" />
+  </xacro:if>
+  <xacro:if value="${lidar_model == 'slamtec_rplidar_a2'}">
+    <xacro:include filename="$(find ros_components_description)/urdf/slamtec_rplidar_a2.urdf.xacro"
+      ns="lidar" />
+    <xacro:lidar.slamtec_rplidar_a2
+      parent_link="${lidar_parent_link}"
+      xyz="${lidar_xyz}"
+      rpy="${lidar_rpy}"
+      use_gpu="${lidar_use_gpu}"
+      simulation_engine="$(arg simulation_engine)" />
+  </xacro:if>
+  <xacro:if value="${lidar_model == 'slamtec_rplidar_a3'}">
+    <xacro:include filename="$(find ros_components_description)/urdf/slamtec_rplidar_a3.urdf.xacro"
+      ns="lidar" />
+    <xacro:lidar.slamtec_rplidar_a3
+      parent_link="${lidar_parent_link}"
+      xyz="${lidar_xyz}"
+      rpy="${lidar_rpy}"
+      use_gpu="${lidar_use_gpu}"
+      simulation_engine="$(arg simulation_engine)" />
+  </xacro:if>
+  <xacro:if value="${lidar_model == 'velodyne_puck'}">
+    <xacro:include filename="$(find ros_components_description)/urdf/velodyne_puck.urdf.xacro"
+      ns="lidar" />
+    <xacro:lidar.velodyne_puck
+      parent_link="${lidar_parent_link}"
+      xyz="${lidar_xyz}"
+      rpy="${lidar_rpy}"
+      use_gpu="${lidar_use_gpu}"
+      simulation_engine="$(arg simulation_engine)"
+      topic="velodyne_points" />
+  </xacro:if>
+  <xacro:if value="${lidar_model == 'ouster_os1_32'}">
+    <xacro:include filename="$(find ros_components_description)/urdf/ouster_os1_32.urdf.xacro"
+      ns="lidar" />
+    <xacro:lidar.ouster_os1_32
+      parent_link="${lidar_parent_link}"
+      xyz="${lidar_xyz}"
+      rpy="${lidar_rpy}"
+      use_gpu="${lidar_use_gpu}"
+      simulation_engine="$(arg simulation_engine)" />
+  </xacro:if>
+  <!-- INCLUDE CAMERA -->
+  <xacro:property name="camera_model" value="$(arg camera_model)" />
+  <xacro:property name="camera_parent_link" value="camera_mount_link" />
+  <xacro:property name="camera_xyz" value="0.0 0.0 0.0" />
+  <xacro:property name="camera_rpy" value="0.0 0.0 0.0" />
+  <xacro:if value="${camera_model == 'intel_realsense_d435'}">
+    <xacro:include
+      filename="$(find rosbot_xl_description)/urdf/components/intel_realsense_d435.urdf.xacro"
+      ns="camera" />
+    <xacro:camera.intel_realsense_d435
+      parent="${camera_parent_link}"
+      use_nominal_extrinsics="true"
+      add_plug="false"
+      use_mesh="true"
+      simulation_engine="$(arg simulation_engine)">
+      <origin xyz="${camera_xyz}" rpy="${camera_rpy}" />
+    </xacro:camera.intel_realsense_d435>
+    <xacro:property name="camera_set" value="True" />
+  </xacro:if>
+  <xacro:property name="include_camera_mount" value="$(arg include_camera_mount)" />
+  <xacro:if value="${include_camera_mount or camera_set}">
+    <xacro:include filename="$(find rosbot_xl_description)/urdf/components/camera_mount.urdf.xacro"
+      ns="camera_mount" />
+    <xacro:camera_mount.camera_mount
+      parent_link="cover_link"
+      xyz="-0.12 0.0 0.0"
+      rpy="0.0 0.0 0.0"
+      camera_mount_angle_1="0.0"
+      camera_mount_angle_2="0.0" />
+  </xacro:if>
 </robot>

Commit message: Temporarily remove realsense camera
needs more work to complete and urdf interface refactor is needed

File: rosbot_xl_description/urdf/rosbot_xl.urdf.xacro (robot description, xacro)
@@ -5,6 +5,6 @@
   <xacro:arg name="simulation_engine" default="ignition-gazebo" />
   <xacro:arg name="lidar_model" default="slamtec_rplidar_s1" />
-  <xacro:arg name="camera_model" default="intel_realsense_d435" />
-  <xacro:arg name="include_camera_mount" default="true" />
+  <xacro:arg name="camera_model" default="None" />
+  <xacro:arg name="include_camera_mount" default="false" />
   <xacro:include filename="$(find rosbot_xl_description)/urdf/rosbot_xl_macro.urdf.xacro"
     ns="husarion" />
@@ -66,35 +66,7 @@
       topic="velodyne_points" />
   </xacro:if>
-  <xacro:if value="${lidar_model == 'ouster_os1_32'}">
-    <xacro:include filename="$(find ros_components_description)/urdf/ouster_os1_32.urdf.xacro"
-      ns="lidar" />
-    <xacro:lidar.ouster_os1_32
-      parent_link="${lidar_parent_link}"
-      xyz="${lidar_xyz}"
-      rpy="${lidar_rpy}"
-      use_gpu="${lidar_use_gpu}"
-      simulation_engine="$(arg simulation_engine)" />
-  </xacro:if>
-  <!-- INCLUDE CAMERA -->
-  <xacro:property name="camera_model" value="$(arg camera_model)" />
-  <xacro:property name="camera_parent_link" value="camera_mount_link" />
-  <xacro:property name="camera_xyz" value="0.0 0.0 0.0" />
-  <xacro:property name="camera_rpy" value="0.0 0.0 0.0" />
-  <xacro:if value="${camera_model == 'intel_realsense_d435'}">
-    <xacro:include
-      filename="$(find rosbot_xl_description)/urdf/components/intel_realsense_d435.urdf.xacro"
-      ns="camera" />
-    <xacro:camera.intel_realsense_d435
-      parent="${camera_parent_link}"
-      use_nominal_extrinsics="true"
-      add_plug="false"
-      use_mesh="true"
-      simulation_engine="$(arg simulation_engine)">
-      <origin xyz="${camera_xyz}" rpy="${camera_rpy}" />
-    </xacro:camera.intel_realsense_d435>
-    <xacro:property name="camera_set" value="True" />
-  </xacro:if>
+  <!-- INCLUDE CAMERA MOUNT -->
   <xacro:property name="include_camera_mount" value="$(arg include_camera_mount)" />
-  <xacro:if value="${include_camera_mount or camera_set}">
+  <xacro:if value="${include_camera_mount}">
     <xacro:include filename="$(find rosbot_xl_description)/urdf/components/camera_mount.urdf.xacro"
       ns="camera_mount" />
