Commit message: Add realsense camera

File: rosbot_xl_description/urdf/rosbot_xl.urdf.xacro (robot description, xacro)
@@ -5,9 +5,10 @@
   <xacro:arg name="mecanum" default="false" />
   <xacro:arg name="lidar_model" default="slamtec_rplidar_s1" />
-  <xacro:arg name="camera_model" default="None" />
-  <xacro:arg name="include_camera_mount" default="false" />
+  <xacro:arg name="camera_model" default="intel_realsense_d435" />
+  <xacro:arg name="include_camera_mount" default="true" />
   <xacro:include filename="$(find rosbot_xl_description)/urdf/rosbot_xl_macro.urdf.xacro"
     ns="husarion" />
-  <xacro:husarion.rosbot_xl_robot use_sim="$(arg use_sim)" mecanum="$(arg mecanum)" simulation_engine='$(arg simulation_engine)'/>
+  <xacro:husarion.rosbot_xl_robot use_sim="$(arg use_sim)" mecanum="$(arg mecanum)"
+    simulation_engine='$(arg simulation_engine)' />
   <xacro:include filename="$(find rosbot_xl_description)/urdf/components/antenna.urdf.xacro"
     ns="antenna" />
@@ -68,5 +69,5 @@
   <!-- INCLUDE CAMERA MOUNT -->
   <xacro:property name="include_camera_mount" value="$(arg include_camera_mount)" />
-  <xacro:if value="${include_camera_mount}">
+  <xacro:if value="${include_camera_mount or camera_model == 'intel_realsense_d435'}">
     <xacro:include filename="$(find rosbot_xl_description)/urdf/components/camera_mount.urdf.xacro"
       ns="camera_mount" />
@@ -78,3 +79,20 @@
       camera_mount_angle_2="0.0" />
   </xacro:if>
+  <!-- INCLUDE CAMERA -->
+  <xacro:property name="camera_model" value="$(arg camera_model)" />
+  <xacro:property name="camera_parent_link" value="camera_mount_link" />
+  <xacro:property name="camera_xyz" value="0.0 0.0 0.0" />
+  <xacro:property name="camera_rpy" value="0.0 0.0 0.0" />
+  <xacro:if value="${camera_model == 'intel_realsense_d435'}">
+    <xacro:include
+      filename="$(find realsense2_description)/urdf/_d435.urdf.xacro"
+      ns="camera" />
+    <xacro:camera.sensor_d435
+      parent="${camera_parent_link}"
+      use_nominal_extrinsics="true"
+      add_plug="false"
+      use_mesh="true">
+      <origin xyz="${camera_xyz}" rpy="${camera_rpy}" />
+    </xacro:camera.sensor_d435>
+  </xacro:if>
 </robot>

Commit message: Move realsense d435 to ros_component_description and update including

File: rosbot_xl_description/urdf/rosbot_xl.urdf.xacro (robot description, xacro)
@@ -86,14 +86,14 @@
   <xacro:if value="${camera_model == 'intel_realsense_d435'}">
     <xacro:include
-      filename="$(find rosbot_xl_description)/urdf/components/intel_realsense_d435.urdf.xacro"
+      filename="$(find ros_components_description)/urdf/intel_realsense_d435.urdf.xacro"
       ns="camera" />
     <xacro:camera.intel_realsense_d435
-      parent="${camera_parent_link}"
+      parent_link="${camera_parent_link}"
+      xyz="${camera_xyz}"
+      rpy="${camera_rpy}"
+      name="camera"
+      topic="camera"
       use_nominal_extrinsics="true"
-      add_plug="false"
-      use_mesh="true"
-      simulation_engine="$(arg simulation_engine)">
-      <origin xyz="${camera_xyz}" rpy="${camera_rpy}" />
-    </xacro:camera.intel_realsense_d435>
+      simulation_engine="$(arg simulation_engine)" />
   </xacro:if>
 </robot>

Commit message: Fix rosbot urdf

File: rosbot_xl_description/urdf/rosbot_xl.urdf.xacro (robot description, xacro)
@@ -67,16 +67,4 @@
       topic="velodyne_points" />
   </xacro:if>
-  <!-- INCLUDE CAMERA MOUNT -->
-  <xacro:property name="include_camera_mount" value="$(arg include_camera_mount)" />
-  <xacro:if value="${include_camera_mount or camera_model == 'intel_realsense_d435'}">
-    <xacro:include filename="$(find rosbot_xl_description)/urdf/components/camera_mount.urdf.xacro"
-      ns="camera_mount" />
-    <xacro:camera_mount.camera_mount
-      parent_link="cover_link"
-      xyz="-0.12 0.0 0.0"
-      rpy="0.0 0.0 0.0"
-      camera_mount_angle_1="0.0"
-      camera_mount_angle_2="0.0" />
-  </xacro:if>
   <!-- INCLUDE CAMERA -->
   <xacro:property name="camera_model" value="$(arg camera_model)" />
@@ -97,3 +85,15 @@
       simulation_engine="$(arg simulation_engine)" />
   </xacro:if>
+  <!-- INCLUDE CAMERA MOUNT -->
+  <xacro:property name="include_camera_mount" value="$(arg include_camera_mount)" />
+  <xacro:if value="${include_camera_mount or camera_model == 'intel_realsense_d435'}">
+    <xacro:include filename="$(find rosbot_xl_description)/urdf/components/camera_mount.urdf.xacro"
+      ns="camera_mount" />
+    <xacro:camera_mount.camera_mount
+      parent_link="cover_link"
+      xyz="-0.12 0.0 0.0"
+      rpy="0.0 0.0 0.0"
+      camera_mount_angle_1="0.0"
+      camera_mount_angle_2="0.0" />
+  </xacro:if>
 </robot>

Commit message: Add simulation_controllers_config_file and simulation_engine arguments

File: rosbot_xl_description/urdf/rosbot_xl.urdf.xacro (robot description, xacro)
@@ -1,13 +1,17 @@
 <?xml version='1.0'?>
 <robot name="rosbot_xl" xmlns:xacro="http://www.ros.org/wiki/xacro">
-  <xacro:arg name="use_sim" default="false" />
-  <xacro:arg name="simulation_engine" default="ignition-gazebo" />
   <xacro:arg name="mecanum" default="false" />
   <xacro:arg name="lidar_model" default="slamtec_rplidar_s1" />
   <xacro:arg name="camera_model" default="None" />
   <xacro:arg name="include_camera_mount" default="false" />
+  <xacro:arg name="use_sim" default="false" />
+  <xacro:arg name="simulation_engine" default="ignition-gazebo" />
+  <xacro:arg name="simulation_controllers_config_file"
+    default="$(find rosbot_xl_controller)/config/diff_drive_controller.yaml" />
   <xacro:include filename="$(find rosbot_xl_description)/urdf/rosbot_xl_macro.urdf.xacro"
     ns="husarion" />
-  <xacro:husarion.rosbot_xl_robot use_sim="$(arg use_sim)" mecanum="$(arg mecanum)" simulation_engine='$(arg simulation_engine)'/>
+  <xacro:husarion.rosbot_xl_robot use_sim="$(arg use_sim)" mecanum="$(arg mecanum)"
+    simulation_engine="$(arg simulation_engine)"
+    simulation_controllers_config_file="$(arg simulation_controllers_config_file)" />
   <xacro:include filename="$(find rosbot_xl_description)/urdf/components/antenna.urdf.xacro"
     ns="antenna" />

File: rosbot_xl_description/urdf/rosbot_xl_macro.urdf.xacro (robot description, xacro)
@@ -1,5 +1,6 @@
 <?xml version='1.0'?>
 <robot xmlns:xacro="http://wiki.ros.org/xacro">
-  <xacro:macro name="rosbot_xl_robot" params="use_sim mecanum simulation_engine">
+  <xacro:macro name="rosbot_xl_robot"
+    params="use_sim mecanum simulation_engine simulation_controllers_config_file">
     <xacro:if value="${mecanum}">
       <xacro:property name="wheel_radius" value="0.05" />
@@ -14,8 +15,12 @@
     <xacro:body.body wheel_radius="${wheel_radius}" />
     <!-- WHEEL DECLARATION -->
-    <xacro:wheel.wheel wheel_radius="${wheel_radius}" prefix="fl" mecanum="${mecanum}" use_sim="$(arg use_sim)" />
-    <xacro:wheel.wheel wheel_radius="${wheel_radius}" prefix="fr" mecanum="${mecanum}" use_sim="$(arg use_sim)" />
-    <xacro:wheel.wheel wheel_radius="${wheel_radius}" prefix="rl" mecanum="${mecanum}" use_sim="$(arg use_sim)" />
-    <xacro:wheel.wheel wheel_radius="${wheel_radius}" prefix="rr" mecanum="${mecanum}" use_sim="$(arg use_sim)" />
+    <xacro:wheel.wheel wheel_radius="${wheel_radius}" prefix="fl" mecanum="${mecanum}"
+      use_sim="$(arg use_sim)" />
+    <xacro:wheel.wheel wheel_radius="${wheel_radius}" prefix="fr" mecanum="${mecanum}"
+      use_sim="$(arg use_sim)" />
+    <xacro:wheel.wheel wheel_radius="${wheel_radius}" prefix="rl" mecanum="${mecanum}"
+      use_sim="$(arg use_sim)" />
+    <xacro:wheel.wheel wheel_radius="${wheel_radius}" prefix="rr" mecanum="${mecanum}"
+      use_sim="$(arg use_sim)" />
     <!-- ROS2 CONTROL -->
     <xacro:unless value="$(arg use_sim)">
@@ -56,8 +61,8 @@
           <!-- order of velocity commands to be published in motors_cmd Float32MultiArray msg -->
           <param name="velocity_command_joint_order">
-                rr_wheel_joint,
-                rl_wheel_joint,
-                fr_wheel_joint,
-                fl_wheel_joint
+            rr_wheel_joint,
+            rl_wheel_joint,
+            fr_wheel_joint,
+            fl_wheel_joint
           </param>
         </xacro:unless>
@@ -103,11 +108,7 @@
       <xacro:if value="${simulation_engine == 'ignition-gazebo'}">
         <gazebo>
-          <plugin filename="ign_ros2_control-system" name="ign_ros2_control::IgnitionROS2ControlPlugin">
-            <xacro:if value="${mecanum}">
-              <parameters>$(find rosbot_xl_controller)/config/mecanum_drive_controller.yaml</parameters>
-            </xacro:if>
-            <xacro:unless value="${mecanum}">
-              <parameters>$(find rosbot_xl_controller)/config/diff_drive_controller.yaml</parameters>
-            </xacro:unless>
+          <plugin filename="ign_ros2_control-system"
+            name="ign_ros2_control::IgnitionROS2ControlPlugin">
+            <parameters>${simulation_controllers_config_file}</parameters>
             <controller_manager_prefix_node_name>simulation</controller_manager_prefix_node_name>
             <ros>

Commit message: add ZED urdf + list of choices

File: rosbot_xl_description/urdf/rosbot_xl.urdf.xacro (robot description, xacro)
@@ -3,5 +3,5 @@
   <xacro:arg name="mecanum" default="false" />
   <xacro:arg name="lidar_model" default="slamtec_rplidar_s1" />
-  <xacro:arg name="camera_model" default="None" />
+  <xacro:arg name="camera_model" default="stereolabs_zed2" />
   <xacro:arg name="include_camera_mount" default="false" />
   <xacro:arg name="use_sim" default="false" />
@@ -24,5 +24,5 @@
   <xacro:property name="lidar_model" value="$(arg lidar_model)" />
   <xacro:property name="lidar_parent_link" value="cover_link" />
-  <xacro:property name="lidar_xyz" value="0.0 0.0 0.0" />
+  <xacro:property name="lidar_xyz" value="0.02 0.0 0.0" />
   <xacro:property name="lidar_rpy" value="0.0 0.0 0.0" />
   <xacro:property name="lidar_use_gpu" value="true" />
@@ -90,7 +90,39 @@
       simulation_engine="$(arg simulation_engine)" />
   </xacro:if>
-  <!-- INCLUDE CAMERA MOUNT -->
+  <xacro:if value="${camera_model.startswith('stereolabs')}">
+    <xacro:if value="${camera_model == 'stereolabs_zed'}">
+      <xacro:property name="camera_model_type" value="zed" />
+    </xacro:if>
+    <xacro:if value="${camera_model == 'stereolabs_zedm'}">
+      <xacro:property name="camera_model_type" value="zedm" />
+    </xacro:if>
+    <xacro:if value="${camera_model == 'stereolabs_zed2'}">
+      <xacro:property name="camera_model_type" value="zed2" />
+    </xacro:if>
+    <xacro:if value="${camera_model == 'stereolabs_zed2i'}">
+      <xacro:property name="camera_model_type" value="zed2i" />
+    </xacro:if>
+    <xacro:if value="${camera_model == 'stereolabs_zedx'}">
+      <xacro:property name="camera_model_type" value="zedx" />
+    </xacro:if>
+    <xacro:if value="${camera_model == 'stereolabs_zedxm'}">
+      <xacro:property name="camera_model_type" value="zedxm" />
+    </xacro:if>
+    <xacro:include
+    filename="$(find ros_components_description)/urdf/stereolabs_zed.urdf.xacro"
+    ns="camera" />
+    <xacro:camera.zed_camera
+      parent_link="${camera_parent_link}"
+      xyz="${camera_xyz}"
+      rpy="${camera_rpy}"
+      model="${camera_model_type}"
+      name="camera"
+      topic="camera"
+      use_nominal_extrinsics="$(arg use_sim)"
+      simulation_engine="$(arg simulation_engine)" />
+  </xacro:if>
+  <!-- INCLUDE CAMERA MOUNT - add if camera_model is not empty -->
   <xacro:property name="include_camera_mount" value="$(arg include_camera_mount)" />
-  <xacro:if value="${include_camera_mount or camera_model == 'intel_realsense_d435'}">
+  <xacro:if value="${include_camera_mount or camera_model != ''}">
     <xacro:include filename="$(find rosbot_xl_description)/urdf/components/camera_mount.urdf.xacro"
       ns="camera_mount" />

Commit message: add ZED urdf + list of choices (#49)
* add ZED urdf + list of choices

* choices to root dir

* readme

* Update README.md

* Update README.md

* fix gz bridge

* Remapping

* Add word

* add suggestions

* add urdf tests

* Add None and velodyne to test

* Update pre-commit and fix tests

File: rosbot_xl_description/urdf/rosbot_xl.urdf.xacro (robot description, xacro)
@@ -3,5 +3,5 @@
   <xacro:arg name="mecanum" default="false" />
   <xacro:arg name="lidar_model" default="slamtec_rplidar_s1" />
-  <xacro:arg name="camera_model" default="None" />
+  <xacro:arg name="camera_model" default="intel_realsense_d435" />
   <xacro:arg name="include_camera_mount" default="false" />
   <xacro:arg name="use_sim" default="false" />
@@ -24,5 +24,5 @@
   <xacro:property name="lidar_model" value="$(arg lidar_model)" />
   <xacro:property name="lidar_parent_link" value="cover_link" />
-  <xacro:property name="lidar_xyz" value="0.0 0.0 0.0" />
+  <xacro:property name="lidar_xyz" value="0.02 0.0 0.0" />
   <xacro:property name="lidar_rpy" value="0.0 0.0 0.0" />
   <xacro:property name="lidar_use_gpu" value="true" />
@@ -90,7 +90,39 @@
       simulation_engine="$(arg simulation_engine)" />
   </xacro:if>
-  <!-- INCLUDE CAMERA MOUNT -->
+  <xacro:if value="${camera_model.startswith('stereolabs')}">
+    <xacro:if value="${camera_model == 'stereolabs_zed'}">
+      <xacro:property name="camera_model_type" value="zed" />
+    </xacro:if>
+    <xacro:if value="${camera_model == 'stereolabs_zedm'}">
+      <xacro:property name="camera_model_type" value="zedm" />
+    </xacro:if>
+    <xacro:if value="${camera_model == 'stereolabs_zed2'}">
+      <xacro:property name="camera_model_type" value="zed2" />
+    </xacro:if>
+    <xacro:if value="${camera_model == 'stereolabs_zed2i'}">
+      <xacro:property name="camera_model_type" value="zed2i" />
+    </xacro:if>
+    <xacro:if value="${camera_model == 'stereolabs_zedx'}">
+      <xacro:property name="camera_model_type" value="zedx" />
+    </xacro:if>
+    <xacro:if value="${camera_model == 'stereolabs_zedxm'}">
+      <xacro:property name="camera_model_type" value="zedxm" />
+    </xacro:if>
+    <xacro:include
+    filename="$(find ros_components_description)/urdf/stereolabs_zed.urdf.xacro"
+    ns="camera" />
+    <xacro:camera.zed_camera
+      parent_link="${camera_parent_link}"
+      xyz="${camera_xyz}"
+      rpy="${camera_rpy}"
+      model="${camera_model_type}"
+      name="camera"
+      topic="camera"
+      use_nominal_extrinsics="$(arg use_sim)"
+      simulation_engine="$(arg simulation_engine)" />
+  </xacro:if>
+  <!-- INCLUDE CAMERA MOUNT - add if camera_model is not empty -->
   <xacro:property name="include_camera_mount" value="$(arg include_camera_mount)" />
-  <xacro:if value="${include_camera_mount or camera_model == 'intel_realsense_d435'}">
+  <xacro:if value="${include_camera_mount or camera_model != 'None'}">
     <xacro:include filename="$(find rosbot_xl_description)/urdf/components/camera_mount.urdf.xacro"
       ns="camera_mount" />

Commit message: delete unnecessary

File: rosbot_xl_description/urdf/rosbot_xl.urdf.xacro (robot description, xacro)
@@ -24,5 +24,5 @@
   <xacro:property name="lidar_model" value="$(arg lidar_model)" />
   <xacro:property name="lidar_parent_link" value="cover_link" />
-  <xacro:property name="lidar_xyz" value="0.02 0.0 0.0" />
+  <xacro:property name="lidar_xyz" value="0.0 0.0 0.0" />
   <xacro:property name="lidar_rpy" value="0.0 0.0 0.0" />
   <xacro:property name="lidar_use_gpu" value="true" />
@@ -116,6 +116,4 @@
       xyz="${camera_xyz}"
       rpy="${camera_rpy}"
-      name="camera"
-      topic="camera"
       use_nominal_extrinsics="$(arg use_sim)"
       simulation_engine="$(arg simulation_engine)" />
@@ -129,5 +127,4 @@
       xyz="${camera_xyz}"
       rpy="${camera_rpy}"
-      name="camera"
       simulation_engine="$(arg simulation_engine)" />
   </xacro:if>
@@ -159,5 +156,4 @@
       rpy="${camera_rpy}"
       model="${camera_model_type}"
-      name="camera"
       topic="${camera_model_type}"
       simulation_engine="$(arg simulation_engine)" />

Commit message: test_pass

File: rosbot_xl_description/urdf/rosbot_xl.urdf.xacro (robot description, xacro)
@@ -24,20 +24,9 @@
   <xacro:property name="lidar_model" value="$(arg lidar_model)" />
   <xacro:property name="lidar_parent_link" value="cover_link" />
-  <xacro:property name="lidar_xyz" value="0.0 0.0 0.0" />
+  <xacro:property name="lidar_xyz" value="0.02 0.0 0.0" />
   <xacro:property name="lidar_rpy" value="0.0 0.0 0.0" />
   <xacro:property name="lidar_use_gpu" value="true" />
   <!-- use_gpu has to be set to true, CPU lidar doesn't work in ignition -
     https://github.com/gazebosim/gz-sensors/issues/26 -->
-  <xacro:if value="${lidar_model == 'ouster_os1_32'}">
-    <xacro:include filename="$(find ros_components_description)/urdf/ouster_os1_32.urdf.xacro"
-      ns="lidar" />
-    <xacro:lidar.ouster_os1_32
-      parent_link="${lidar_parent_link}"
-      xyz="${lidar_xyz}"
-      rpy="${lidar_rpy}"
-      use_gpu="${lidar_use_gpu}"
-      simulation_engine="$(arg simulation_engine)"
-      topic="velodyne_points" />
-  </xacro:if>
   <xacro:if value="${lidar_model == 'slamtec_rplidar_s1'}">
     <xacro:include filename="$(find ros_components_description)/urdf/slamtec_rplidar_s1.urdf.xacro"
@@ -156,5 +145,4 @@
       rpy="${camera_rpy}"
       model="${camera_model_type}"
-      topic="${camera_model_type}"
       simulation_engine="$(arg simulation_engine)" />
   </xacro:if>
