Commit message: Add namespace (#59)
* added tf_prefixes to the urdf

Signed-off-by: Jakub Delicat <jakub.delicat@husarion.com>

* add namespace to world list

Signed-off-by: Jakub Delicat <jakub.delicat@husarion.com>

* tf_prefix for controller

Signed-off-by: Jakub Delicat <jakub.delicat@husarion.com>

* added namespace in mecanum test

Signed-off-by: Jakub Delicat <jakub.delicat@husarion.com>

* Added namespace to bringup

Signed-off-by: Jakub Delicat <jakub.delicat@husarion.com>

* added fixed namespaces to description and controller

Signed-off-by: Jakub Delicat <jakub.delicat@husarion.com>

* Updated worldlist

Signed-off-by: Jakub Delicat <jakub.delicat@husarion.com>

* added multirobot test to controllers

Signed-off-by: Jakub Delicat <jakub.delicat@husarion.com>

* Added rosbot_xl_bringup multirobot test

Signed-off-by: Jakub Delicat <jakub.delicat@husarion.com>

* fixed .repos

Signed-off-by: Jakub Delicat <jakub.delicat@husarion.com>

* updated submodules

Signed-off-by: Jakub Delicat <jakub.delicat@husarion.com>

* updated industrial

Signed-off-by: Jakub Delicat <jakub.delicat@husarion.com>

* first simulation launch

Signed-off-by: Jakub Delicat <jakub.delicat@husarion.com>

* moved remapings to the urdf of intel

Signed-off-by: Jakub Delicat <jakub.delicat@husarion.com>

* updated submodules

Signed-off-by: Jakub Delicat <jakub.delicat@husarion.com>

* Added tf fixer | remapped pointcloud topic in .yaml

Signed-off-by: Jakub Delicat <jakub.delicat@husarion.com>

* added astra

Signed-off-by: Jakub Delicat <jakub.delicat@husarion.com>

* Added zed

Signed-off-by: Jakub Delicat <jakub.delicat@husarion.com>

* Added namespaced velodyne

Signed-off-by: Jakub Delicat <jakub.delicat@husarion.com>

* added remappings for velodyne

Signed-off-by: Jakub Delicat <jakub.delicat@husarion.com>

* added tests from rosbot_ros | fixed imu

Signed-off-by: Jakub Delicat <jakub.delicat@husarion.com>

* add to the worldlist

Signed-off-by: Jakub Delicat <jakub.delicat@husarion.com>

* lint | added multirobot simulation tests

Signed-off-by: Jakub Delicat <jakub.delicat@husarion.com>

* added multirobot tests | added tf_ros2_py dependency to the rosbot_ros

Signed-off-by: Jakub Delicat <jakub.delicat@husarion.com>

* fixed xacro test

Signed-off-by: Jakub Delicat <jakub.delicat@husarion.com>

* fixed removeing gz tests

Signed-off-by: Jakub Delicat <jakub.delicat@husarion.com>

* created src insisde industrial ci

Signed-off-by: Jakub Delicat <jakub.delicat@husarion.com>

* removed geometry2

Signed-off-by: Jakub Delicat <jakub.delicat@husarion.com>

* Update industrial_ci.yaml

* added psutil dep

Signed-off-by: Jakub Delicat <jakub.delicat@husarion.com>

* added psutil dep

Signed-off-by: Jakub Delicat <jakub.delicat@husarion.com>

* added psutil dep

Signed-off-by: Jakub Delicat <jakub.delicat@husarion.com>

* formatted package.xml files | removed one robot from controller tests

Signed-off-by: Jakub Delicat <jakub.delicat@husarion.com>

* updated package.xml in rosbot_xl_description

Signed-off-by: Jakub Delicat <jakub.delicat@husarion.com>

* updated tests

Signed-off-by: Jakub Delicat <jakub.delicat@husarion.com>

* Removed multirobot tests

Signed-off-by: Jakub Delicat <jakub.delicat@husarion.com>

* Removed multirobot tests

Signed-off-by: Jakub Delicat <jakub.delicat@husarion.com>

* Revert "Removed multirobot tests"

This reverts commit 30cf4c9beaed45f9c719c1a32722946a8d616e0b.

* Added delayed spawn for controllers

Signed-off-by: Jakub Delicat <jakub.delicat@husarion.com>

* Added spawner to worldlist

Signed-off-by: Jakub Delicat <jakub.delicat@husarion.com>

* bringup and controllers passes industrial

Signed-off-by: Jakub Delicat <jakub.delicat@husarion.com>

* Testing gazebo

Signed-off-by: Jakub Delicat <jakub.delicat@husarion.com>

* industrial passes

Signed-off-by: Jakub Delicat <jakub.delicat@husarion.com>

* Passing industrial tests

Signed-off-by: Jakub Delicat <jakub.delicat@husarion.com>

* removed comments

Signed-off-by: Jakub Delicat <jakub.delicat@husarion.com>

* Added bringup and controller tests

Signed-off-by: Jakub Delicat <jakub.delicat@husarion.com>

* typo

Signed-off-by: Jakub Delicat <jakub.delicat@husarion.com>

* Update test_multirobot_controllers.py

* updated repos

Signed-off-by: Jakub Delicat <jakub.delicat@husarion.com>

* rosbot_hardware_interfaces main to ros2

Signed-off-by: Jakub Delicat <jakub.delicat@husarion.com>

* Add namespace suggestions (#60)

* Workflow merge many steps and pre-commit

* test bringup refactor

* test controller refactor

* test

* New tests

* typo

* 2024 Husarion copyright

* Jakub suggestions

* revert older version of black

* Add info

* Next suggestions

* spell fix

* remove sleep

* remove submodule

* debug fix

* timeout increase

* Apply suggestions from code review

Co-authored-by: Jakub Delicat <109142865+delihus@users.noreply.github.com>

* Apply suggestions from code review

* Update .github/workflows/bump_version.yaml

---------

Co-authored-by: Jakub Delicat <109142865+delihus@users.noreply.github.com>

---------

Signed-off-by: Jakub Delicat <jakub.delicat@husarion.com>
Co-authored-by: rafal-gorecki <126687345+rafal-gorecki@users.noreply.github.com>

File: rosbot_xl_description/urdf/rosbot_xl.urdf.xacro (robot description, xacro)
@@ -7,11 +7,12 @@
   <xacro:arg name="use_sim" default="false" />
   <xacro:arg name="simulation_engine" default="ignition-gazebo" />
-  <xacro:arg name="simulation_controllers_config_file"
-    default="$(find rosbot_xl_controller)/config/diff_drive_controller.yaml" />
+  <xacro:arg name="namespace" default="None" />
   <xacro:include filename="$(find rosbot_xl_description)/urdf/rosbot_xl_macro.urdf.xacro"
     ns="husarion" />
-  <xacro:husarion.rosbot_xl_robot use_sim="$(arg use_sim)" mecanum="$(arg mecanum)"
+  <xacro:husarion.rosbot_xl_robot
+    use_sim="$(arg use_sim)"
+    mecanum="$(arg mecanum)"
     simulation_engine="$(arg simulation_engine)"
-    simulation_controllers_config_file="$(arg simulation_controllers_config_file)" />
+    namespace="$(arg namespace)" />
   <xacro:include filename="$(find rosbot_xl_description)/urdf/components/antenna.urdf.xacro"
     ns="antenna" />
@@ -37,5 +38,6 @@
       rpy="${lidar_rpy}"
       use_gpu="${lidar_use_gpu}"
-      simulation_engine="$(arg simulation_engine)" />
+      simulation_engine="$(arg simulation_engine)"
+      namespace="$(arg namespace)" />
   </xacro:if>
   <xacro:if value="${lidar_model == 'slamtec_rplidar_s2'}">
@@ -47,5 +49,6 @@
       rpy="${lidar_rpy}"
       use_gpu="${lidar_use_gpu}"
-      simulation_engine="$(arg simulation_engine)" />
+      simulation_engine="$(arg simulation_engine)"
+      namespace="$(arg namespace)" />
   </xacro:if>
   <xacro:if value="${lidar_model == 'slamtec_rplidar_s3'}">
@@ -57,5 +60,6 @@
       rpy="${lidar_rpy}"
       use_gpu="${lidar_use_gpu}"
-      simulation_engine="$(arg simulation_engine)" />
+      simulation_engine="$(arg simulation_engine)"
+      namespace="$(arg namespace)" />
   </xacro:if>
   <xacro:if value="${lidar_model == 'slamtec_rplidar_a2'}">
@@ -67,5 +71,6 @@
       rpy="${lidar_rpy}"
       use_gpu="${lidar_use_gpu}"
-      simulation_engine="$(arg simulation_engine)" />
+      simulation_engine="$(arg simulation_engine)"
+      namespace="$(arg namespace)" />
   </xacro:if>
   <xacro:if value="${lidar_model == 'slamtec_rplidar_a3'}">
@@ -77,5 +82,6 @@
       rpy="${lidar_rpy}"
       use_gpu="${lidar_use_gpu}"
-      simulation_engine="$(arg simulation_engine)" />
+      simulation_engine="$(arg simulation_engine)"
+      namespace="$(arg namespace)" />
   </xacro:if>
   <xacro:if value="${lidar_model == 'velodyne_puck'}">
@@ -88,5 +94,6 @@
       use_gpu="${lidar_use_gpu}"
       simulation_engine="$(arg simulation_engine)"
-      topic="velodyne_points" />
+      topic="velodyne_points"
+      namespace="$(arg namespace)" />
   </xacro:if>
   <!-- INCLUDE CAMERA -->
@@ -106,5 +113,6 @@
       rpy="${camera_rpy}"
       use_nominal_extrinsics="$(arg use_sim)"
-      simulation_engine="$(arg simulation_engine)" />
+      simulation_engine="$(arg simulation_engine)"
+      namespace="$(arg namespace)" />
   </xacro:if>
   <xacro:if value="${camera_model == 'orbbec_astra'}">
@@ -116,5 +124,6 @@
       xyz="${camera_xyz}"
       rpy="${camera_rpy}"
-      simulation_engine="$(arg simulation_engine)" />
+      simulation_engine="$(arg simulation_engine)"
+      namespace="$(arg namespace)" />
   </xacro:if>
   <xacro:if value="${camera_model.startswith('stereolabs')}">
@@ -145,5 +154,6 @@
       rpy="${camera_rpy}"
       model="${camera_model_type}"
-      simulation_engine="$(arg simulation_engine)" />
+      simulation_engine="$(arg simulation_engine)"
+      namespace="$(arg namespace)" />
   </xacro:if>
   <!-- INCLUDE CAMERA MOUNT - add if camera_model is not empty -->

File: rosbot_xl_description/urdf/rosbot_xl_macro.urdf.xacro (robot description, xacro)
@@ -2,5 +2,13 @@
 <robot xmlns:xacro="http://wiki.ros.org/xacro">
   <xacro:macro name="rosbot_xl_robot"
-    params="use_sim mecanum simulation_engine simulation_controllers_config_file">
+    params="use_sim mecanum simulation_engine namespace">
+    <xacro:if value="${namespace == 'None'}">
+      <xacro:property name="ns" value="" />
+      <xacro:property name="gz_control_namespace" value="/" />
+    </xacro:if>
+    <xacro:unless value="${namespace == 'None'}">
+        <xacro:property name="ns" value="${namespace}/" />
+        <xacro:property name="gz_control_namespace" value="${namespace}" />
+    </xacro:unless>
     <xacro:if value="${mecanum}">
       <xacro:property name="wheel_radius" value="0.05" />
@@ -15,15 +23,15 @@
     <xacro:body.body wheel_radius="${wheel_radius}" />
     <!-- WHEEL DECLARATION -->
-    <xacro:wheel.wheel wheel_radius="${wheel_radius}" prefix="fl" mecanum="${mecanum}"
+    <xacro:wheel.wheel wheel_radius="${wheel_radius}" side="fl" mecanum="${mecanum}"
       use_sim="$(arg use_sim)" />
-    <xacro:wheel.wheel wheel_radius="${wheel_radius}" prefix="fr" mecanum="${mecanum}"
+    <xacro:wheel.wheel wheel_radius="${wheel_radius}" side="fr" mecanum="${mecanum}"
       use_sim="$(arg use_sim)" />
-    <xacro:wheel.wheel wheel_radius="${wheel_radius}" prefix="rl" mecanum="${mecanum}"
+    <xacro:wheel.wheel wheel_radius="${wheel_radius}" side="rl" mecanum="${mecanum}"
       use_sim="$(arg use_sim)" />
-    <xacro:wheel.wheel wheel_radius="${wheel_radius}" prefix="rr" mecanum="${mecanum}"
+    <xacro:wheel.wheel wheel_radius="${wheel_radius}" side="rr" mecanum="${mecanum}"
       use_sim="$(arg use_sim)" />
     <!-- ROS2 CONTROL -->
     <xacro:unless value="$(arg use_sim)">
-      <ros2_control name="imu" type="sensor">
+      <ros2_control name="${ns}imu" type="sensor">
         <hardware>
           <plugin>rosbot_hardware_interfaces/RosbotImuSensor</plugin>
@@ -31,5 +39,5 @@
           <param name="connection_check_period_ms">500</param>
         </hardware>
-        <sensor name="imu">
+        <sensor name="${ns}imu">
           <state_interface name="orientation.x" />
           <state_interface name="orientation.y" />
@@ -45,5 +53,5 @@
       </ros2_control>
     </xacro:unless>
-    <ros2_control name="wheels" type="system">
+    <ros2_control name="${ns}wheels" type="system">
       <hardware>
         <xacro:if value="${use_sim}">
@@ -90,5 +98,5 @@
       <xacro:if value="${use_sim}">
         <xacro:if value="${simulation_engine == 'ignition-gazebo'}">
-          <sensor name="imu">
+          <sensor name="${ns}imu">
             <state_interface name="orientation.x" />
             <state_interface name="orientation.y" />
@@ -108,23 +116,30 @@
       <xacro:if value="${simulation_engine == 'ignition-gazebo'}">
         <gazebo>
-          <plugin filename="ign_ros2_control-system"
-            name="ign_ros2_control::IgnitionROS2ControlPlugin">
-            <parameters>${simulation_controllers_config_file}</parameters>
-            <controller_manager_prefix_node_name>simulation</controller_manager_prefix_node_name>
+          <plugin filename="ign_ros2_control-system" name="ign_ros2_control::IgnitionROS2ControlPlugin">
+            <xacro:if value="${mecanum}">
+              <parameters>$(find rosbot_xl_controller)/config/mecanum_drive_controller.yaml</parameters>
+            </xacro:if>
+            <xacro:unless value="${mecanum}">
+              <parameters>$(find rosbot_xl_controller)/config/diff_drive_controller.yaml</parameters>
+            </xacro:unless>
             <ros>
-              <remapping>/rosbot_xl_base_controller/cmd_vel_unstamped:=/cmd_vel</remapping>
+              <namespace>${gz_control_namespace}</namespace>
+              <remapping>rosbot_xl_base_controller/cmd_vel_unstamped:=cmd_vel</remapping>
+              <remapping>/tf:=tf</remapping>
             </ros>
           </plugin>
         </gazebo>
         <gazebo reference="imu_link">
-          <sensor name="imu" type="imu">
-            <plugin filename="ignition-gazebo-imu-system" name="ignition::gazebo::systems::Imu"></plugin>
+          <sensor name="${ns}imu" type="imu">
             <always_on>true</always_on>
             <update_rate>25</update_rate>
-            <topic>imu/data_raw</topic>
+            <topic>${ns}imu/data_raw</topic>
             <visualize>false</visualize>
             <enable_metrics>false</enable_metrics>
             <frame_id>imu_link</frame_id>
             <ignition_frame_id>imu_link</ignition_frame_id>
+            <ros>
+              <namespace>${ns}</namespace>
+            </ros>
           </sensor>
         </gazebo>

File: rosbot_xl_description/urdf/wheel.urdf.xacro (robot description, xacro)
@@ -1,5 +1,5 @@
 <?xml version="1.0" encoding="utf-8"?>
 <robot xmlns:xacro="http://www.ros.org/wiki/xacro">
-  <xacro:macro name="wheel" params="wheel_radius prefix mecanum use_sim">
+  <xacro:macro name="wheel" params="wheel_radius side mecanum use_sim">
     <xacro:property name="wheel_separation_x" value="0.170" />
     <xacro:if value="${mecanum}">
@@ -21,5 +21,5 @@
       <xacro:property name="wheel_separation_y" value="0.248" />
     </xacro:unless>
-    <xacro:if value="${prefix == 'fl'}">
+    <xacro:if value="${side == 'fl'}">
       <xacro:property name="x" value="${wheel_separation_x/2}" />
       <xacro:property name="y" value="${wheel_separation_y/2}" />
@@ -28,5 +28,5 @@
       <xacro:property name="fdir" value="1 -1 0" />
     </xacro:if>
-    <xacro:if value="${prefix == 'fr'}">
+    <xacro:if value="${side == 'fr'}">
       <xacro:property name="x" value="${wheel_separation_x/2}" />
       <xacro:property name="y" value="${-wheel_separation_y/2}" />
@@ -35,5 +35,5 @@
       <xacro:property name="fdir" value="1 1 0" />
     </xacro:if>
-    <xacro:if value="${prefix == 'rl'}">
+    <xacro:if value="${side == 'rl'}">
       <xacro:property name="x" value="${-wheel_separation_x/2}" />
       <xacro:property name="y" value="${wheel_separation_y/2}" />
@@ -42,5 +42,5 @@
       <xacro:property name="fdir" value="1 1 0" />
     </xacro:if>
-    <xacro:if value="${prefix == 'rr'}">
+    <xacro:if value="${side == 'rr'}">
       <xacro:property name="x" value="${-wheel_separation_x/2}" />
       <xacro:property name="y" value="${-wheel_separation_y/2}" />
@@ -49,7 +49,7 @@
       <xacro:property name="fdir" value="1 -1 0" />
     </xacro:if>
-    <joint name="${prefix}_wheel_joint" type="continuous">
+    <joint name="${side}_wheel_joint" type="continuous">
       <parent link="body_link" />
-      <child link="${prefix}_wheel_link" />
+      <child link="${side}_wheel_link" />
       <origin xyz="${x} ${y} 0.0" rpy="0.0 0.0 0.0" />
       <axis xyz="0.0 1.0 0.0" />
@@ -57,5 +57,5 @@
       <dynamics damping="0.001" friction="0.001" />
     </joint>
-    <link name="${prefix}_wheel_link">
+    <link name="${side}_wheel_link">
       <visual>
         <geometry>
@@ -78,5 +78,5 @@
     </link>
     <xacro:if value="${use_sim}">
-      <gazebo reference="${prefix}_wheel_link" xmlns:ignition="http://ignitionrobotics.org/schema">
+      <gazebo reference="${side}_wheel_link" xmlns:ignition="http://ignitionrobotics.org/schema">
         <collision>
           <surface>

Commit message: Fix components urdf

File: rosbot_xl_description/urdf/rosbot_xl.urdf.xacro (robot description, xacro)
@@ -27,7 +27,4 @@
   <xacro:property name="lidar_xyz" value="0.02 0.0 0.0" />
   <xacro:property name="lidar_rpy" value="0.0 0.0 0.0" />
-  <xacro:property name="lidar_use_gpu" value="true" />
-  <!-- use_gpu has to be set to true, CPU lidar doesn't work in ignition -
-    https://github.com/gazebosim/gz-sensors/issues/26 -->
   <xacro:if value="${lidar_model == 'slamtec_rplidar_s1'}">
     <xacro:include filename="$(find ros_components_description)/urdf/slamtec_rplidar_s1.urdf.xacro"
@@ -37,6 +34,4 @@
       xyz="${lidar_xyz}"
       rpy="${lidar_rpy}"
-      use_gpu="${lidar_use_gpu}"
-      simulation_engine="$(arg simulation_engine)"
       namespace="$(arg namespace)" />
   </xacro:if>
@@ -48,6 +43,4 @@
       xyz="${lidar_xyz}"
       rpy="${lidar_rpy}"
-      use_gpu="${lidar_use_gpu}"
-      simulation_engine="$(arg simulation_engine)"
       namespace="$(arg namespace)" />
   </xacro:if>
@@ -59,6 +52,4 @@
       xyz="${lidar_xyz}"
       rpy="${lidar_rpy}"
-      use_gpu="${lidar_use_gpu}"
-      simulation_engine="$(arg simulation_engine)"
       namespace="$(arg namespace)" />
   </xacro:if>
@@ -70,6 +61,4 @@
       xyz="${lidar_xyz}"
       rpy="${lidar_rpy}"
-      use_gpu="${lidar_use_gpu}"
-      simulation_engine="$(arg simulation_engine)"
       namespace="$(arg namespace)" />
   </xacro:if>
@@ -81,6 +70,4 @@
       xyz="${lidar_xyz}"
       rpy="${lidar_rpy}"
-      use_gpu="${lidar_use_gpu}"
-      simulation_engine="$(arg simulation_engine)"
       namespace="$(arg namespace)" />
   </xacro:if>
@@ -92,6 +79,4 @@
       xyz="${lidar_xyz}"
       rpy="${lidar_rpy}"
-      use_gpu="${lidar_use_gpu}"
-      simulation_engine="$(arg simulation_engine)"
       topic="velodyne_points"
       namespace="$(arg namespace)" />
@@ -113,5 +98,4 @@
       rpy="${camera_rpy}"
       use_nominal_extrinsics="$(arg use_sim)"
-      simulation_engine="$(arg simulation_engine)"
       namespace="$(arg namespace)" />
   </xacro:if>
@@ -124,5 +108,4 @@
       xyz="${camera_xyz}"
       rpy="${camera_rpy}"
-      simulation_engine="$(arg simulation_engine)"
       namespace="$(arg namespace)" />
   </xacro:if>
@@ -154,5 +137,4 @@
       rpy="${camera_rpy}"
       model="${camera_model_type}"
-      simulation_engine="$(arg simulation_engine)"
       namespace="$(arg namespace)" />
   </xacro:if>

Commit message: Fix components urdf (#68)
* Fix components urdf

* unused topic remove

File: rosbot_xl_description/urdf/rosbot_xl.urdf.xacro (robot description, xacro)
@@ -27,7 +27,4 @@
   <xacro:property name="lidar_xyz" value="0.02 0.0 0.0" />
   <xacro:property name="lidar_rpy" value="0.0 0.0 0.0" />
-  <xacro:property name="lidar_use_gpu" value="true" />
-  <!-- use_gpu has to be set to true, CPU lidar doesn't work in ignition -
-    https://github.com/gazebosim/gz-sensors/issues/26 -->
   <xacro:if value="${lidar_model == 'slamtec_rplidar_s1'}">
     <xacro:include filename="$(find ros_components_description)/urdf/slamtec_rplidar_s1.urdf.xacro"
@@ -37,6 +34,4 @@
       xyz="${lidar_xyz}"
       rpy="${lidar_rpy}"
-      use_gpu="${lidar_use_gpu}"
-      simulation_engine="$(arg simulation_engine)"
       namespace="$(arg namespace)" />
   </xacro:if>
@@ -48,6 +43,4 @@
       xyz="${lidar_xyz}"
       rpy="${lidar_rpy}"
-      use_gpu="${lidar_use_gpu}"
-      simulation_engine="$(arg simulation_engine)"
       namespace="$(arg namespace)" />
   </xacro:if>
@@ -59,6 +52,4 @@
       xyz="${lidar_xyz}"
       rpy="${lidar_rpy}"
-      use_gpu="${lidar_use_gpu}"
-      simulation_engine="$(arg simulation_engine)"
       namespace="$(arg namespace)" />
   </xacro:if>
@@ -70,6 +61,4 @@
       xyz="${lidar_xyz}"
       rpy="${lidar_rpy}"
-      use_gpu="${lidar_use_gpu}"
-      simulation_engine="$(arg simulation_engine)"
       namespace="$(arg namespace)" />
   </xacro:if>
@@ -81,6 +70,4 @@
       xyz="${lidar_xyz}"
       rpy="${lidar_rpy}"
-      use_gpu="${lidar_use_gpu}"
-      simulation_engine="$(arg simulation_engine)"
       namespace="$(arg namespace)" />
   </xacro:if>
@@ -92,7 +79,4 @@
       xyz="${lidar_xyz}"
       rpy="${lidar_rpy}"
-      use_gpu="${lidar_use_gpu}"
-      simulation_engine="$(arg simulation_engine)"
-      topic="velodyne_points"
       namespace="$(arg namespace)" />
   </xacro:if>
@@ -113,5 +97,4 @@
       rpy="${camera_rpy}"
       use_nominal_extrinsics="$(arg use_sim)"
-      simulation_engine="$(arg simulation_engine)"
       namespace="$(arg namespace)" />
   </xacro:if>
@@ -124,5 +107,4 @@
       xyz="${camera_xyz}"
       rpy="${camera_rpy}"
-      simulation_engine="$(arg simulation_engine)"
       namespace="$(arg namespace)" />
   </xacro:if>
@@ -154,5 +136,4 @@
       rpy="${camera_rpy}"
       model="${camera_model_type}"
-      simulation_engine="$(arg simulation_engine)"
       namespace="$(arg namespace)" />
   </xacro:if>
