Commit message: Add controller_config_path arg

File: rosbot_xl_description/urdf/rosbot_xl.urdf.xacro (robot description, xacro)
@@ -8,18 +8,20 @@
   <xacro:arg name="simulation_engine" default="ignition-gazebo" />
   <xacro:arg name="namespace" default="None" />
+  <xacro:arg name="controller_config_file" default="$(find rosbot_xl_controller)/config/diff_drive_controller.yaml" />
   <xacro:include filename="$(find rosbot_xl_description)/urdf/rosbot_xl_macro.urdf.xacro"
     ns="husarion" />
   <xacro:husarion.rosbot_xl_robot
-    use_sim="$(arg use_sim)"
+    controller_config_file="$(arg controller_config_file)"
     mecanum="$(arg mecanum)"
+    namespace="$(arg namespace)"
     simulation_engine="$(arg simulation_engine)"
-    namespace="$(arg namespace)" />
+    use_sim="$(arg use_sim)" />
   <xacro:include filename="$(find rosbot_xl_description)/urdf/components/antenna.urdf.xacro"
     ns="antenna" />
   <xacro:antenna.antenna
-  parent_link="body_link"
-  xyz="-0.155 -0.055 0.065"
-  rpy="0.0 0.0 0.0"
-  antenna_angle="0.0" />
+    parent_link="body_link"
+    xyz="-0.155 -0.055 0.065"
+    rpy="0.0 0.0 0.0"
+    antenna_angle="0.0" />
   <!-- INCLUDE LIDAR -->
   <xacro:property name="lidar_model" value="$(arg lidar_model)" />
@@ -33,6 +35,5 @@
       parent_link="${lidar_parent_link}"
       xyz="${lidar_xyz}"
-      rpy="${lidar_rpy}"
-      namespace="$(arg namespace)" />
+      rpy="${lidar_rpy}" />
   </xacro:if>
   <xacro:if value="${lidar_model == 'slamtec_rplidar_s2'}">
@@ -42,6 +43,5 @@
       parent_link="${lidar_parent_link}"
       xyz="${lidar_xyz}"
-      rpy="${lidar_rpy}"
-      namespace="$(arg namespace)" />
+      rpy="${lidar_rpy}" />
   </xacro:if>
   <xacro:if value="${lidar_model == 'slamtec_rplidar_s3'}">
@@ -51,6 +51,5 @@
       parent_link="${lidar_parent_link}"
       xyz="${lidar_xyz}"
-      rpy="${lidar_rpy}"
-      namespace="$(arg namespace)" />
+      rpy="${lidar_rpy}" />
   </xacro:if>
   <xacro:if value="${lidar_model == 'slamtec_rplidar_a2'}">
@@ -60,6 +59,5 @@
       parent_link="${lidar_parent_link}"
       xyz="${lidar_xyz}"
-      rpy="${lidar_rpy}"
-      namespace="$(arg namespace)" />
+      rpy="${lidar_rpy}" />
   </xacro:if>
   <xacro:if value="${lidar_model == 'slamtec_rplidar_a3'}">
@@ -69,6 +67,5 @@
       parent_link="${lidar_parent_link}"
       xyz="${lidar_xyz}"
-      rpy="${lidar_rpy}"
-      namespace="$(arg namespace)" />
+      rpy="${lidar_rpy}" />
   </xacro:if>
   <xacro:if value="${lidar_model == 'velodyne_puck'}">
@@ -78,6 +75,5 @@
       parent_link="${lidar_parent_link}"
       xyz="${lidar_xyz}"
-      rpy="${lidar_rpy}"
-      namespace="$(arg namespace)" />
+      rpy="${lidar_rpy}" />
   </xacro:if>
   <!-- INCLUDE CAMERA -->
@@ -96,6 +92,5 @@
       xyz="${camera_xyz}"
       rpy="${camera_rpy}"
-      use_nominal_extrinsics="$(arg use_sim)"
-      namespace="$(arg namespace)" />
+      use_nominal_extrinsics="$(arg use_sim)" />
   </xacro:if>
   <xacro:if value="${camera_model == 'orbbec_astra'}">
@@ -106,6 +101,5 @@
       parent_link="${camera_parent_link}"
       xyz="${camera_xyz}"
-      rpy="${camera_rpy}"
-      namespace="$(arg namespace)" />
+      rpy="${camera_rpy}" />
   </xacro:if>
   <xacro:if value="${camera_model.startswith('stereolabs')}">
@@ -135,6 +129,5 @@
       xyz="${camera_xyz}"
       rpy="${camera_rpy}"
-      model="${camera_model_type}"
-      namespace="$(arg namespace)" />
+      model="${camera_model_type}" />
   </xacro:if>
   <!-- INCLUDE CAMERA MOUNT - add if camera_model is not empty -->

File: rosbot_xl_description/urdf/rosbot_xl_macro.urdf.xacro (robot description, xacro)
@@ -2,12 +2,14 @@
 <robot xmlns:xacro="http://wiki.ros.org/xacro">
   <xacro:macro name="rosbot_xl_robot"
-    params="use_sim mecanum simulation_engine namespace">
+    params="controller_config_file
+            mecanum
+            namespace
+            simulation_engine
+            use_sim">
     <xacro:if value="${namespace == 'None'}">
       <xacro:property name="ns" value="" />
-      <xacro:property name="gz_control_namespace" value="/" />
     </xacro:if>
     <xacro:unless value="${namespace == 'None'}">
-        <xacro:property name="ns" value="${namespace}/" />
-        <xacro:property name="gz_control_namespace" value="${namespace}" />
+      <xacro:property name="ns" value="${namespace}/" />
     </xacro:unless>
     <xacro:if value="${mecanum}">
@@ -19,4 +21,6 @@
     <!-- INCLUDE ROBOT PARTS DEFINITIONS -->
     <xacro:include filename="$(find rosbot_xl_description)/urdf/body.urdf.xacro" ns="body" />
+    <xacro:include filename="$(find rosbot_xl_description)/urdf/gazebo.urdf.xacro" ns="gazebo" />
+    <xacro:include filename="$(find rosbot_xl_description)/urdf/webots.urdf.xacro" ns="webots" />
     <xacro:include filename="$(find rosbot_xl_description)/urdf/wheel.urdf.xacro" ns="wheel" />
     <!-- BODY DECLARATION -->
@@ -115,47 +119,9 @@
     <xacro:if value="${use_sim}">
       <xacro:if value="${simulation_engine == 'ignition-gazebo'}">
-        <gazebo>
-          <plugin filename="ign_ros2_control-system" name="ign_ros2_control::IgnitionROS2ControlPlugin">
-            <xacro:if value="${mecanum}">
-              <parameters>$(find rosbot_xl_controller)/config/mecanum_drive_controller.yaml</parameters>
-            </xacro:if>
-            <xacro:unless value="${mecanum}">
-              <parameters>$(find rosbot_xl_controller)/config/diff_drive_controller.yaml</parameters>
-            </xacro:unless>
-            <ros>
-              <namespace>${gz_control_namespace}</namespace>
-              <remapping>rosbot_xl_base_controller/cmd_vel_unstamped:=cmd_vel</remapping>
-              <remapping>/tf:=tf</remapping>
-            </ros>
-          </plugin>
-        </gazebo>
-        <gazebo reference="imu_link">
-          <sensor name="${ns}imu" type="imu">
-            <always_on>true</always_on>
-            <update_rate>25</update_rate>
-            <topic>${ns}imu/data_raw</topic>
-            <visualize>false</visualize>
-            <enable_metrics>false</enable_metrics>
-            <frame_id>imu_link</frame_id>
-            <ignition_frame_id>imu_link</ignition_frame_id>
-            <ros>
-              <namespace>${ns}</namespace>
-            </ros>
-          </sensor>
-        </gazebo>
+        <xacro:gazebo.controller config_file="${controller_config_file}" namespace="${namespace}" />
+        <xacro:gazebo.imu reference_frame="imu_link" namespace="${namespace}" />
       </xacro:if>
       <xacro:if value="${simulation_engine == 'webots'}">
-        <webots>
-          <plugin type="webots_ros2_control::Ros2Control" />
-          <plugin type="webots_ros2_driver::Ros2IMU">
-            <enabled>true</enabled>
-            <topicName>/imu_broadcaster/imu</topicName>
-            <alwaysOn>true</alwaysOn>
-            <frameName>imu_link</frameName>
-            <gyroName>imu gyro</gyroName>
-            <accelerometerName>imu accelerometer</accelerometerName>
-            <inertialUnitName>imu inertial_unit</inertialUnitName>
-          </plugin>
-        </webots>
+        <xacro:webots.controller />
       </xacro:if>
     </xacro:if>
