Commit message: Changes in description package

File: rosbot_xl_description/urdf/rosbot_xl.urdf.xacro (robot description, xacro)
@@ -6,8 +6,7 @@
   <xacro:arg name="include_camera_mount" default="false" />
   <xacro:arg name="use_sim" default="false" />
-  <xacro:arg name="simulation_engine" default="ignition-gazebo" />
   <xacro:arg name="namespace" default="None" />
   <xacro:arg name="controller_config_file" default="$(find rosbot_xl_controller)/config/diff_drive_controller.yaml" />
-  <xacro:include filename="$(find rosbot_xl_description)/urdf/rosbot_xl_macro.urdf.xacro"
+  <xacro:include filename="$(find rosbot_xl_description)/urdf/rosbot_xl/rosbot_xl_macro.urdf.xacro"
     ns="husarion" />
   <xacro:husarion.rosbot_xl_robot
@@ -15,7 +14,6 @@
     mecanum="$(arg mecanum)"
     namespace="$(arg namespace)"
-    simulation_engine="$(arg simulation_engine)"
     use_sim="$(arg use_sim)" />
-  <xacro:include filename="$(find rosbot_xl_description)/urdf/components/antenna.urdf.xacro"
+  <xacro:include filename="$(find rosbot_xl_description)/urdf/rosbot_xl/components/antenna.urdf.xacro"
     ns="antenna" />
   <xacro:antenna.antenna
@@ -29,43 +27,27 @@
   <xacro:property name="lidar_xyz" value="0.02 0.0 0.0" />
   <xacro:property name="lidar_rpy" value="0.0 0.0 0.0" />
-  <xacro:if value="${lidar_model == 'slamtec_rplidar_s1'}">
-    <xacro:include filename="$(find ros_components_description)/urdf/slamtec_rplidar_s1.urdf.xacro"
+  <xacro:if value="${lidar_model.startswith('stereolabs')}">
+    <xacro:if value="${lidar_model == 'slamtec_rplidar_s1'}">
+      <xacro:property name="lidar_model_type" value="s1" />
+    </xacro:if>
+    <xacro:if value="${lidar_model == 'slamtec_rplidar_s2'}">
+      <xacro:property name="lidar_model_type" value="s2" />
+    </xacro:if>
+    <xacro:if value="${lidar_model == 'slamtec_rplidar_s3'}">
+      <xacro:property name="lidar_model_type" value="s3" />
+    </xacro:if>
+    <xacro:if value="${lidar_model == 'slamtec_rplidar_a2'}">
+      <xacro:property name="lidar_model_type" value="a2" />
+    </xacro:if>
+    <xacro:if value="${lidar_model == 'slamtec_rplidar_a3'}">
+      <xacro:property name="lidar_model_type" value="a3" />
+    </xacro:if>
+    <xacro:include filename="$(find ros_components_description)/urdf/slamtec_rplidar.urdf.xacro"
       ns="lidar" />
-    <xacro:lidar.slamtec_rplidar_s1
+    <xacro:lidar.slamtec_rplidar
       parent_link="${lidar_parent_link}"
       xyz="${lidar_xyz}"
-      rpy="${lidar_rpy}" />
-  </xacro:if>
-  <xacro:if value="${lidar_model == 'slamtec_rplidar_s2'}">
-    <xacro:include filename="$(find ros_components_description)/urdf/slamtec_rplidar_s2.urdf.xacro"
-      ns="lidar" />
-    <xacro:lidar.slamtec_rplidar_s2
-      parent_link="${lidar_parent_link}"
-      xyz="${lidar_xyz}"
-      rpy="${lidar_rpy}" />
-  </xacro:if>
-  <xacro:if value="${lidar_model == 'slamtec_rplidar_s3'}">
-    <xacro:include filename="$(find ros_components_description)/urdf/slamtec_rplidar_s3.urdf.xacro"
-      ns="lidar" />
-    <xacro:lidar.slamtec_rplidar_s3
-      parent_link="${lidar_parent_link}"
-      xyz="${lidar_xyz}"
-      rpy="${lidar_rpy}" />
-  </xacro:if>
-  <xacro:if value="${lidar_model == 'slamtec_rplidar_a2'}">
-    <xacro:include filename="$(find ros_components_description)/urdf/slamtec_rplidar_a2.urdf.xacro"
-      ns="lidar" />
-    <xacro:lidar.slamtec_rplidar_a2
-      parent_link="${lidar_parent_link}"
-      xyz="${lidar_xyz}"
-      rpy="${lidar_rpy}" />
-  </xacro:if>
-  <xacro:if value="${lidar_model == 'slamtec_rplidar_a3'}">
-    <xacro:include filename="$(find ros_components_description)/urdf/slamtec_rplidar_a3.urdf.xacro"
-      ns="lidar" />
-    <xacro:lidar.slamtec_rplidar_a3
-      parent_link="${lidar_parent_link}"
-      xyz="${lidar_xyz}"
-      rpy="${lidar_rpy}" />
+      rpy="${lidar_rpy}"
+      model="${lidar_model_type}" />
   </xacro:if>
   <xacro:if value="${lidar_model == 'velodyne_puck'}">
@@ -134,5 +116,5 @@
   <xacro:property name="include_camera_mount" value="$(arg include_camera_mount)" />
   <xacro:if value="${include_camera_mount or camera_model != 'None'}">
-    <xacro:include filename="$(find rosbot_xl_description)/urdf/components/camera_mount.urdf.xacro"
+    <xacro:include filename="$(find rosbot_xl_description)/urdf/rosbot_xl/components/camera_mount.urdf.xacro"
       ns="camera_mount" />
     <xacro:camera_mount.camera_mount

File: rosbot_xl_description/urdf/rosbot_xl/body.urdf.xacro (robot description, xacro)
@@ -11,5 +11,5 @@
       <visual>
         <geometry>
-          <mesh filename="package://rosbot_xl_description/meshes/body.dae" scale="1 1 1" />
+          <mesh filename="package://rosbot_xl_description/meshes/rosbot_xl/body.dae" scale="1 1 1" />
         </geometry>
         <origin xyz="0.0 0.0 0.0" rpy="0.0 0.0 0.0" />
@@ -17,5 +17,5 @@
       <collision>
         <geometry>
-          <mesh filename="package://rosbot_xl_description/meshes/body_colision.stl" scale="1 1 1" />
+          <mesh filename="package://rosbot_xl_description/meshes/rosbot_xl/body_colision.stl" scale="1 1 1" />
         </geometry>
         <origin xyz="0.0 0.0 0.0" rpy="0.0 0.0 0.0" />

File: rosbot_xl_description/urdf/rosbot_xl/components/antenna.urdf.xacro (robot description, xacro)
@@ -21,5 +21,5 @@
       <visual>
         <geometry>
-          <mesh filename="package://rosbot_xl_description/meshes/components/antenna_connector.dae"
+          <mesh filename="package://rosbot_xl_description/meshes/rosbot_xl/components/antenna_connector.dae"
             scale="1 1 1" />
         </geometry>
@@ -35,5 +35,5 @@
       <visual>
         <geometry>
-          <mesh filename="package://rosbot_xl_description/meshes/components/antenna.dae"
+          <mesh filename="package://rosbot_xl_description/meshes/rosbot_xl/components/antenna.dae"
             scale="1 1 1" />
         </geometry>

File: rosbot_xl_description/urdf/rosbot_xl/components/camera_mount.urdf.xacro (robot description, xacro)
@@ -21,5 +21,5 @@
       <visual>
         <geometry>
-          <mesh filename="package://rosbot_xl_description/meshes/components/camera_mount_bot.dae"
+          <mesh filename="package://rosbot_xl_description/meshes/rosbot_xl/components/camera_mount_bot.dae"
       scale="1 1 1" />
         </geometry>
@@ -42,5 +42,5 @@
       <visual>
         <geometry>
-          <mesh filename="package://rosbot_xl_description/meshes/components/camera_mount_mid.dae"
+          <mesh filename="package://rosbot_xl_description/meshes/rosbot_xl/components/camera_mount_mid.dae"
       scale="1 1 1" />
         </geometry>
@@ -63,5 +63,5 @@
       <visual>
         <geometry>
-          <mesh filename="package://rosbot_xl_description/meshes/components/camera_mount_top.dae"
+          <mesh filename="package://rosbot_xl_description/meshes/rosbot_xl/components/camera_mount_top.dae"
       scale="1 1 1" />
         </geometry>

File: rosbot_xl_description/urdf/rosbot_xl/gazebo.urdf.xacro (robot description, xacro)
@@ -6,9 +6,9 @@
     </xacro:if>
     <gazebo>
-      <plugin filename="ign_ros2_control-system" name="ign_ros2_control::IgnitionROS2ControlPlugin">
+      <plugin filename="gz_ros2_control-system" name="gz_ros2_control::GazeboSimROS2ControlPlugin">
         <parameters>${config_file}</parameters>
         <ros>
           <namespace>${namespace}</namespace>
-          <remapping>rosbot_base_controller/cmd_vel_unstamped:=cmd_vel</remapping>
+          <remapping>rosbot_base_controller/cmd_vel:=cmd_vel</remapping>
           <remapping>/tf:=tf</remapping>
         </ros>

File: rosbot_xl_description/urdf/rosbot_xl/rosbot_xl_macro.urdf.xacro (robot description, xacro)
@@ -5,5 +5,4 @@
             mecanum
             namespace
-            simulation_engine
             use_sim">
     <xacro:if value="${namespace == 'None'}">
@@ -20,19 +19,16 @@
     </xacro:unless>
     <!-- INCLUDE ROBOT PARTS DEFINITIONS -->
-    <xacro:include filename="$(find rosbot_xl_description)/urdf/body.urdf.xacro" ns="body" />
-    <xacro:include filename="$(find rosbot_xl_description)/urdf/gazebo.urdf.xacro" ns="gazebo" />
-    <xacro:include filename="$(find rosbot_xl_description)/urdf/webots.urdf.xacro" ns="webots" />
-    <xacro:include filename="$(find rosbot_xl_description)/urdf/wheel.urdf.xacro" ns="wheel" />
+    <xacro:include filename="$(find rosbot_xl_description)/urdf/rosbot_xl/body.urdf.xacro" ns="body" />
+    <xacro:include filename="$(find rosbot_xl_description)/urdf/rosbot_xl/gazebo.urdf.xacro" ns="gazebo" />
+    <xacro:include filename="$(find rosbot_xl_description)/urdf/rosbot_xl/webots.urdf.xacro" ns="webots" />
+    <xacro:include filename="$(find rosbot_xl_description)/urdf/rosbot_xl/wheel.urdf.xacro" ns="wheel" />
+/rosbot_xl
     <!-- BODY DECLARATION -->
     <xacro:body.body wheel_radius="${wheel_radius}" />
     <!-- WHEEL DECLARATION -->
-    <xacro:wheel.wheel wheel_radius="${wheel_radius}" side="fl" mecanum="${mecanum}"
-      use_sim="$(arg use_sim)" />
-    <xacro:wheel.wheel wheel_radius="${wheel_radius}" side="fr" mecanum="${mecanum}"
-      use_sim="$(arg use_sim)" />
-    <xacro:wheel.wheel wheel_radius="${wheel_radius}" side="rl" mecanum="${mecanum}"
-      use_sim="$(arg use_sim)" />
-    <xacro:wheel.wheel wheel_radius="${wheel_radius}" side="rr" mecanum="${mecanum}"
-      use_sim="$(arg use_sim)" />
+    <xacro:wheel.wheel wheel_radius="${wheel_radius}" side="fl" mecanum="${mecanum}" />
+    <xacro:wheel.wheel wheel_radius="${wheel_radius}" side="fr" mecanum="${mecanum}" />
+    <xacro:wheel.wheel wheel_radius="${wheel_radius}" side="rl" mecanum="${mecanum}" />
+    <xacro:wheel.wheel wheel_radius="${wheel_radius}" side="rr" mecanum="${mecanum}" />
     <!-- ROS2 CONTROL -->
     <xacro:unless value="$(arg use_sim)">
@@ -60,10 +56,5 @@
       <hardware>
         <xacro:if value="${use_sim}">
-          <xacro:if value="${simulation_engine == 'ignition-gazebo'}">
-            <plugin>ign_ros2_control/IgnitionSystem</plugin>
-          </xacro:if>
-          <xacro:if value="${simulation_engine == 'webots'}">
-            <plugin>webots_ros2_control::Ros2ControlSystem</plugin>
-          </xacro:if>
+          <plugin>gz_ros2_control/GazeboSimSystem</plugin>
         </xacro:if>
         <xacro:unless value="$(arg use_sim)">
@@ -101,28 +92,21 @@
       </joint>
       <xacro:if value="${use_sim}">
-        <xacro:if value="${simulation_engine == 'ignition-gazebo'}">
-          <sensor name="${ns}imu">
-            <state_interface name="orientation.x" />
-            <state_interface name="orientation.y" />
-            <state_interface name="orientation.z" />
-            <state_interface name="orientation.w" />
-            <state_interface name="angular_velocity.x" />
-            <state_interface name="angular_velocity.y" />
-            <state_interface name="angular_velocity.z" />
-            <state_interface name="linear_acceleration.x" />
-            <state_interface name="linear_acceleration.y" />
-            <state_interface name="linear_acceleration.z" />
-          </sensor>
-        </xacro:if>
+        <sensor name="${ns}imu">
+          <state_interface name="orientation.x" />
+          <state_interface name="orientation.y" />
+          <state_interface name="orientation.z" />
+          <state_interface name="orientation.w" />
+          <state_interface name="angular_velocity.x" />
+          <state_interface name="angular_velocity.y" />
+          <state_interface name="angular_velocity.z" />
+          <state_interface name="linear_acceleration.x" />
+          <state_interface name="linear_acceleration.y" />
+          <state_interface name="linear_acceleration.z" />
+        </sensor>
       </xacro:if>
     </ros2_control>
     <xacro:if value="${use_sim}">
-      <xacro:if value="${simulation_engine == 'ignition-gazebo'}">
-        <xacro:gazebo.controller config_file="${controller_config_file}" namespace="${namespace}" />
-        <xacro:gazebo.imu reference_frame="imu_link" namespace="${namespace}" />
-      </xacro:if>
-      <xacro:if value="${simulation_engine == 'webots'}">
-        <xacro:webots.controller />
-      </xacro:if>
+      <xacro:gazebo.controller config_file="${controller_config_file}" namespace="${namespace}" />
+      <xacro:gazebo.imu reference_frame="imu_link" namespace="${namespace}" />
     </xacro:if>
   </xacro:macro>

File: rosbot_xl_description/urdf/rosbot_xl/wheel.urdf.xacro (robot description, xacro)
@@ -1,5 +1,5 @@
 <?xml version="1.0" encoding="utf-8"?>
 <robot xmlns:xacro="http://www.ros.org/wiki/xacro">
-  <xacro:macro name="wheel" params="wheel_radius side mecanum use_sim">
+  <xacro:macro name="wheel" params="wheel_radius side mecanum">
     <xacro:property name="wheel_separation_x" value="0.170" />
     <xacro:if value="${mecanum}">
@@ -24,5 +24,5 @@
       <xacro:property name="x" value="${wheel_separation_x/2}" />
       <xacro:property name="y" value="${wheel_separation_y/2}" />
-      <xacro:property name="mesh" value="package://rosbot_xl_description/meshes/${wheel_file}_b.dae" />
+      <xacro:property name="mesh" value="package://rosbot_xl_description/meshes/rosbot_xl/${wheel_file}_b.dae" />
       <xacro:property name="visual_rotation" value="${pi}" />
       <xacro:property name="fdir" value="1 -1 0" />
@@ -31,5 +31,5 @@
       <xacro:property name="x" value="${wheel_separation_x/2}" />
       <xacro:property name="y" value="${-wheel_separation_y/2}" />
-      <xacro:property name="mesh" value="package://rosbot_xl_description/meshes/${wheel_file}_a.dae" />
+      <xacro:property name="mesh" value="package://rosbot_xl_description/meshes/rosbot_xl/${wheel_file}_a.dae" />
       <xacro:property name="visual_rotation" value="${pi}" />
       <xacro:property name="fdir" value="1 1 0" />
@@ -38,5 +38,5 @@
       <xacro:property name="x" value="${-wheel_separation_x/2}" />
       <xacro:property name="y" value="${wheel_separation_y/2}" />
-      <xacro:property name="mesh" value="package://rosbot_xl_description/meshes/${wheel_file}_a.dae" />
+      <xacro:property name="mesh" value="package://rosbot_xl_description/meshes/rosbot_xl/${wheel_file}_a.dae" />
       <xacro:property name="visual_rotation" value="${0.0}" />
       <xacro:property name="fdir" value="1 1 0" />
@@ -45,5 +45,5 @@
       <xacro:property name="x" value="${-wheel_separation_x/2}" />
       <xacro:property name="y" value="${-wheel_separation_y/2}" />
-      <xacro:property name="mesh" value="package://rosbot_xl_description/meshes/${wheel_file}_b.dae" />
+      <xacro:property name="mesh" value="package://rosbot_xl_description/meshes/rosbot_xl/${wheel_file}_b.dae" />
       <xacro:property name="visual_rotation" value="${0.0}" />
       <xacro:property name="fdir" value="1 -1 0" />
@@ -77,19 +77,36 @@
       </inertial>
     </link>
-    <xacro:if value="${use_sim}">
-      <gazebo reference="${side}_wheel_link" xmlns:ignition="http://ignitionrobotics.org/schema">
+    <gazebo reference="${side}_wheel_link" xmlns:gz="http://gazeborobotics.org/schema">
+      <xacro:unless value="${mecanum}">
         <collision>
           <surface>
             <friction>
               <ode>
-                <mu>1.0</mu>
-                <mu2>0.0</mu2>
-                <fdir1 ignition:expressed_in="base_link">${fdir}</fdir1>
+                <mu>1</mu>
+                <mu2>1</mu2>
+                <slip1>0.035</slip1>
+                <slip2>0</slip2>
+                <fdir1>0 0 1</fdir1>
               </ode>
             </friction>
           </surface>
         </collision>
-      </gazebo>
-    </xacro:if>
+      </xacro:unless>
+      <xacro:if value="${mecanum}">
+        <collision>
+          <surface>
+            <friction>
+              <ode>
+                <mu>0.8</mu>
+                <mu2>0.2</mu2>
+                  <slip1>0.035</slip1>
+                <slip2>0</slip2>
+                <fdir1 gz:expressed_in="base_link">${fdir}</fdir1>
+              </ode>
+            </friction>
+          </surface>
+        </collision>
+      </xacro:if>
+    </gazebo>
   </xacro:macro>
 </robot>

Commit message: remove comaera lidar arg

File: rosbot_xl_description/urdf/rosbot_xl.urdf.xacro (robot description, xacro)
@@ -2,7 +2,4 @@
 <robot name="rosbot_xl" xmlns:xacro="http://www.ros.org/wiki/xacro">
   <xacro:arg name="mecanum" default="false" />
-  <xacro:arg name="lidar_model" default="slamtec_rplidar_s1" />
-  <xacro:arg name="camera_model" default="intel_realsense_d435" />
-  <xacro:arg name="include_camera_mount" default="false" />
   <xacro:arg name="use_sim" default="false" />
   <xacro:arg name="namespace" default="None" />
@@ -22,98 +19,9 @@
     rpy="0.0 0.0 0.0"
     antenna_angle="0.0" />
-  <!-- INCLUDE LIDAR -->
-  <xacro:property name="lidar_model" value="$(arg lidar_model)" />
-  <xacro:property name="lidar_parent_link" value="cover_link" />
-  <xacro:property name="lidar_xyz" value="0.02 0.0 0.0" />
-  <xacro:property name="lidar_rpy" value="0.0 0.0 0.0" />
-  <xacro:if value="${lidar_model.startswith('stereolabs')}">
-    <xacro:if value="${lidar_model == 'slamtec_rplidar_s1'}">
-      <xacro:property name="lidar_model_type" value="s1" />
-    </xacro:if>
-    <xacro:if value="${lidar_model == 'slamtec_rplidar_s2'}">
-      <xacro:property name="lidar_model_type" value="s2" />
-    </xacro:if>
-    <xacro:if value="${lidar_model == 'slamtec_rplidar_s3'}">
-      <xacro:property name="lidar_model_type" value="s3" />
-    </xacro:if>
-    <xacro:if value="${lidar_model == 'slamtec_rplidar_a2'}">
-      <xacro:property name="lidar_model_type" value="a2" />
-    </xacro:if>
-    <xacro:if value="${lidar_model == 'slamtec_rplidar_a3'}">
-      <xacro:property name="lidar_model_type" value="a3" />
-    </xacro:if>
-    <xacro:include filename="$(find ros_components_description)/urdf/slamtec_rplidar.urdf.xacro"
-      ns="lidar" />
-    <xacro:lidar.slamtec_rplidar
-      parent_link="${lidar_parent_link}"
-      xyz="${lidar_xyz}"
-      rpy="${lidar_rpy}"
-      model="${lidar_model_type}" />
-  </xacro:if>
-  <xacro:if value="${lidar_model == 'velodyne_puck'}">
-    <xacro:include filename="$(find ros_components_description)/urdf/velodyne_puck.urdf.xacro"
-      ns="lidar" />
-    <xacro:lidar.velodyne_puck
-      parent_link="${lidar_parent_link}"
-      xyz="${lidar_xyz}"
-      rpy="${lidar_rpy}" />
-  </xacro:if>
-  <!-- INCLUDE CAMERA -->
-  <xacro:property name="camera_model" value="$(arg camera_model)" />
   <xacro:property name="camera_parent_link" value="camera_mount_link" />
   <xacro:property name="camera_xyz" value="0.0 0.0 0.0" />
   <xacro:property name="camera_rpy" value="0.0 0.0 0.0" />
-  <!-- nominal_extrinsics should be used only in simulation, when using real camera it should publish
-    calibrated ones -->
-  <xacro:if value="${camera_model == 'intel_realsense_d435'}">
-    <xacro:include
-      filename="$(find ros_components_description)/urdf/intel_realsense_d435.urdf.xacro"
-      ns="camera" />
-    <xacro:camera.intel_realsense_d435
-      parent_link="${camera_parent_link}"
-      xyz="${camera_xyz}"
-      rpy="${camera_rpy}"
-      use_nominal_extrinsics="$(arg use_sim)" />
-  </xacro:if>
-  <xacro:if value="${camera_model == 'orbbec_astra'}">
-    <xacro:include
-      filename="$(find ros_components_description)/urdf/orbbec_astra.urdf.xacro"
-      ns="camera" />
-    <xacro:camera.orbbec_astra
-      parent_link="${camera_parent_link}"
-      xyz="${camera_xyz}"
-      rpy="${camera_rpy}" />
-  </xacro:if>
-  <xacro:if value="${camera_model.startswith('stereolabs')}">
-    <xacro:if value="${camera_model == 'stereolabs_zed'}">
-      <xacro:property name="camera_model_type" value="zed" />
-    </xacro:if>
-    <xacro:if value="${camera_model == 'stereolabs_zedm'}">
-      <xacro:property name="camera_model_type" value="zedm" />
-    </xacro:if>
-    <xacro:if value="${camera_model == 'stereolabs_zed2'}">
-      <xacro:property name="camera_model_type" value="zed2" />
-    </xacro:if>
-    <xacro:if value="${camera_model == 'stereolabs_zed2i'}">
-      <xacro:property name="camera_model_type" value="zed2i" />
-    </xacro:if>
-    <xacro:if value="${camera_model == 'stereolabs_zedx'}">
-      <xacro:property name="camera_model_type" value="zedx" />
-    </xacro:if>
-    <xacro:if value="${camera_model == 'stereolabs_zedxm'}">
-      <xacro:property name="camera_model_type" value="zedxm" />
-    </xacro:if>
-    <xacro:include
-    filename="$(find ros_components_description)/urdf/stereolabs_zed.urdf.xacro"
-    ns="camera" />
-    <xacro:camera.zed_camera
-      parent_link="${camera_parent_link}"
-      xyz="${camera_xyz}"
-      rpy="${camera_rpy}"
-      model="${camera_model_type}" />
-  </xacro:if>
-  <!-- INCLUDE CAMERA MOUNT - add if camera_model is not empty -->
   <xacro:property name="include_camera_mount" value="$(arg include_camera_mount)" />
-  <xacro:if value="${include_camera_mount or camera_model != 'None'}">
+  <!-- TODO <xacro:if value="${include_camera_mount or camera_model != 'None'}"> -->
     <xacro:include filename="$(find rosbot_xl_description)/urdf/rosbot_xl/components/camera_mount.urdf.xacro"
       ns="camera_mount" />
@@ -124,4 +32,4 @@
       camera_mount_angle_1="0.0"
       camera_mount_angle_2="0.0" />
-  </xacro:if>
+  <!-- </xacro:if> -->
 </robot>
