Commit message: fix

File: rosbot_xl_description/urdf/rosbot_xl.urdf.xacro (robot description, xacro)
@@ -1,6 +1,6 @@
 <?xml version='1.0'?>
 <robot name="rosbot_xl" xmlns:xacro="http://www.ros.org/wiki/xacro">
-  <xacro:arg name="components_config_path" default="$(find husarion_ugv_description)/config/components.yaml" />
-  <xacro:arg name="controller_config_file" default="$(find rosbot_xl_controller)/config/diff_drive_controller.yaml" />
+  <xacro:arg name="components_config" default="$(find rosbot_xl_description)/config/components.yaml" />
+  <xacro:arg name="controller_config" default="$(find rosbot_xl_controller)/config/diff_drive_controller.yaml" />
   <xacro:arg name="mecanum" default="false" />
   <xacro:arg name="namespace" default="" />
@@ -9,5 +9,5 @@
     ns="husarion" />
   <xacro:husarion.rosbot_xl_robot
-    controller_config_file="$(arg controller_config_file)"
+    controller_config="$(arg controller_config)"
     mecanum="$(arg mecanum)"
     namespace="$(arg namespace)"
@@ -24,10 +24,10 @@
       camera_mount_angle_2="0.0" />
   <!-- </xacro:if> -->
-  <xacro:property name="components_config_path_property" value="$(arg components_config_path)" />
-  <xacro:unless value="${components_config_path_property == 'None'}">
+  <xacro:property name="components_config_property" value="$(arg components_config)" />
+  <xacro:unless value="${components_config_property == 'None'}">
     <xacro:include filename="$(find ros_components_description)/urdf/components.urdf.xacro"
       ns="husarion_components" />
     <xacro:husarion_components.create_components
-      components_config_path="${components_config_path_property}"
+      components_config="${components_config_property}"
       namespace="$(arg namespace)"
     />

File: rosbot_xl_description/urdf/rosbot_xl/rosbot_xl_macro.urdf.xacro (robot description, xacro)
@@ -2,12 +2,12 @@
 <robot xmlns:xacro="http://wiki.ros.org/xacro">
   <xacro:macro name="rosbot_xl_robot"
-    params="controller_config_file
+    params="controller_config
             mecanum
             namespace
             use_sim">
-    <xacro:if value="${namespace == 'None'}">
+    <xacro:if value="${namespace == ''}">
       <xacro:property name="ns" value="" />
     </xacro:if>
-    <xacro:unless value="${namespace == 'None'}">
+    <xacro:unless value="${namespace == ''}">
       <xacro:property name="ns" value="${namespace}/" />
     </xacro:unless>
@@ -109,5 +109,5 @@
     </ros2_control>
     <xacro:if value="${use_sim}">
-      <xacro:gazebo.controller config_file="${controller_config_file}" namespace="${namespace}" />
+      <xacro:gazebo.controller config_file="${controller_config}" namespace="${namespace}" />
       <xacro:gazebo.imu reference_frame="imu_link" namespace="${namespace}" />
     </xacro:if>

Commit message: Fix components

File: rosbot_xl_description/urdf/rosbot_xl.urdf.xacro (robot description, xacro)
@@ -3,4 +3,5 @@
   <xacro:arg name="components_config" default="$(find rosbot_xl_description)/config/components.yaml" />
   <xacro:arg name="controller_config" default="$(find rosbot_xl_controller)/config/diff_drive_controller.yaml" />
+  <xacro:arg name="include_camera_mount" default="false" />
   <xacro:arg name="mecanum" default="false" />
   <xacro:arg name="namespace" default="" />
@@ -13,8 +14,6 @@
     namespace="$(arg namespace)"
     use_sim="$(arg use_sim)" />
-  <xacro:property name="include_camera_mount" value="$(arg include_camera_mount)" />
-  <!-- TODO <xacro:if value="${include_camera_mount or camera_model != 'None'}"> -->
-    <xacro:include filename="$(find rosbot_xl_description)/urdf/rosbot_xl/components/camera_mount.urdf.xacro"
-      ns="camera_mount" />
+  <xacro:if value="$(arg include_camera_mount)">
+    <xacro:include filename="$(find rosbot_xl_description)/urdf/rosbot_xl/components/camera_mount.urdf.xacro" ns="camera_mount" />
     <xacro:camera_mount.camera_mount
       parent_link="cover_link"
@@ -23,13 +22,9 @@
       camera_mount_angle_1="0.0"
       camera_mount_angle_2="0.0" />
-  <!-- </xacro:if> -->
-  <xacro:property name="components_config_property" value="$(arg components_config)" />
-  <xacro:unless value="${components_config_property == 'None'}">
-    <xacro:include filename="$(find ros_components_description)/urdf/components.urdf.xacro"
-      ns="husarion_components" />
-    <xacro:husarion_components.create_components
-      components_config="${components_config_property}"
-      namespace="$(arg namespace)"
-    />
-  </xacro:unless>
+  </xacro:if>
+  <xacro:include filename="$(find ros_components_description)/urdf/components.urdf.xacro" ns="components" />
+  <xacro:components.create_components
+    components_config_path="$(arg components_config)"
+    namespace=""
+  />
 </robot>
