Commit message: Fixes

File: rosbot_description/urdf/rosbot/components/vl53lox.urdf.xacro (robot description, xacro)
@@ -3,10 +3,5 @@
   <!-- vl53lox defining macro -->
   <xacro:macro name="vl53lox" params="parent xyz rpy prefix namespace">
-    <xacro:if value="${namespace == 'None'}">
-      <xacro:property name="namespace_ext" value="" />
-    </xacro:if>
-    <xacro:unless value="${namespace == 'None'}">
-        <xacro:property name="namespace_ext" value="${namespace}/" />
-    </xacro:unless>
+    <xacro:property name="ns" value="${namespace + '/' if namespace != '' else ''}" />
     <joint name="${parent}_${prefix}_range_joint" type="fixed">
       <origin xyz="${xyz}" rpy="${rpy}" />
@@ -18,6 +13,6 @@
     https://github.com/gazebosim/gz-sensors/issues/19 -->
     <gazebo reference="${prefix}_range">
-      <sensor name="${namespace_ext}${prefix}_range" type='gpu_lidar'>
-        <topic>${namespace_ext}range/${prefix}</topic>
+      <sensor name="${ns}${prefix}_range" type='gpu_lidar'>
+        <topic>${ns}range/${prefix}</topic>
         <gz_frame_id>${prefix}_range</gz_frame_id>
         <update_rate>5.0</update_rate>

File: rosbot_description/urdf/rosbot/rosbot_macro.urdf.xacro (robot description, xacro)
@@ -2,5 +2,5 @@
 <robot xmlns:xacro="http://wiki.ros.org/xacro">
   <xacro:macro name="rosbot" params="mecanum namespace use_sim">
-    <xacro:property name="ns" value="${namespace + '/' if namespace != 'None' else ''}" />
+    <xacro:property name="ns" value="${namespace + '/' if namespace != '' else ''}" />
     <xacro:property name="wheel_radius" value="${0.0470 if mecanum else 0.0425}" />
     <!-- INCLUDE ROBOT PARTS DEFINITIONS -->
@@ -94,13 +94,11 @@
         <plugin filename="gz_ros2_control-system" name="gz_ros2_control::GazeboSimROS2ControlPlugin">
           <xacro:if value="${mecanum}">
-            <parameters>$(find rosbot_controller)/config/mecanum_drive_controller.yaml</parameters>
+            <parameters>$(find rosbot_controller)/config/rosbot/mecanum_drive_controller.yaml</parameters>
           </xacro:if>
           <xacro:unless value="${mecanum}">
-            <parameters>$(find rosbot_controller)/config/diff_drive_controller.yaml</parameters>
+            <parameters>$(find rosbot_controller)/config/rosbot/diff_drive_controller.yaml</parameters>
           </xacro:unless>
           <ros>
-            <xacro:unless value="${namespace == 'None'}">
-              <namespace>${namespace}</namespace>
-            </xacro:unless>
+            <namespace>${ns}</namespace>
             <remapping>rosbot_base_controller/cmd_vel:=cmd_vel</remapping>
           </ros>

File: rosbot_description/urdf/rosbot_xl.urdf.xacro (robot description, xacro)
@@ -7,5 +7,5 @@
   <xacro:arg name="namespace" default="" />
   <xacro:arg name="use_sim" default="false" />
-  <xacro:include filename="$(find rosbot_description)/urdf/rosbot_xl/rosbot_macro.urdf.xacro"
+  <xacro:include filename="$(find rosbot_description)/urdf/rosbot_xl/rosbot_xl_macro.urdf.xacro"
     ns="husarion" />
   <xacro:husarion.rosbot_robot

File: rosbot_description/urdf/rosbot_xl/gazebo.urdf.xacro (robot description, xacro)
@@ -2,7 +2,4 @@
 <robot xmlns:xacro="http://wiki.ros.org/xacro">
   <xacro:macro name="controller" params="config_file namespace:=''">
-    <xacro:if value="${namespace == 'None'}">
-      <xacro:property name="namespace" value="" />
-    </xacro:if>
     <gazebo>
       <plugin filename="gz_ros2_control-system" name="gz_ros2_control::GazeboSimROS2ControlPlugin">
@@ -29,10 +26,5 @@
   <!-- IMU specification: https://dl.btc.pl/kamami_wa/bst_bno055_ds000_12.pdf -->
   <xacro:macro name="imu" params="reference_frame namespace:=''">
-    <xacro:if value="${namespace == 'None'}">
-      <xacro:property name="ns" value="" />
-    </xacro:if>
-    <xacro:unless value="${namespace == 'None'}">
-        <xacro:property name="ns" value="${namespace}/" />
-    </xacro:unless>
+    <xacro:property name="ns" value="${namespace + '/' if namespace != '' else ''}" />
     <gazebo reference="${reference_frame}">
       <sensor name="${ns}imu" type="imu">
@@ -43,5 +35,5 @@
         <enable_metrics>false</enable_metrics>
         <frame_id>imu_link</frame_id>
-        <ignition_frame_id>imu_link</ignition_frame_id>
+        <gz_frame_id>imu_link</gz_frame_id>
         <imu>
           <angular_velocity>

File: rosbot_description/urdf/rosbot_xl/rosbot_xl_macro.urdf.xacro (robot description, xacro)
@@ -6,16 +6,6 @@
             namespace
             use_sim">
-    <xacro:if value="${namespace == ''}">
-      <xacro:property name="ns" value="" />
-    </xacro:if>
-    <xacro:unless value="${namespace == ''}">
-      <xacro:property name="ns" value="${namespace}/" />
-    </xacro:unless>
-    <xacro:if value="${mecanum}">
-      <xacro:property name="wheel_radius" value="0.05" />
-    </xacro:if>
-    <xacro:unless value="${mecanum}">
-      <xacro:property name="wheel_radius" value="0.048" />
-    </xacro:unless>
+    <xacro:property name="ns" value="${namespace + '/' if namespace != '' else ''}" />
+    <xacro:property name="wheel_radius" value="${0.05 if mecanum else 0.048}" />
     <!-- INCLUDE ROBOT PARTS DEFINITIONS -->
     <xacro:include filename="$(find rosbot_description)/urdf/rosbot_xl/body.urdf.xacro" ns="body" />
@@ -38,6 +28,6 @@
         <hardware>
           <plugin>rosbot_hardware_interfaces/RosbotImuSensor</plugin>
-          <param name="connection_timeout_ms">120000</param>
-          <param name="connection_check_period_ms">500</param>
+          <param name="connection_timeout_ms">30000</param>
+          <param name="connection_check_period_ms">1000</param>
         </hardware>
         <sensor name="${ns}imu">
@@ -62,6 +52,6 @@
         <xacro:unless value="$(arg use_sim)">
           <plugin>rosbot_hardware_interfaces/RosbotSystem</plugin>
-          <param name="connection_timeout_ms">120000</param>
-          <param name="connection_check_period_ms">500</param>
+          <param name="connection_timeout_ms">30000</param>
+          <param name="connection_check_period_ms">1000</param>
           <!-- order of velocity commands to be published in motors_cmd Float32MultiArray msg -->
           <param name="velocity_command_joint_order">
