Commit message: Simplify URDF

File: rosbot_description/urdf/common/gazebo.urdf.xacro (robot description, xacro)
@@ -34,5 +34,4 @@
         <visualize>false</visualize>
         <enable_metrics>false</enable_metrics>
-        <frame_id>imu_link</frame_id>
         <gz_frame_id>imu_link</gz_frame_id>
         <imu>

File: rosbot_description/urdf/rosbot.urdf.xacro (robot description, xacro)
@@ -1,18 +1,19 @@
 <?xml version='1.0'?>
 <robot name="rosbot" xmlns:xacro="http://www.ros.org/wiki/xacro">
-  <xacro:arg name="use_sim" default="false" />
+  <xacro:arg name="controller_config" default="$(find rosbot_controller)/config/rosbot_xl/diff_drive_controller.yaml" />
   <xacro:arg name="mecanum" default="false" />
   <xacro:arg name="namespace" default="" />
+  <xacro:arg name="use_sim" default="false" />
   <xacro:include filename="$(find rosbot_description)/urdf/rosbot/rosbot_macro.urdf.xacro" ns="husarion" />
   <xacro:include filename="$(find ros_components_description)/urdf/slamtec_rplidar.urdf.xacro" ns="lidar" />
 	<xacro:include filename="$(find depthai_descriptions)/urdf/include/depthai_macro.urdf.xacro" ns="camera" />
   <xacro:husarion.rosbot
+    controller_config="$(arg controller_config)"
     mecanum="$(arg mecanum)"
-    use_sim="$(arg use_sim)"
-    namespace="$(arg namespace)" />
+    namespace="$(arg namespace)"
+    use_sim="$(arg use_sim)" />
   <xacro:lidar.slamtec_rplidar
     parent_link="cover_link"
     xyz="0.02 0.0 0.0"
-    rpy="0.0 0.0 0.0"
     model="s2"
     namespace="$(arg namespace)" />

File: rosbot_description/urdf/rosbot/body.urdf.xacro (robot description, xacro)
@@ -2,5 +2,5 @@
 <robot xmlns:xacro="http://www.ros.org/wiki/xacro">
   <!-- body defining macro -->
-  <xacro:macro name="body" params="wheel_radius mecanum namespace">
+  <xacro:macro name="body" params="wheel_radius namespace">
     <xacro:include filename="$(find rosbot_description)/urdf/rosbot/components/vl53lox.urdf.xacro" ns="range_sensor" />
     <link name="base_link" />

File: rosbot_description/urdf/rosbot/rosbot_macro.urdf.xacro (robot description, xacro)
@@ -1,121 +1,38 @@
 <?xml version='1.0'?>
 <robot xmlns:xacro="http://wiki.ros.org/xacro">
-  <xacro:macro name="rosbot" params="mecanum namespace use_sim">
+  <xacro:macro name="rosbot"
+    params="controller_config
+            mecanum
+            namespace
+            use_sim">
+    <!-- PROPERTIES -->
     <xacro:property name="ns" value="${namespace + '/' if namespace != '' else ''}" />
-    <xacro:property name="wheel_radius" value="${0.0470 if mecanum else 0.0425}" />
-    <!-- INCLUDE ROBOT PARTS DEFINITIONS -->
+    <xacro:property name="wheel_radius" value="${0.047 if mecanum else 0.0425}" />
+    <!-- INCLUDE ROBOT MACRO -->
+    <xacro:include filename="$(find rosbot_description)/urdf/common/gazebo.urdf.xacro" ns="gazebo" />
+    <xacro:include filename="$(find rosbot_description)/urdf/common/ros2_control.urdf.xacro" ns="ros2_control" />
+    <!-- <xacro:include filename="$(find rosbot_description)/urdf/common/webots.urdf.xacro" ns="webots" /> -->
     <xacro:include filename="$(find rosbot_description)/urdf/rosbot/body.urdf.xacro" ns="body" />
     <xacro:include filename="$(find rosbot_description)/urdf/rosbot/wheel.urdf.xacro" ns="wheel" />
-    <!-- BODY DECLARATION -->
-    <xacro:body.body wheel_radius="${wheel_radius}" mecanum="${mecanum}" namespace="${namespace}" />
-    <!-- WHEEL DECLARATION -->
+    <!-- BODY -->
+    <xacro:body.body wheel_radius="${wheel_radius}" namespace="${namespace}" />
+    <!-- WHEEL -->
+    <xacro:wheel.wheel wheel_radius="${wheel_radius}" side="fl" mecanum="${mecanum}" />
     <xacro:wheel.wheel wheel_radius="${wheel_radius}" side="fr" mecanum="${mecanum}" />
-    <xacro:wheel.wheel wheel_radius="${wheel_radius}" side="fl" mecanum="${mecanum}" />
     <xacro:wheel.wheel wheel_radius="${wheel_radius}" side="rl" mecanum="${mecanum}" />
     <xacro:wheel.wheel wheel_radius="${wheel_radius}" side="rr" mecanum="${mecanum}" />
-    <!-- ROS2 CONTROL -->
-    <xacro:unless value="$(arg use_sim)">
-      <ros2_control name="${ns}imu" type="sensor">
-        <hardware>
-          <plugin>rosbot_hardware_interfaces/RosbotImuSensor</plugin>
-          <param name="connection_timeout_ms">30000</param>
-          <param name="connection_check_period_ms">1000</param>
-        </hardware>
-        <sensor name="${ns}imu">
-          <state_interface name="orientation.x" />
-          <state_interface name="orientation.y" />
-          <state_interface name="orientation.z" />
-          <state_interface name="orientation.w" />
-          <state_interface name="angular_velocity.x" />
-          <state_interface name="angular_velocity.y" />
-          <state_interface name="angular_velocity.z" />
-          <state_interface name="linear_acceleration.x" />
-          <state_interface name="linear_acceleration.y" />
-          <state_interface name="linear_acceleration.z" />
-        </sensor>
-      </ros2_control>
+    <!-- HARDWARE PLUGINS -->
+    <xacro:unless value="${use_sim}">
+      <xacro:ros2_control.imu namespace="${namespace}" />
+      <xacro:ros2_control.rosbot_system namespace="${namespace}" />
     </xacro:unless>
-    <ros2_control name="${ns}rosbot_system" type="system">
-      <hardware>
-        <xacro:unless value="$(arg use_sim)">
-          <plugin>rosbot_hardware_interfaces/RosbotSystem</plugin>
-          <param name="connection_timeout_ms">30000</param>
-          <param name="connection_check_period_ms">1000</param>
-          <!-- Firmware from https://github.com/husarion/rosbot_ros2_firmware could not override this names -->
-          <param name="velocity_command_joint_order">
-                rr_wheel_joint,
-                rl_wheel_joint,
-                fr_wheel_joint,
-                fl_wheel_joint
-          </param>
-        </xacro:unless>
-        <xacro:if value="$(arg use_sim)">
-          <plugin>gz_ros2_control/GazeboSimSystem</plugin>
-        </xacro:if>
-      </hardware>
-      <joint name="fl_wheel_joint">
-        <command_interface name="velocity" />
-        <state_interface name="position" />
-        <state_interface name="velocity" />
-      </joint>
-      <joint name="fr_wheel_joint">
-        <command_interface name="velocity" />
-        <state_interface name="position" />
-        <state_interface name="velocity" />
-      </joint>
-      <joint name="rl_wheel_joint">
-        <command_interface name="velocity" />
-        <state_interface name="position" />
-        <state_interface name="velocity" />
-      </joint>
-      <joint name="rr_wheel_joint">
-        <command_interface name="velocity" />
-        <state_interface name="position" />
-        <state_interface name="velocity" />
-      </joint>
-      <xacro:if value="${use_sim}">
-        <sensor name="${ns}imu">
-          <state_interface name="orientation.x" />
-          <state_interface name="orientation.y" />
-          <state_interface name="orientation.z" />
-          <state_interface name="orientation.w" />
-          <state_interface name="angular_velocity.x" />
-          <state_interface name="angular_velocity.y" />
-          <state_interface name="angular_velocity.z" />
-          <state_interface name="linear_acceleration.x" />
-          <state_interface name="linear_acceleration.y" />
-          <state_interface name="linear_acceleration.z" />
-        </sensor>
-      </xacro:if>
-    </ros2_control>
-    <!-- GAZEBO PLUGINS DECLARATION -->
+    <!-- GAZEBO PLUGINS -->
     <xacro:if value="${use_sim}">
-      <gazebo>
-        <plugin filename="gz_ros2_control-system" name="gz_ros2_control::GazeboSimROS2ControlPlugin">
-          <xacro:if value="${mecanum}">
-            <parameters>$(find rosbot_controller)/config/rosbot/mecanum_drive_controller.yaml</parameters>
-          </xacro:if>
-          <xacro:unless value="${mecanum}">
-            <parameters>$(find rosbot_controller)/config/rosbot/diff_drive_controller.yaml</parameters>
-          </xacro:unless>
-          <ros>
-            <namespace>${ns}</namespace>
-            <remapping>rosbot_base_controller/cmd_vel:=cmd_vel</remapping>
-          </ros>
-        </plugin>
-      </gazebo>
-      <gazebo reference="imu_link">
-        <sensor name="${ns}imu" type="imu">
-          <always_on>true</always_on>
-          <update_rate>25</update_rate>
-          <topic>imu/data_raw</topic>
-          <visualize>false</visualize>
-          <enable_metrics>false</enable_metrics>
-          <gz_frame_id>imu_link</gz_frame_id>
-          <ros>
-            <namespace>${namespace}</namespace>
-          </ros>
-        </sensor>
-      </gazebo>
+      <xacro:ros2_control.gz_rosbot_system namespace="${namespace}" />
+      <xacro:gazebo.controller config_file="${controller_config}" namespace="${namespace}" />
+      <xacro:gazebo.imu reference_frame="imu_link" namespace="${namespace}" />
+      <!-- <xacro:if value="${simulation_engine == 'webots'}">
+        <xacro:webots.controller />
+      </xacro:if> -->
     </xacro:if>
   </xacro:macro>

File: rosbot_description/urdf/rosbot/wheel.urdf.xacro (robot description, xacro)
@@ -2,5 +2,5 @@
 <robot xmlns:xacro="http://www.ros.org/wiki/xacro">
   <!-- wheel defining macro -->
-  <xacro:macro name="wheel" params="wheel_radius side mecanum ">
+  <xacro:macro name="wheel" params="mecanum side wheel_radius">
     <xacro:property name="wheel_separation_x" value="0.106" />
     <xacro:if value="${mecanum}">

File: rosbot_description/urdf/rosbot_xl.urdf.xacro (robot description, xacro)
@@ -2,5 +2,5 @@
 <robot name="rosbot_xl" xmlns:xacro="http://www.ros.org/wiki/xacro">
   <xacro:arg name="components_config" default="$(find rosbot_description)/config/components.yaml" />
-  <xacro:arg name="controller_config" default="$(find rosbot_controller)/config/diff_drive_controller.yaml" />
+  <xacro:arg name="controller_config" default="$(find rosbot_controller)/config/rosbot_xl/diff_drive_controller.yaml" />
   <xacro:arg name="include_camera_mount" default="false" />
   <xacro:arg name="mecanum" default="false" />
@@ -9,18 +9,10 @@
   <xacro:include filename="$(find rosbot_description)/urdf/rosbot_xl/rosbot_xl_macro.urdf.xacro"
     ns="husarion" />
-  <xacro:husarion.rosbot_robot
+  <xacro:husarion.rosbot_xl
     controller_config="$(arg controller_config)"
+    include_camera_mount="$(arg include_camera_mount)"
     mecanum="$(arg mecanum)"
     namespace="$(arg namespace)"
     use_sim="$(arg use_sim)" />
-  <xacro:if value="$(arg include_camera_mount)">
-    <xacro:include filename="$(find rosbot_description)/urdf/rosbot_xl/components/camera_mount.urdf.xacro" ns="camera_mount" />
-    <xacro:camera_mount.camera_mount
-      parent_link="cover_link"
-      xyz="-0.1 0.0 0.0"
-      rpy="0.0 0.0 0.0"
-      camera_mount_angle_1="0.0"
-      camera_mount_angle_2="0.0" />
-  </xacro:if>
   <xacro:include filename="$(find ros_components_description)/urdf/components.urdf.xacro" ns="components" />
   <xacro:components.create_components

File: rosbot_description/urdf/rosbot_xl/components/antenna.urdf.xacro (robot description, xacro)
@@ -2,21 +2,18 @@
 <robot xmlns:xacro="http://www.ros.org/wiki/xacro">
   <xacro:macro name="antenna"
-    params="parent_link xyz rpy
-            tf_prefix:=None
-            antenna_angle:=0.0">
-    <xacro:if value="${tf_prefix == 'None'}">
-      <xacro:property name="tf_prefix_ext" value="" />
-    </xacro:if>
-    <xacro:unless value="${tf_prefix == 'None'}">
-      <xacro:property name="tf_prefix_ext" value="${tf_prefix}_" />
-    </xacro:unless>
+               params="parent_link
+                       xyz:='0.0 0.0 0.0'
+                       rpy:='0.0 0.0 0.0'
+                       tf_prefix:=''
+                       antenna_angle:=0.0">
+    <xacro:property name="prefix" value="${tf_prefix + '_' if tf_prefix != '' else ''}" />
     <xacro:property name="antenna_length" value="0.1" />
     <xacro:property name="antenna_radius" value="0.0052" />
-    <joint name="${parent_link.rstrip('_link')}_to_${tf_prefix_ext}antenna_connector_joint" type="fixed">
+    <joint name="${parent_link.rstrip('_link')}_to_${prefix}antenna_connector_joint" type="fixed">
       <origin xyz="${xyz}" rpy="${rpy}" />
       <parent link="${parent_link}" />
-      <child link="${tf_prefix_ext}antenna_connector_link" />
+      <child link="${prefix}antenna_connector_link" />
     </joint>
-    <link name="${tf_prefix_ext}antenna_connector_link">
+    <link name="${prefix}antenna_connector_link">
       <visual>
         <geometry>
@@ -27,10 +24,10 @@
       </visual>
     </link>
-    <joint name="${tf_prefix_ext}antenna_connector_to_${tf_prefix_ext}antenna_joint" type="fixed">
+    <joint name="${prefix}antenna_connector_to_${prefix}antenna_joint" type="fixed">
       <origin xyz="-0.013 0.0 0.008" rpy="0.0 ${antenna_angle} 0.0" />
-      <parent link="${tf_prefix_ext}antenna_connector_link" />
-      <child link="${tf_prefix_ext}antenna_link" />
+      <parent link="${prefix}antenna_connector_link" />
+      <child link="${prefix}antenna_link" />
     </joint>
-    <link name="${tf_prefix_ext}antenna_link">
+    <link name="${prefix}antenna_link">
       <visual>
         <geometry>

File: rosbot_description/urdf/rosbot_xl/components/camera_mount.urdf.xacro (robot description, xacro)
@@ -2,25 +2,21 @@
 <robot xmlns:xacro="http://www.ros.org/wiki/xacro">
   <xacro:macro name="camera_mount"
-    params="parent_link xyz rpy
-                       tf_prefix:=None
+               params="parent_link
+                       xyz:='0.0 0.0 0.0'
+                       rpy:='0.0 0.0 0.0'
+                       tf_prefix:=''
                        camera_mount_angle_1:=0.0
                        camera_mount_angle_2:=0.0">
-    <xacro:if value="${tf_prefix == 'None'}">
-      <xacro:property name="tf_prefix_ext" value="" />
-    </xacro:if>
-    <xacro:unless value="${tf_prefix == 'None'}">
-      <xacro:property name="tf_prefix_ext" value="${tf_prefix}_" />
-    </xacro:unless>
-    <joint name="${parent_link.rstrip('_link')}_to_${tf_prefix_ext}camera_mount_bot_joint"
+    <xacro:property name="prefix" value="${tf_prefix + '_' if tf_prefix != '' else ''}" />
+    <joint name="${parent_link.rstrip('_link')}_to_${prefix}camera_mount_bot_joint"
       type="fixed">
       <origin xyz="${xyz}" rpy="${rpy}" />
       <parent link="${parent_link}" />
-      <child link="${tf_prefix_ext}camera_mount_bot_link" />
+      <child link="${prefix}camera_mount_bot_link" />
     </joint>
-    <link name="${tf_prefix_ext}camera_mount_bot_link">
+    <link name="${prefix}camera_mount_bot_link">
       <visual>
         <geometry>
-          <mesh filename="package://rosbot_description/meshes/rosbot_xl/components/camera_mount_bot.dae"
-      scale="1 1 1" />
+          <mesh filename="package://rosbot_description/meshes/rosbot_xl/components/camera_mount_bot.dae" scale="1 1 1" />
         </geometry>
         <origin xyz="0.0 0.0 0.0" rpy="0.0 0.0 0.0" />
@@ -33,15 +29,13 @@
       </collision>
     </link>
-    <joint name="${tf_prefix_ext}camera_mount_bot_to_${tf_prefix_ext}camera_mount_mid_joint"
-      type="fixed">
+    <joint name="${prefix}camera_mount_bot_to_${prefix}camera_mount_mid_joint" type="fixed">
       <origin xyz="0.0 0.0 0.016" rpy="0.0 ${camera_mount_angle_1} 0.0" />
-      <parent link="${tf_prefix_ext}camera_mount_bot_link" />
-      <child link="${tf_prefix_ext}camera_mount_mid_link" />
+      <parent link="${prefix}camera_mount_bot_link" />
+      <child link="${prefix}camera_mount_mid_link" />
     </joint>
-    <link name="${tf_prefix_ext}camera_mount_mid_link">
+    <link name="${prefix}camera_mount_mid_link">
       <visual>
         <geometry>
-          <mesh filename="package://rosbot_description/meshes/rosbot_xl/components/camera_mount_mid.dae"
-      scale="1 1 1" />
+          <mesh filename="package://rosbot_description/meshes/rosbot_xl/components/camera_mount_mid.dae" scale="1 1 1" />
         </geometry>
         <origin xyz="0.0 0.0 0.0" rpy="0.0 0.0 0.0" />
@@ -54,11 +48,10 @@
       </collision>
     </link>
-    <joint name="${tf_prefix_ext}camera_mount_mid_to_${tf_prefix_ext}camera_mount_top_joint"
-      type="fixed">
+    <joint name="${prefix}camera_mount_mid_to_${prefix}camera_mount_top_joint" type="fixed">
       <origin xyz="0.0 0.0 0.086" rpy="0.0 ${camera_mount_angle_2} 0.0" />
-      <parent link="${tf_prefix_ext}camera_mount_mid_link" />
-      <child link="${tf_prefix_ext}camera_mount_top_link" />
+      <parent link="${prefix}camera_mount_mid_link" />
+      <child link="${prefix}camera_mount_top_link" />
     </joint>
-    <link name="${tf_prefix_ext}camera_mount_top_link">
+    <link name="${prefix}camera_mount_top_link">
       <visual>
         <geometry>
@@ -75,11 +68,11 @@
       </collision>
     </link>
-    <joint name="${tf_prefix_ext}camera_mount_top_to_${tf_prefix_ext}camera_mount_joint"
+    <joint name="${prefix}camera_mount_top_to_${prefix}camera_mount_joint"
       type="fixed">
       <origin xyz="0.0 -0.00232 0.019" rpy="0.0 0.0 0.0" />
-      <parent link="${tf_prefix_ext}camera_mount_top_link" />
-      <child link="${tf_prefix_ext}camera_mount_link" />
+      <parent link="${prefix}camera_mount_top_link" />
+      <child link="${prefix}camera_mount_link" />
     </joint>
-    <link name="${tf_prefix_ext}camera_mount_link" />
+    <link name="${prefix}camera_mount_link" />
   </xacro:macro>
 </robot>
