Commit message: Simplify URDF

File: rosbot_description/urdf/rosbot_xl/rosbot_xl_macro.urdf.xacro (robot description, xacro)
@@ -1,104 +1,45 @@
 <?xml version='1.0'?>
 <robot xmlns:xacro="http://wiki.ros.org/xacro">
-  <xacro:macro name="rosbot_robot"
+  <xacro:macro name="rosbot_xl"
     params="controller_config
+            include_camera_mount
             mecanum
             namespace
             use_sim">
+    <!-- PROPERTIES -->
     <xacro:property name="ns" value="${namespace + '/' if namespace != '' else ''}" />
     <xacro:property name="wheel_radius" value="${0.05 if mecanum else 0.048}" />
-    <!-- INCLUDE ROBOT PARTS DEFINITIONS -->
+    <!-- INCLUDE ROBOT MACRO -->
+    <xacro:include filename="$(find rosbot_description)/urdf/common/gazebo.urdf.xacro" ns="gazebo" />
+    <xacro:include filename="$(find rosbot_description)/urdf/common/ros2_control.urdf.xacro" ns="ros2_control" />
+    <!-- <xacro:include filename="$(find rosbot_description)/urdf/common/webots.urdf.xacro" ns="webots" /> -->
     <xacro:include filename="$(find rosbot_description)/urdf/rosbot_xl/body.urdf.xacro" ns="body" />
     <xacro:include filename="$(find rosbot_description)/urdf/rosbot_xl/components/antenna.urdf.xacro" ns="antenna" />
-    <xacro:include filename="$(find rosbot_description)/urdf/rosbot_xl/gazebo.urdf.xacro" ns="gazebo" />
-    <xacro:include filename="$(find rosbot_description)/urdf/rosbot_xl/webots.urdf.xacro" ns="webots" />
     <xacro:include filename="$(find rosbot_description)/urdf/rosbot_xl/wheel.urdf.xacro" ns="wheel" />
-    <!-- BODY DECLARATION -->
+    <xacro:include filename="$(find rosbot_description)/urdf/rosbot_xl/components/camera_mount.urdf.xacro" ns="camera_mount" />
+    <!-- BODY -->
     <xacro:body.body wheel_radius="${wheel_radius}" />
-    <!-- ANTENNA DECLARATION -->
-    <xacro:antenna.antenna parent_link="body_link" xyz="-0.155 -0.055 0.065" rpy="0.0 0.0 0.0" antenna_angle="0.0" />
-    <!-- WHEEL DECLARATION -->
+    <xacro:antenna.antenna parent_link="cover_link" xyz="-0.155 -0.055 -0.02" />
+    <xacro:if value="$(arg include_camera_mount)">
+      <xacro:camera_mount.camera_mount parent_link="cover_link" xyz="-0.1 0.0 0.0" />
+    </xacro:if>
+    <!-- WHEEL -->
     <xacro:wheel.wheel wheel_radius="${wheel_radius}" side="fl" mecanum="${mecanum}" />
     <xacro:wheel.wheel wheel_radius="${wheel_radius}" side="fr" mecanum="${mecanum}" />
     <xacro:wheel.wheel wheel_radius="${wheel_radius}" side="rl" mecanum="${mecanum}" />
     <xacro:wheel.wheel wheel_radius="${wheel_radius}" side="rr" mecanum="${mecanum}" />
-    <!-- ROS2 CONTROL -->
-    <xacro:unless value="$(arg use_sim)">
-      <ros2_control name="${ns}imu" type="sensor">
-        <hardware>
-          <plugin>rosbot_hardware_interfaces/RosbotImuSensor</plugin>
-          <param name="connection_timeout_ms">30000</param>
-          <param name="connection_check_period_ms">1000</param>
-        </hardware>
-        <sensor name="${ns}imu">
-          <state_interface name="orientation.x" />
-          <state_interface name="orientation.y" />
-          <state_interface name="orientation.z" />
-          <state_interface name="orientation.w" />
-          <state_interface name="angular_velocity.x" />
-          <state_interface name="angular_velocity.y" />
-          <state_interface name="angular_velocity.z" />
-          <state_interface name="linear_acceleration.x" />
-          <state_interface name="linear_acceleration.y" />
-          <state_interface name="linear_acceleration.z" />
-        </sensor>
-      </ros2_control>
+    <!-- HARDWARE PLUGINS -->
+    <xacro:unless value="${use_sim}">
+      <xacro:ros2_control.imu namespace="${namespace}" />
+      <xacro:ros2_control.rosbot_system namespace="${namespace}" />
     </xacro:unless>
-    <ros2_control name="${ns}wheels" type="system">
-      <hardware>
-        <xacro:if value="${use_sim}">
-          <plugin>gz_ros2_control/GazeboSimSystem</plugin>
-        </xacro:if>
-        <xacro:unless value="$(arg use_sim)">
-          <plugin>rosbot_hardware_interfaces/RosbotSystem</plugin>
-          <param name="connection_timeout_ms">30000</param>
-          <param name="connection_check_period_ms">1000</param>
-          <!-- order of velocity commands to be published in motors_cmd Float32MultiArray msg -->
-          <param name="velocity_command_joint_order">
-            rr_wheel_joint,
-            rl_wheel_joint,
-            fr_wheel_joint,
-            fl_wheel_joint
-          </param>
-        </xacro:unless>
-      </hardware>
-      <joint name="fl_wheel_joint">
-        <command_interface name="velocity" />
-        <state_interface name="position" />
-        <state_interface name="velocity" />
-      </joint>
-      <joint name="fr_wheel_joint">
-        <command_interface name="velocity" />
-        <state_interface name="position" />
-        <state_interface name="velocity" />
-      </joint>
-      <joint name="rl_wheel_joint">
-        <command_interface name="velocity" />
-        <state_interface name="position" />
-        <state_interface name="velocity" />
-      </joint>
-      <joint name="rr_wheel_joint">
-        <command_interface name="velocity" />
-        <state_interface name="position" />
-        <state_interface name="velocity" />
-      </joint>
-      <xacro:if value="${use_sim}">
-        <sensor name="${ns}imu">
-          <state_interface name="orientation.x" />
-          <state_interface name="orientation.y" />
-          <state_interface name="orientation.z" />
-          <state_interface name="orientation.w" />
-          <state_interface name="angular_velocity.x" />
-          <state_interface name="angular_velocity.y" />
-          <state_interface name="angular_velocity.z" />
-          <state_interface name="linear_acceleration.x" />
-          <state_interface name="linear_acceleration.y" />
-          <state_interface name="linear_acceleration.z" />
-        </sensor>
-      </xacro:if>
-    </ros2_control>
+    <!-- GAZEBO PLUGINS -->
     <xacro:if value="${use_sim}">
+      <xacro:ros2_control.gz_rosbot_system namespace="${namespace}" />
       <xacro:gazebo.controller config_file="${controller_config}" namespace="${namespace}" />
       <xacro:gazebo.imu reference_frame="imu_link" namespace="${namespace}" />
+      <!-- <xacro:if value="${simulation_engine == 'webots'}">
+        <xacro:webots.controller />
+      </xacro:if> -->
     </xacro:if>
   </xacro:macro>

File: rosbot_description/urdf/rosbot_xl/wheel.urdf.xacro (robot description, xacro)
@@ -1,5 +1,5 @@
 <?xml version="1.0" encoding="utf-8"?>
 <robot xmlns:xacro="http://www.ros.org/wiki/xacro">
-  <xacro:macro name="wheel" params="wheel_radius side mecanum">
+  <xacro:macro name="wheel" params="mecanum side wheel_radius">
     <xacro:property name="wheel_separation_x" value="0.170" />
     <xacro:if value="${mecanum}">

Commit message: Fix hw and sim tests

File: rosbot_description/urdf/common/gazebo.urdf.xacro (robot description, xacro)
@@ -7,6 +7,8 @@
         <ros>
           <namespace>${namespace}</namespace>
+          <remapping>/diagnostics:=diagnostics</remapping>
           <remapping>rosbot_base_controller/cmd_vel:=cmd_vel</remapping>
           <remapping>/tf:=tf</remapping>
+          <remapping>/tf_static:=tf_static</remapping>
         </ros>
       </plugin>

File: rosbot_description/urdf/rosbot.urdf.xacro (robot description, xacro)
@@ -1,5 +1,5 @@
 <?xml version='1.0'?>
 <robot name="rosbot" xmlns:xacro="http://www.ros.org/wiki/xacro">
-  <xacro:arg name="controller_config" default="$(find rosbot_controller)/config/rosbot/diff_drive_controller.yaml" />
+  <xacro:arg name="controller_config" default="" />
   <xacro:arg name="mecanum" default="false" />
   <xacro:arg name="namespace" default="" />

File: rosbot_description/urdf/rosbot/rosbot_macro.urdf.xacro (robot description, xacro)
@@ -7,5 +7,4 @@
             use_sim">
     <!-- PROPERTIES -->
-    <xacro:property name="ns" value="${namespace + '/' if namespace != '' else ''}" />
     <xacro:property name="wheel_radius" value="${0.047 if mecanum else 0.0425}" />
     <!-- INCLUDE ROBOT MACRO -->

File: rosbot_description/urdf/rosbot_xl.urdf.xacro (robot description, xacro)
@@ -2,5 +2,5 @@
 <robot name="rosbot_xl" xmlns:xacro="http://www.ros.org/wiki/xacro">
   <xacro:arg name="components_config" default="$(find rosbot_description)/config/components.yaml" />
-  <xacro:arg name="controller_config" default="$(find rosbot_controller)/config/rosbot_xl/diff_drive_controller.yaml" />
+  <xacro:arg name="controller_config" default="" />
   <xacro:arg name="include_camera_mount" default="false" />
   <xacro:arg name="mecanum" default="false" />

File: rosbot_description/urdf/rosbot_xl/rosbot_xl_macro.urdf.xacro (robot description, xacro)
@@ -8,5 +8,4 @@
             use_sim">
     <!-- PROPERTIES -->
-    <xacro:property name="ns" value="${namespace + '/' if namespace != '' else ''}" />
     <xacro:property name="wheel_radius" value="${0.05 if mecanum else 0.048}" />
     <!-- INCLUDE ROBOT MACRO -->
